File: PCB/Kicad/io_controller/timer.kicad_sch (KiCad schematic)
At the start: 5 parts, among them U7 NE555D, U8 74LS377

Commit message: initial version of io controller schematic
Parts:
- removed U8: 74LS377, symbol 74xx:74LS377
- added U38: 74LS195, symbol 74xx:74LS195
Connections:
- net VCC: now also U7.4 (R), U38.16 (VCC), U38.7 (P3)
- net clk: now also U38.10 (CP)
- net clkint_en: now also U38.9 (~{PE}); no longer U7.4 (R)
- net timerpulse renamed pulse
- net pulse: now also U38.2 (J), U38.3 (~{K})
- new net: U38.14 (Q1), U38.5 (P1)
- new net: U38.15 (Q0), U38.4 (P0)
- new net int: U38.13 (Q2), U38.6 (P2)
- new net ~{read}: U38.1 (~{MR})
- no-connect marks 7 -> 3
Other:
- note added: "when clkint_en goes low, SR stops changing"

Commit message: io controller WIP ; simulated timer ; adjusted decoder ; adjusted LEDs
Parts:
- added Ct2, Ct3: 0.1u, Capacitor_SMD:C_0603_1608Metric, symbol Device:C
- added Dt1: yellow, LED_SMD:LED_0603_1608Metric, symbol Device:LED
- added Rt3: 680, Resistor_SMD:R_0402_1005Metric, symbol Device:R
- Ct1: renamed from C7; footprint (none) -> Capacitor_SMD:C_Elec_3x5.4
- Rt1: renamed from R17; footprint (none) -> Resistor_SMD:R_0402_1005Metric
- Rt2: renamed from R18; footprint (none) -> Resistor_SMD:R_0402_1005Metric
- Ut2: renamed from U38; footprint (none) -> Package_SO:SOIC-16_3.9x9.9mm_P1.27mm
- renumbered U7 to Ut1
Connections:
- net GND: now also Ut2.8 (GND), Ct2.2, Ct3.2, Rt3.2
- net VCC: now also Ct2.1, Ct3.1
- net int: now also Dt1.2 (A)
- net q1: now reaches Ut2.14 (Q1), Ut2.5 (P1)
- net q0: now reaches Ut2.15 (Q0), Ut2.4 (P0)
- net pulse: no longer names the net of Ut1.3 (Q), Ut2.2 (J), Ut2.3 (~{K})
- new net: Dt1.1 (K), Rt3.1
Other:
- note added: "somewhat breaks when reading more often than once every 1ms"
- note added: "when clkint_en goes low, shiftreg stops changing"
- note removed: "I hope these values are right, doublecheck them w/ datasheet to get ~1ms cycle"
- note removed: "when clkint_en goes low, SR stops changing"
- company: (none) -> AGH Logic Unit
- title: (none) -> Timer

Commit message: primarily keyboard decoder finish ; preliminary layout
Connections:
- net VCC: no longer Ut1.4 (R)
- new net enable: Ut1.4 (R)
Changed lines of the file:
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@@
 	(wire
 		(pts
-			(xy 46.355 72.39) (xy 50.8 72.39)
+			(xy 76.2 62.23) (xy 113.03 62.23)
 		)
 		(stroke
@@
 	(wire
 		(pts
-			(xy 76.2 62.23) (xy 113.03 62.23)
+			(xy 132.08 74.93) (xy 132.08 80.01)
 		)
 		(stroke
@@
 		)
 	)
-	(wire
-		(pts
-			(xy 132.08 74.93) (xy 132.08 80.01)
-		)
-		(stroke
-			(width 0)
-			(type default)
-		)
-	)
 	(label "q1"
 		(at 137.795 64.77 180)
@@
 		)
 	)
-	(label "q2"
-		(at 163.195 67.31 0)
-		(effects
-			(font
-				(size 1.27 1.27)
-			)
-			(justify left bottom)
-		)
-	)
-	(label "q2"
-		(at 137.795 67.31 180)
-		(effects
-			(font
-				(size 1.27 1.27)
-			)
-			(justify right bottom)
-		)
-	)
 	(label "q0"
 		(at 137.795 62.23 180)
@@
 			)
 			(justify left bottom)
+		)
+	)
+	(label "int"
+		(at 137.795 67.31 180)
+		(effects
+			(font
+				(size 1.27 1.27)
+			)
+			(justify right bottom)
 		)
 	)
@@
 		(shape input)
 		(at 137.795 77.47 180)
+		(effects
+			(font
+				(size 1.27 1.27)
+			)
+			(justify right)
+		)
+	)
+	(hierarchical_label "enable"
+		(shape input)
+		(at 50.8 72.39 180)
 		(effects
 			(font
@@
 					(unit 1)
 				)
-			)
-		)
-	)
-	(symbol
-		(lib_id "power:VCC")
-		(at 46.355 72.39 0)
-		(unit 1)
-		(exclude_from_sim no)
-		(in_bom yes)
-		(on_board yes)
-		(dnp no)
-		(fields_autoplaced yes)
-		(property "Reference" "#PWR0131"
-			(at 46.355 76.2 0)
-			(effects
-				(font
-					(size 1.27 1.27)
-				)
-				(hide yes)
-			)
-		)
-		(property "Value" "VCC"
-			(at 46.355 67.31 0)
-			(effects
-				(font
-					(size 1.27 1.27)
-				)
-			)
-		)
-		(property "Footprint" ""
-			(at 46.355 72.39 0)
-			(effects
-				(font
-					(size 1.27 1.27)
-				)
-				(hide yes)
-			)
-		)
-		(property "Datasheet" ""
-			(at 46.355 72.39 0)
-			(effects
-				(font
-					(size 1.27 1.27)
-				)
-				(hide yes)
-			)
-		)
-		(property "Description" "Power symbol creates a global label with name \"VCC\""
-			(at 46.355 72.39 0)
-			(effects
-				(font
-					(size 1.27 1.27)
-				)
-				(hide yes)
-			)
-		)
-		(pin "1"
-		)
-		(instances
-			(project ""
-				(path "/dccec861-b967-466c-843e-d6d1ad6064ce/b2a66210-0f57-47f7-af2e-0fa71fd479f3"
-					(reference "#PWR0131")
-					(unit 1)
-				)
