File: PCB/Kicad/io_controller/io_controller.kicad_pcb (KiCad board)
At the start: 6 copper layers, 0 parts

Commit message: io controller WIP ; simulated timer ; adjusted decoder ; adjusted LEDs
Parts:
- added C1: 0.1u, Capacitor_SMD:C_0402_1005Metric, F.Cu at (97.5, 62.0)
- added C2: 0.1u, Capacitor_SMD:C_0402_1005Metric, F.Cu at (80.0, 62.0)
- added Cd1: 0.1u, Capacitor_SMD:C_0402_1005Metric, F.Cu at (54.9, 49.5)
- added Cd2: 0.1u, Capacitor_SMD:C_0402_1005Metric, F.Cu at (54.9, 59.5)
- added Cd3: 0.1u, Capacitor_SMD:C_0402_1005Metric, F.Cu at (54.9, 69.5)
- added Cd4: 0.1u, Capacitor_SMD:C_0402_1005Metric, F.Cu at (42.4, 49.5)
- added Cd5: 0.1u, Capacitor_SMD:C_0402_1005Metric, F.Cu at (42.4, 59.5)
- added Cd6: 0.1u, Capacitor_SMD:C_0402_1005Metric, F.Cu at (42.4, 69.5)
- added Cd7: 0.1u, Capacitor_SMD:C_0402_1005Metric, F.Cu at (54.9, 39.5)
- added Ct1: 33n, Capacitor_SMD:C_Elec_3x5.4, F.Cu at (123.0, 35.0)
- added Ct2: 0.1u, Capacitor_SMD:C_0603_1608Metric, F.Cu at (127.9, 26.0)
- added Ct3: 0.1u, Capacitor_SMD:C_0603_1608Metric, F.Cu at (116.0, 29.0)
- added Dd1: yellow, LED_SMD:LED_0603_1608Metric, F.Cu at (26.8, 25.0)
- added Dd2: yellow, LED_SMD:LED_0603_1608Metric, F.Cu at (26.8, 27.0)
- added Dd3: yellow, LED_SMD:LED_0603_1608Metric, F.Cu at (26.8, 29.0)
- added Dd4: yellow, LED_SMD:LED_0603_1608Metric, F.Cu at (26.8, 31.0)
- added Dd5: yellow, LED_SMD:LED_0603_1608Metric, F.Cu at (26.8, 33.0)
- added Dd6: yellow, LED_SMD:LED_0603_1608Metric, F.Cu at (26.8, 35.0)
- added Dl1: red, LED_SMD:LED_0603_1608Metric, F.Cu at (95.0, 70.0)
- added Dl10: red, LED_SMD:LED_0603_1608Metric, F.Cu at (77.0, 70.0)
- added Dl11: red, LED_SMD:LED_0603_1608Metric, F.Cu at (75.0, 70.0)
- added Dl12: red, LED_SMD:LED_0603_1608Metric, F.Cu at (73.0, 70.0)
- added Dl13: red, LED_SMD:LED_0603_1608Metric, F.Cu at (71.0, 70.0)
- added Dl14: red, LED_SMD:LED_0603_1608Metric, F.Cu at (69.0, 70.0)
- added Dl15: red, LED_SMD:LED_0603_1608Metric, F.Cu at (67.0, 70.0)
- added Dl16: red, LED_SMD:LED_0603_1608Metric, F.Cu at (65.0, 70.0)
- added Dl2: red, LED_SMD:LED_0603_1608Metric, F.Cu at (93.0, 70.0)
- added Dl3: red, LED_SMD:LED_0603_1608Metric, F.Cu at (91.0, 70.0)
- added Dl4: red, LED_SMD:LED_0603_1608Metric, F.Cu at (89.0, 70.0)
- added Dl5: red, LED_SMD:LED_0603_1608Metric, F.Cu at (87.0, 70.0)
- added Dl6: red, LED_SMD:LED_0603_1608Metric, F.Cu at (85.0, 70.0)
- added Dl7: red, LED_SMD:LED_0603_1608Metric, F.Cu at (83.0, 70.0)
- added Dl8: red, LED_SMD:LED_0603_1608Metric, F.Cu at (81.0, 70.0)
- added Dl9: red, LED_SMD:LED_0603_1608Metric, F.Cu at (79.0, 70.0)
- added Dt1: yellow, LED_SMD:LED_0603_1608Metric, F.Cu at (109.0, 36.0)
- added Rd1: 470, Resistor_SMD:R_0402_1005Metric, F.Cu at (22.5, 25.0)
- added Rd2: 470, Resistor_SMD:R_0402_1005Metric, F.Cu at (22.5, 27.0)
- added Rd3: 470, Resistor_SMD:R_0402_1005Metric, F.Cu at (22.5, 29.0)
- added Rd4: 470, Resistor_SMD:R_0402_1005Metric, F.Cu at (22.5, 31.0)
- added Rd5: 470, Resistor_SMD:R_0402_1005Metric, F.Cu at (22.5, 33.0)
- added Rd6: 470, Resistor_SMD:R_0402_1005Metric, F.Cu at (22.5, 35.0)
- added Rl1: 680, Resistor_SMD:R_0402_1005Metric, F.Cu at (95.0, 74.5)
- added Rl10: 680, Resistor_SMD:R_0402_1005Metric, F.Cu at (77.0, 74.5)
- added Rl11: 680, Resistor_SMD:R_0402_1005Metric, F.Cu at (75.0, 74.5)
- added Rl12: 680, Resistor_SMD:R_0402_1005Metric, F.Cu at (73.0, 74.5)
- added Rl13: 680, Resistor_SMD:R_0402_1005Metric, F.Cu at (71.0, 74.5)
- added Rl14: 680, Resistor_SMD:R_0402_1005Metric, F.Cu at (69.0, 74.5)
- added Rl15: 680, Resistor_SMD:R_0402_1005Metric, F.Cu at (67.0, 74.5)
- added Rl16: 680, Resistor_SMD:R_0402_1005Metric, F.Cu at (65.0, 74.5)
- added Rl2: 680, Resistor_SMD:R_0402_1005Metric, F.Cu at (93.0, 74.5)
- added Rl3: 680, Resistor_SMD:R_0402_1005Metric, F.Cu at (91.0, 74.5)
- added Rl4: 680, Resistor_SMD:R_0402_1005Metric, F.Cu at (89.0, 74.5)
- added Rl5: 680, Resistor_SMD:R_0402_1005Metric, F.Cu at (87.0, 74.5)
- added Rl6: 680, Resistor_SMD:R_0402_1005Metric, F.Cu at (85.0, 74.5)
- added Rl7: 680, Resistor_SMD:R_0402_1005Metric, F.Cu at (83.0, 74.5)
- added Rl8: 680, Resistor_SMD:R_0402_1005Metric, F.Cu at (81.0, 74.5)
- added Rl9: 680, Resistor_SMD:R_0402_1005Metric, F.Cu at (79.0, 74.5)
- added Rt1: 4.7k, Resistor_SMD:R_0402_1005Metric, F.Cu at (124.0, 31.0)
- added Rt2: 22k, Resistor_SMD:R_0402_1005Metric, F.Cu at (122.0, 31.0)
- added Rt3: 680, Resistor_SMD:R_0402_1005Metric, F.Cu at (105.5, 36.0)
- added Ud1: 74LS02, Package_SO:SO-14_3.9x8.65mm_P1.27mm, F.Cu at (48.9, 46.5)
- added Ud2: 74LS02, Package_SO:SO-14_3.9x8.65mm_P1.27mm, F.Cu at (48.9, 56.5)
- added Ud3: 74LS02, Package_SO:SO-14_3.9x8.65mm_P1.27mm, F.Cu at (48.9, 66.5)
- added Ud4: 74LS08, Package_SO:SOIC-14_3.9x8.7mm_P1.27mm, F.Cu at (36.5, 46.5)
- added Ud5: 74LS08, Package_SO:SOIC-14_3.9x8.7mm_P1.27mm, F.Cu at (36.5, 56.5)
- added Ud6: 74LS08, Package_SO:SOIC-14_3.9x8.7mm_P1.27mm, F.Cu at (36.5, 66.5)
- added Ud7: 74LS08, Package_SO:SOIC-14_3.9x8.7mm_P1.27mm, F.Cu at (48.9, 36.5)
- added Ul1: 74LS377, Package_SO:SOIC-20W_7.5x12.8mm_P1.27mm, F.Cu at (88.7, 57.0)
- added Ul2: 74LS377, Package_SO:SOIC-20W_7.5x12.8mm_P1.27mm, F.Cu at (72.0, 57.0)
- added Ut1: NE555D, Package_SO:SOIC-8_3.9x4.9mm_P1.27mm, F.Cu at (122.9, 26.0)
- added Ut2: 74LS195, Package_SO:SOIC-16_3.9x9.9mm_P1.27mm, F.Cu at (109.0, 26.0)
Routing:
- net /ioid0: track 0.00 -> 1.27 mm
- net /ioid1: track 0.00 -> 1.27 mm
Other:
- board outline added: 120 x 100 mm
- board text added: "Decoder"
- board text added: "LEDs"
- board text added: "LSb"
- board text added: "MSb"
- board text added: "Timer"
- board text added: "control unit interface"
- board text added: "int"
- board text added: "isclk"
- board text added: "isgpu"
- board text added: "iskeyboard"
- board text added: "isled"
- board text added: "read"
- board text added: "regfile interface"
- board text added: "write"

Commit message: more spice models and bugfixes ; more tests of io_controller - mostly keyboard
Parts:
- removed C2: 0.1u, Capacitor_SMD:C_0402_1005Metric
- removed Dl10, Dl11, Dl12, Dl13, Dl14, Dl15, Dl16, Dl9: red, LED_SMD:LED_0603_1608Metric
- removed Rl10, Rl11, Rl12, Rl13, Rl14, Rl15, Rl16, Rl9: 680, Resistor_SMD:R_0402_1005Metric
- removed Ul2: 74LS377, Package_SO:SOIC-20W_7.5x12.8mm_P1.27mm
- added Co1: 0.1u, Capacitor_SMD:C_0402_1005Metric, F.Cu at (69.8, 64.3)
- added Co2: 0.1u, Capacitor_SMD:C_0402_1005Metric, F.Cu at (90.1, 63.5)
- added J1: Conn_02x10_Odd_Even, Connector_IDC:IDC-Header_2x10_P2.54mm_Horizontal, F.Cu at (68.6, 29.8)
- added J2: Conn_02x10_Odd_Even, Connector_IDC:IDC-Header_2x10_P2.54mm_Horizontal, F.Cu at (123.2, 29.8)
- added Uki1: 74LS195, Package_SO:SOIC-16_3.9x9.9mm_P1.27mm, F.Cu at (116.5, 80.3)
- added Uki10: 74LS377, Package_SO:SSOP-20_5.3x7.2mm_P0.65mm, F.Cu at (107.1, 78.8)
- added Uki11: 74LS377, Package_SO:SSOP-20_5.3x7.2mm_P0.65mm, F.Cu at (107.1, 87.6)
- added Uki12: 74LS377, Package_SO:SSOP-20_5.3x7.2mm_P0.65mm, F.Cu at (107.1, 96.4)
- added Uki13: 74LS377, Package_SO:SSOP-20_5.3x7.2mm_P0.65mm, F.Cu at (107.1, 105.2)
- added Uki2: 74LS195, Package_SO:SOIC-16_3.9x9.9mm_P1.27mm, F.Cu at (125.0, 80.3)
- added Uki3: 74LS195, Package_SO:SOIC-16_3.9x9.9mm_P1.27mm, F.Cu at (133.4, 80.3)
- added Uki4: 74LS195, Package_SO:SOIC-16_3.9x9.9mm_P1.27mm, F.Cu at (116.5, 91.9)
- added Uki5: 74LS195, Package_SO:SOIC-16_3.9x9.9mm_P1.27mm, F.Cu at (125.0, 91.9)
- added Uki6: 74LS195, Package_SO:SOIC-16_3.9x9.9mm_P1.27mm, F.Cu at (133.4, 91.9)
- added Uki7: 74LS195, Package_SO:SOIC-16_3.9x9.9mm_P1.27mm, F.Cu at (116.5, 103.5)
- added Uki8: 74LS195, Package_SO:SOIC-16_3.9x9.9mm_P1.27mm, F.Cu at (125.0, 103.5)
- added Uki9: 74LS195, Package_SO:SOIC-16_3.9x9.9mm_P1.27mm, F.Cu at (133.4, 103.5)
- added Uo1: 74LS245, Package_SO:SOIC-20W_7.5x12.8mm_P1.27mm, F.Cu at (64.8, 72.4)
- added Uo2: 74LS245, Package_SO:SOIC-20W_7.5x12.8mm_P1.27mm, F.Cu at (94.8, 71.8)
- moved Dt1 101.0 mm to (204.8, 68.1)
- moved Rt3 101.0 mm to (201.3, 68.1)
- moved Ct1 101.0 mm to (218.8, 67.1)
- moved Ct2 101.0 mm to (223.7, 58.1)
- moved Ct3 101.0 mm to (211.8, 61.1)
- moved Rt1 101.0 mm to (219.8, 63.1)
- moved Rt2 101.0 mm to (217.8, 63.1)
- moved Ut1 101.0 mm to (218.7, 58.1)
- moved Ut2 101.0 mm to (204.8, 58.1)
- moved C1 33.0 mm to (71.6, 82.5)
- moved Ul1 31.6 mm to (79.4, 87.2), turned to 90 degrees
- moved Rl1 27.0 mm to (86.1, 100.0)
- moved Rl2 27.0 mm to (84.1, 100.0)
- moved Rl3 27.0 mm to (82.1, 100.0)
- moved Rl4 27.0 mm to (80.1, 100.0)
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Connections:
- Ud6 pad 13: /decoder/keyaval -> GND
Routing:
- net /iobus7: track 0.00 -> 28.6 mm
- net /iobus6: track 0.00 -> 28.6 mm
- net /iobus5: track 0.00 -> 28.6 mm
- net /iobus4: track 0.00 -> 28.6 mm
- net /iobus3: track 0.00 -> 28.6 mm
- net /iobus2: track 0.00 -> 28.6 mm
- net /iobus1: track 0.00 -> 28.6 mm
- net /iobus0: track 0.00 -> 28.6 mm
Other:
- board size 120 x 100 mm -> 136.5 x 100 mm

Commit message: primarily keyboard decoder finish ; preliminary layout
Parts:
- added Ck1: 0.1u, Capacitor_SMD:C_0402_1005Metric, F.Cu at (102.2, 21.1)
- added Ck2: 0.1u, Capacitor_SMD:C_0402_1005Metric, F.Cu at (104.1, 21.1)
- added Ckd1: 0.1u, Capacitor_SMD:C_0402_1005Metric, F.Cu at (100.5, 24.9)
- added Ckd2: 0.1u, Capacitor_SMD:C_0402_1005Metric, F.Cu at (102.5, 24.9)
- added Ckd3: 0.1u, Capacitor_SMD:C_0402_1005Metric, F.Cu at (104.5, 24.9)
- added Ckd4: 0.1u, Capacitor_SMD:C_0402_1005Metric, F.Cu at (106.4, 24.9)
- added Ckd5: 0.1u, Capacitor_SMD:C_0402_1005Metric, F.Cu at (108.4, 24.9)
- added Ckd6: 0.1u, Capacitor_SMD:C_0402_1005Metric, F.Cu at (110.4, 24.9)
- added Ckd7: 0.1u, Capacitor_SMD:C_0402_1005Metric, F.Cu at (112.3, 24.9)
- added Ckd8: 0.1u, Capacitor_SMD:C_0402_1005Metric, F.Cu at (114.3, 24.9)
- added Cki1: 0.1u, Capacitor_SMD:C_0402_1005Metric, F.Cu at (155.6, 26.0)
- added Cki10: 0.1u, Capacitor_SMD:C_0402_1005Metric, F.Cu at (158.4, 31.9)
- added Cki11: 0.1u, Capacitor_SMD:C_0402_1005Metric, F.Cu at (158.4, 33.9)
- added Cki12: 0.1u, Capacitor_SMD:C_0402_1005Metric, F.Cu at (158.4, 35.8)
- added Cki13: 0.1u, Capacitor_SMD:C_0402_1005Metric, F.Cu at (161.3, 26.0)
- added Cki14: 0.1u, Capacitor_SMD:C_0402_1005Metric, F.Cu at (161.3, 27.9)
- added Cki15: 0.1u, Capacitor_SMD:C_0402_1005Metric, F.Cu at (161.3, 29.9)
- added Cki2: 0.1u, Capacitor_SMD:C_0402_1005Metric, F.Cu at (155.6, 27.9)
- added Cki3: 0.1u, Capacitor_SMD:C_0402_1005Metric, F.Cu at (155.6, 29.9)
- added Cki4: 0.1u, Capacitor_SMD:C_0402_1005Metric, F.Cu at (155.6, 31.9)
- added Cki5: 0.1u, Capacitor_SMD:C_0402_1005Metric, F.Cu at (155.6, 33.9)
- added Cki6: 0.1u, Capacitor_SMD:C_0402_1005Metric, F.Cu at (155.6, 35.8)
- added Cki7: 0.1u, Capacitor_SMD:C_0402_1005Metric, F.Cu at (158.4, 26.0)
- added Cki8: 0.1u, Capacitor_SMD:C_0402_1005Metric, F.Cu at (158.4, 27.9)
- added Cki9: 0.1u, Capacitor_SMD:C_0402_1005Metric, F.Cu at (158.4, 29.9)
- added Dio1: green, Diode_SMD:D_0603_1608Metric, F.Cu at (22.9, 88.4)
- added Dio2: green, Diode_SMD:D_0603_1608Metric, F.Cu at (55.9, 21.6)
- added H1: MountingHole_Pad, MountingHole:MountingHole_2.2mm_M2_DIN965_Pad, F.Cu at (19.1, 19.1)
- added H2: MountingHole_Pad, MountingHole:MountingHole_2.2mm_M2_DIN965_Pad, F.Cu at (19.1, 113.0)
- added H3: MountingHole_Pad, MountingHole:MountingHole_2.2mm_M2_DIN965_Pad, F.Cu at (162.6, 113.0)
- added H4: MountingHole_Pad, MountingHole:MountingHole_2.2mm_M2_DIN965_Pad, F.Cu at (162.6, 20.3)
- added J4: Conn_01x04, Connector_PinHeader_2.54mm:PinHeader_1x04_P2.54mm_Vertical, F.Cu at (27.9, 104.1)
- added Rio1: 10k, Resistor_SMD:R_0402_1005Metric, F.Cu at (20.3, 88.4)
- added Rio2: 680, Resistor_SMD:R_0402_1005Metric, F.Cu at (22.9, 91.4)
- added Rio3: 680, Resistor_SMD:R_0402_1005Metric, F.Cu at (55.9, 25.4)
- added Ro1: 10k, Resistor_SMD:R_0402_1005Metric, F.Cu at (72.4, 76.7)
- added Ro2: 10k, Resistor_SMD:R_0402_1005Metric, F.Cu at (74.4, 76.7)
- added Ro3: 10k, Resistor_SMD:R_0402_1005Metric, F.Cu at (76.4, 76.7)
- added Ro4: 10k, Resistor_SMD:R_0402_1005Metric, F.Cu at (78.4, 76.7)
- added Ro5: 10k, Resistor_SMD:R_0402_1005Metric, F.Cu at (80.4, 76.7)
- added Ro6: 10k, Resistor_SMD:R_0402_1005Metric, F.Cu at (82.4, 76.7)
- added Ro7: 10k, Resistor_SMD:R_0402_1005Metric, F.Cu at (84.4, 76.7)
- added Ro8: 10k, Resistor_SMD:R_0402_1005Metric, F.Cu at (86.4, 76.7)
- added SW1: SW_DIP_x04, Button_Switch_THT:SW_DIP_SPSTx04_Slide_6.7x11.72mm_W7.62mm_P2.54mm_LowProfile, F.Cu at (30.5, 77.5)
- added Uk1: 74LS377, Package_SO:SSOP-20_5.3x7.2mm_P0.65mm, F.Cu at (159.7, 41.6)
- added Uk2: 74LS02, Package_SO:SOIC-14_3.9x8.7mm_P1.27mm, F.Cu at (158.7, 52.1)
- added Ukd1: 74LS08, Package_SO:SOIC-14_3.9x8.7mm_P1.27mm, F.Cu at (118.0, 85.1)
- added Ukd2: 74LS08, Package_SO:SOIC-14_3.9x8.7mm_P1.27mm, F.Cu at (118.0, 95.2)
- added Ukd3: 74LS08, Package_SO:SOIC-14_3.9x8.7mm_P1.27mm, F.Cu at (130.9, 85.1)
- added Ukd4: 74LS02, Package_SO:SOIC-14_3.9x8.7mm_P1.27mm, F.Cu at (130.9, 95.2)
- added Ukd5: 74LS02, Package_SO:SOIC-14_3.9x8.7mm_P1.27mm, F.Cu at (143.4, 85.1)
- added Ukd6: 74LS377, Package_SO:SSOP-20_5.3x7.2mm_P0.65mm, F.Cu at (154.9, 83.8)
- added Ukd7: AT28C256-15PU, Package_DIP:DIP-28_W15.24mm_Socket, F.Cu at (157.5, 61.0)
- added Ukd8: 74LS377, Package_SO:SSOP-20_5.3x7.2mm_P0.65mm, F.Cu at (143.5, 95.2)
- added Uki14: 74LS377, Package_SO:SSOP-20_5.3x7.2mm_P0.65mm, F.Cu at (93.7, 94.4)
- added Uki15: 74LS377, Package_SO:SSOP-20_5.3x7.2mm_P0.65mm, F.Cu at (103.8, 94.4)
- Uki10, Uki11: value 74LS377 -> 74LS195; footprint Package_SO:SSOP-20_5.3x7.2mm_P0.65mm -> Package_SO:SOIC-16_3.9x9.9mm_P1.27mm
- Uki5: value 74LS195 -> 74LS08; footprint Package_SO:SOIC-16_3.9x9.9mm_P1.27mm -> Package_SO:SOIC-14_3.9x8.7mm_P1.27mm
- moved Uki6 96.7 mm to (37.5, 104.1), turned to 90 degrees
- moved Rt3 79.8 mm to (124.1, 48.1)
- moved Dt1 79.8 mm to (127.6, 48.1)
- moved Ct1 79.8 mm to (141.6, 47.1)
- moved Ct2 79.8 mm to (146.5, 38.1)
- moved Ct3 79.8 mm to (134.6, 41.1)
- moved Rt1 79.8 mm to (142.6, 43.1)
- moved Rt2 79.8 mm to (140.6, 43.1)
- moved Ut1 79.8 mm to (141.5, 38.1)
- moved Ut2 79.8 mm to (127.6, 38.1)
- moved Uki1 77.3 mm to (39.4, 85.7)
- moved Uki2 74.4 mm to (50.7, 85.7)
- moved Uki3 73.9 mm to (59.8, 85.7)
- moved Uki7 67.6 mm to (48.9, 104.1), turned to 90 degrees
- moved Uki8 64.6 mm to (60.3, 104.1), turned to 90 degrees
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Connections:
- net /keyboard/keyboard_input/lowerout0 renamed /keyboard/keyboard_decoder/upper0
- net /keyboard/keyboard_input/lowerout1 renamed /keyboard/keyboard_decoder/upper1
- net /keyboard/keyboard_input/lowerout2 renamed /keyboard/keyboard_decoder/upper2
- net /keyboard/keyboard_input/lowerout3 renamed /keyboard/keyboard_decoder/upper3
- Ud3 pad 1: (no net) -> /~{out_key}
- Ud3 pad 10: /~{out_key} -> unconnected-(Ud3-Pad10)
- Ud3 pad 11: /decoder/~{keyboardclk_en} -> VCC
- Ud3 pad 12: /decoder/~{keyboardclk_en} -> VCC
- Ud3 pad 13: /decoder/key_read -> unconnected-(Ud3-Pad13)
- Ud3 pad 2: (no net) -> /key_read
- Ud3 pad 3: (no net) -> /key_read
- Ud3 pad 4: /decoder/~{keyboardclk_en} -> unconnected-(Ud3-Pad4)
- Ud3 pad 5: Net-(Ud3-Pad5) -> VCC
- Ud3 pad 6: Net-(Ud3-Pad6) -> VCC
- Ud3 pad 8: Net-(Ud3-Pad5) -> VCC
- Ud3 pad 9: Net-(Ud3-Pad5) -> VCC
- Ud6 pad 11: Net-(Ud3-Pad6) -> /key_read
- Ud6 pad 12: Net-(U3-Pad1) -> /decoder/iskeyboard
- Ud6 pad 13: GND -> Net-(Ud6-Pad13)
- Ud7 pad 1: /decoder/iskeyboard -> /keyboard_int
- Ud7 pad 3: Net-(Ud3-Pad5) -> Net-(Ud6-Pad13)
- Uki1 pad 1: /keyboard/keyboard_input/~{rst} -> VCC
- Uki1 pad 10: /keyboard/ps2clk -> /clk
- Uki1 pad 12: Net-(Uki1-Q3) -> /keyboard/keyboard_decoder/rdy
- Uki1 pad 13: unconnected-(Uki1-Q2-Pad13) -> Net-(Uki1-P3)
- Uki1 pad 14: unconnected-(Uki1-Q1-Pad14) -> /keyboard/keyboard_input/~{rst_buf}
- Uki1 pad 15: unconnected-(Uki1-Q0-Pad15) -> Net-(Uki1-P1)
- Uki1 pad 2: GND -> VCC
- Uki1 pad 3: GND -> VCC
- Uki1 pad 4: GND -> /keyboard_enable
- Uki1 pad 5: VCC -> Net-(Uki1-P1)
- Uki1 pad 6: GND -> /keyboard/keyboard_input/rdy
- Uki1 pad 7: GND -> Net-(Uki1-P3)
- Uki1 pad 9: /keyboard/keyboard_input/~{rdy} -> GND
- Uki10 pad 1: /keyboard/keyboard_input/~{rdy} -> /keyboard_enable
- Uki10 pad 10: GND -> /ps2clk
- Uki10 pad 11: /keyboard/clk -> unconnected-(Uki10-~{Q3}-Pad11)
- Uki10 pad 12: Net-(Uki10-Q4) -> /keyboard/keyboard_input/upper2
- Uki10 pad 13: /keyboard/keyboard_input/upper4 -> /keyboard/keyboard_input/upper3
- Uki10 pad 14: /keyboard/keyboard_input/upper5 -> /keyboard/keyboard_input/upper4
- Uki10 pad 15: Net-(Uki10-Q5) -> /keyboard/keyboard_input/upper5
- Uki10 pad 16: Net-(Uki10-Q6) -> VCC
- Uki10 pad 2: Net-(Uki10-Q0) -> /keyboard/keyboard_input/upper6
- Uki10 pad 3: /keyboard/keyboard_input/upper0 -> /keyboard/keyboard_input/upper6
- Uki10 pad 4: /keyboard/keyboard_input/upper1 -> VCC
- Uki10 pad 5: Net-(Uki10-Q1) -> VCC
- Uki10 pad 6: Net-(Uki10-Q2) -> VCC
- Uki10 pad 7: /keyboard/keyboard_input/upper2 -> VCC
- Uki10 pad 8: /keyboard/keyboard_input/upper3 -> GND
- Uki10 pad 9: Net-(Uki10-Q3) -> VCC
- Uki11 pad 1: GND -> /keyboard_enable
- Uki11 pad 10: GND -> /ps2clk
- Uki11 pad 11: /keyboard/clk -> unconnected-(Uki11-~{Q3}-Pad11)
- Uki11 pad 12: /keyboard/keyboard_input/upperout4 -> unconnected-(Uki11-Q3-Pad12)
- Uki11 pad 13: Net-(Uki10-Q4) -> unconnected-(Uki11-Q2-Pad13)
- Uki11 pad 14: Net-(Uki10-Q5) -> /keyboard/keyboard_input/upper0
- Uki11 pad 15: /keyboard/keyboard_input/upperout5 -> /keyboard/keyboard_input/upper1
- Uki11 pad 16: /keyboard/keyboard_input/upperout6 -> VCC
- Uki11 pad 2: /keyboard/keyboard_input/upperout0 -> /keyboard/keyboard_input/upper2
- Uki11 pad 3: Net-(Uki10-Q0) -> /keyboard/keyboard_input/upper2
- Uki11 pad 4: Net-(Uki10-Q1) -> VCC
- Uki11 pad 5: /keyboard/keyboard_input/upperout1 -> VCC
- Uki11 pad 6: /keyboard/keyboard_input/upperout2 -> VCC
- Uki11 pad 7: Net-(Uki10-Q2) -> VCC
- Uki11 pad 8: Net-(Uki10-Q3) -> GND
- Uki11 pad 9: /keyboard/keyboard_input/upperout3 -> VCC
- Uki12 pad 11: /keyboard/clk -> /clk
- Uki12 pad 13: /keyboard/keyboard_input/lower4 -> /keyboard/keyboard_input/upper4
- Uki12 pad 14: /keyboard/keyboard_input/lower5 -> /keyboard/keyboard_input/upper5
- Uki12 pad 17: /keyboard/keyboard_input/lower6 -> /keyboard/keyboard_input/upper6
- Uki12 pad 18: /keyboard/keyboard_input/lower7 -> /keyboard/keyboard_input/upper7
- Uki12 pad 3: /keyboard/keyboard_input/lower0 -> /keyboard/keyboard_input/upper0
- Uki12 pad 4: /keyboard/keyboard_input/lower1 -> /keyboard/keyboard_input/upper1
- Uki12 pad 7: /keyboard/keyboard_input/lower2 -> /keyboard/keyboard_input/upper2
- Uki12 pad 8: /keyboard/keyboard_input/lower3 -> /keyboard/keyboard_input/upper3
- Uki13 pad 11: /keyboard/clk -> /clk
- Uki13 pad 12: /keyboard/keyboard_input/lowerout4 -> /keyboard/keyboard_decoder/upper4
- Uki13 pad 15: /keyboard/keyboard_input/lowerout5 -> /keyboard/keyboard_decoder/upper5
- Uki13 pad 16: /keyboard/keyboard_input/lowerout6 -> /keyboard/keyboard_decoder/upper6
- Uki13 pad 19: /keyboard/keyboard_input/lowerout7 -> /keyboard/keyboard_decoder/upper7
- Uki2 pad 1: /keyboard/keyboard_input/~{rst} -> VCC
- Uki2 pad 10: /keyboard/ps2clk -> /keyboard/keyboard_input/rdyclk
- Uki2 pad 2: Net-(Uki1-Q3) -> /keyboard/keyboard_input/prerdy
- Uki2 pad 3: Net-(Uki1-Q3) -> /keyboard/keyboard_input/prerdy
- Uki2 pad 4: GND -> VCC
- Uki2 pad 9: VCC -> /keyboard/keyboard_input/~{rst_buf}
- Uki3 pad 1: /keyboard/keyboard_input/~{rst} -> VCC
- Uki3 pad 10: /keyboard/ps2clk -> /keyboard/keyboard_input/rdyclk
- Uki3 pad 11: /keyboard/keyboard_input/~{rdy} -> unconnected-(Uki3-~{Q3}-Pad11)
- Uki3 pad 12: /keyboard/keyboard_input/rdy -> Net-(Uki3-Q3)
- Uki3 pad 9: VCC -> /keyboard/keyboard_input/~{rst_buf}
- Uki4 pad 1: /keyboard/keyboard_input/~{rst} -> VCC
- Uki4 pad 10: /keyboard/ps2clk -> /keyboard/keyboard_input/rdyclk
- Uki4 pad 11: unconnected-(Uki4-~{Q3}-Pad11) -> /keyboard/keyboard_input/~{rdy}
- Uki4 pad 12: /keyboard/keyboard_input/lower6 -> /keyboard/keyboard_input/rdy
- Uki4 pad 13: /keyboard/keyboard_input/lower7 -> /keyboard/keyboard_input/prerdy
- Uki4 pad 2: /keyboard/ps2data -> Net-(Uki3-Q3)
- Uki4 pad 3: /keyboard/ps2data -> Net-(Uki3-Q3)
- Uki4 pad 4: VCC -> GND
- Uki4 pad 5: VCC -> GND
- Uki4 pad 6: VCC -> GND
- Uki4 pad 7: VCC -> GND
- Uki4 pad 9: VCC -> /keyboard/keyboard_input/~{rst_buf}
- Uki5 pad 1: /keyboard/keyboard_input/~{rst} -> /ps2clk
- Uki5 pad 10: /keyboard/ps2clk -> Net-(Ukd3-Pad11)
- Uki5 pad 11: unconnected-(Uki5-~{Q3}-Pad11) -> /keyboard_int
- Uki5 pad 12: /keyboard/keyboard_input/lower2 -> /keyboard_enable
- Uki5 pad 13: /keyboard/keyboard_input/lower3 -> Net-(Uki5-Pad13)
- Uki5 pad 14: /keyboard/keyboard_input/lower4 -> VCC
- Uki5 pad 2: /keyboard/keyboard_input/lower6 -> /keyboard_enable
- Uki5 pad 3: /keyboard/keyboard_input/lower6 -> /keyboard/keyboard_input/rdyclk
- Uki5 pad 4: VCC -> Net-(Uk2-Pad1)
- Uki5 pad 5: VCC -> Net-(Uk2-Pad4)
- Uki5 pad 6: VCC -> Net-(Uki5-Pad13)
- Uki5 pad 7: VCC -> GND
- Uki5 pad 8: GND -> /keyboard/keyboard_decoder/shift
- Uki5 pad 9: VCC -> /keyboard_enable
- Uki6 pad 1: /keyboard/keyboard_input/~{rst} -> /keyboard_enable
- Uki6 pad 10: /keyboard/ps2clk -> /ps2clk
- Uki6 pad 12: unconnected-(Uki6-Q3-Pad12) -> /keyboard/keyboard_input/lower6
- Uki6 pad 13: Net-(Uki6-Q2) -> /keyboard/keyboard_input/lower7
- Uki6 pad 14: /keyboard/keyboard_input/lower0 -> unconnected-(Uki6-Q1-Pad14)
- Uki6 pad 15: /keyboard/keyboard_input/lower1 -> unconnected-(Uki6-Q0-Pad15)
- Uki6 pad 2: /keyboard/keyboard_input/lower2 -> /ps2data
- Uki6 pad 3: /keyboard/keyboard_input/lower2 -> /ps2data
- Uki7 pad 1: /keyboard/keyboard_input/~{rst} -> /keyboard_enable
- Uki7 pad 10: /keyboard/ps2clk -> /ps2clk
- Uki7 pad 12: /keyboard/keyboard_input/upper6 -> /keyboard/keyboard_input/lower2
- Uki7 pad 13: /keyboard/keyboard_input/upper7 -> /keyboard/keyboard_input/lower3
- Uki7 pad 14: unconnected-(Uki7-Q1-Pad14) -> /keyboard/keyboard_input/lower4
- Uki7 pad 15: unconnected-(Uki7-Q0-Pad15) -> /keyboard/keyboard_input/lower5
- Uki7 pad 2: Net-(Uki6-Q2) -> /keyboard/keyboard_input/lower6
- Uki7 pad 3: Net-(Uki6-Q2) -> /keyboard/keyboard_input/lower6
- Uki8 pad 1: /keyboard/keyboard_input/~{rst} -> /keyboard_enable
- Uki8 pad 10: /keyboard/ps2clk -> /ps2clk
- Uki8 pad 12: /keyboard/keyboard_input/upper2 -> unconnected-(Uki8-Q3-Pad12)
- Uki8 pad 13: /keyboard/keyboard_input/upper3 -> Net-(Uki8-Q2)
- Uki8 pad 14: /keyboard/keyboard_input/upper4 -> /keyboard/keyboard_input/lower0
- Uki8 pad 15: /keyboard/keyboard_input/upper5 -> /keyboard/keyboard_input/lower1
- Uki8 pad 2: /keyboard/keyboard_input/upper6 -> /keyboard/keyboard_input/lower2
- Uki8 pad 3: /keyboard/keyboard_input/upper6 -> /keyboard/keyboard_input/lower2
- Uki9 pad 1: /keyboard/keyboard_input/~{rst} -> /keyboard_enable
- Uki9 pad 10: /keyboard/ps2clk -> /ps2clk
- Uki9 pad 12: unconnected-(Uki9-Q3-Pad12) -> /keyboard/keyboard_input/upper6
- Uki9 pad 13: unconnected-(Uki9-Q2-Pad13) -> /keyboard/keyboard_input/upper7
- Uki9 pad 14: /keyboard/keyboard_input/upper0 -> unconnected-(Uki9-Q1-Pad14)
- Uki9 pad 15: /keyboard/keyboard_input/upper1 -> unconnected-(Uki9-Q0-Pad15)
- Uki9 pad 2: /keyboard/keyboard_input/upper2 -> Net-(Uki8-Q2)
- Uki9 pad 3: /keyboard/keyboard_input/upper2 -> Net-(Uki8-Q2)
- Uo1 pad 2: /gpuout7 -> GND
- Uo1 pad 3: /gpuout6 -> GND
- Uo1 pad 4: /gpuout5 -> GND
- Uo1 pad 5: /gpuout4 -> GND
- Uo1 pad 6: /gpuout3 -> GND
- Uo1 pad 7: /gpuout2 -> GND
- Uo1 pad 8: /gpuout1 -> GND
- Uo1 pad 9: /gpuout0 -> VCC
- Ut1 pad 4: VCC -> /timer_enable
Other:
- board size 136.5 x 100 mm -> 149.2 x 100 mm
- board text added: "PWR"

Commit message: io controller update
Parts:
- added J3: Mini-DIN-6, mALUch_lib:MiniDin6_PS2, F.Cu at (148.8, 104.0)
- added Rio4: 10k, Resistor_SMD:R_0402_1005Metric, F.Cu at (109.0, 69.5)
- added Rt2: 10k, Resistor_SMD:R_0402_1005Metric, F.Cu at (71.8, 59.6)
- added Rt4: 10k, Resistor_SMD:R_0402_1005Metric, F.Cu at (71.8, 61.6)
- C1, Cd1, Cd2, Cd3, Cd4, Cd5, Cd6, Cd7, Ck1, Ck2, Ckd1, Ckd2, Ckd3, Ckd4, Ckd5, Ckd6, Ckd7, Ckd8, Cki1, Cki10, Cki11, Cki12, Cki13, Cki14, Cki15, Cki2, Cki3, Cki4, Cki5, Cki6, Cki7, Cki8, Cki9, Co1, Co2: value 0.1u -> 100nF
- Ct1: value 33n -> 33u; footprint Capacitor_SMD:C_Elec_3x5.4 -> Capacitor_SMD:C_1206_3216Metric
- Ct2, Ct3: value 0.1u -> 100nF; footprint Capacitor_SMD:C_0603_1608Metric -> Capacitor_SMD:C_0402_1005Metric
- Dio1: value green -> yellow
- Dl1, Dl2, Dl3, Dl4, Dl5, Dl6, Dl7, Dl8: value red -> blue
- J1, J2: footprint Connector_IDC:IDC-Header_2x10_P2.54mm_Horizontal -> mALUch_lib:PinHeader_2x10_P2.54mm_Horizontal
- Rd1, Rd2, Rd3, Rd4, Rd5, Rd6: value 470 -> 680
- Rt1: value 4.7k -> 10k
- Rt3: renamed from Rt2; value 22k -> 10k
- Ud1, Ud2, Ud3, Uk2, Ukd4, Ukd5: value 74LS02 -> 7402
- Ud4, Ud5, Ud6, Ud7, Ukd1, Ukd2, Ukd3, Uki5: value 74LS08 -> 7408; footprint Package_SO:SOIC-14_3.9x8.7mm_P1.27mm -> Package_SO:SO-14_3.9x8.65mm_P1.27mm
- Uk1, Ukd6, Ukd8, Uki12, Uki13, Uki14, Uki15: value 74LS377 -> 74377
- Uki1, Uki10, Uki11, Uki2, Uki3, Uki4, Uki6, Uki7, Uki8, Uki9, Ut2: value 74LS195 -> 74195
- Ul1: value 74LS377 -> 74377; footprint Package_SO:SOIC-20W_7.5x12.8mm_P1.27mm -> Package_SO:SSOP-20_5.3x7.2mm_P0.65mm
- Uo1, Uo2: value 74LS245 -> 74245; footprint Package_SO:SOIC-20W_7.5x12.8mm_P1.27mm -> Package_SO:TSSOP-20_4.4x6.5mm_P0.65mm
- moved J4 119.7 mm to (147.5, 98.0), turned to 90 degrees
- moved Cki1 78.3 mm to (77.4, 31.1)
- moved Cki2 78.3 mm to (77.4, 33.1)
- moved Cki3 78.3 mm to (77.4, 35.0)
- moved Cki4 78.3 mm to (77.4, 37.0)
- moved Cki5 78.3 mm to (77.4, 39.0)
- moved Cki6 78.3 mm to (77.4, 40.9)
- moved Uk1 78.3 mm to (81.5, 46.7)
- moved Cki13 78.3 mm to (83.1, 31.1)
- moved Cki14 78.3 mm to (83.1, 33.1)
- moved Cki15 78.3 mm to (83.1, 35.0)
- moved Uk2 78.3 mm to (80.5, 57.2)
- moved Cki10 78.3 mm to (80.3, 37.0)
- moved Cki11 78.3 mm to (80.3, 39.0)
- moved Cki12 78.3 mm to (80.3, 40.9)
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- renumbered Rt3 to Rt5
Connections:
- net /key_read renamed /decoder/key_read
- net /timer_clk_en renamed /decoder/timerclk_en
- net /~{led_clk_en} renamed /LEDs/~{clk_en}
- net /~{out_gpu} renamed /decoder/~{gpu_out}
- net /~{out_key} renamed /decoder/~{key_out}
- net /~{timer_read} renamed /decoder/~{timer_read}
- Rt3 pad 1: Net-(Ut1-THR) -> Net-(Rt3-Pad1)
- SW1 pad 2: Net-(SW1-Pad2) -> GND
- SW1 pad 3: Net-(SW1-Pad2) -> GND
Routing:
- net /iobus7: track 28.6 -> 0.00 mm
- net /iobus6: track 28.6 -> 0.00 mm
- net /iobus5: track 28.6 -> 0.00 mm
- net /iobus4: track 28.6 -> 0.00 mm
- net /iobus3: track 28.6 -> 0.00 mm
- net /iobus2: track 28.6 -> 0.00 mm
- net /iobus1: track 28.6 -> 0.00 mm
- net /iobus0: track 28.6 -> 0.00 mm
- net Net-(Ud2-Pad11): track 0.00 -> 1.27 mm
Other:
- board size 149.2 x 100 mm -> 150 x 100 mm
