File: PCB/Kicad/io_controller/keyboard_input.kicad_sch (KiCad schematic)
At the start: 13 parts, among them U12 74LS195, U13 74LS195, U14 74LS195, U15 74LS195, U16 74LS195, U17 74LS195, U18 74LS377, U19 74LS377, U20 74LS377, U21 74LS377, U22 74LS195, U23 74LS195, U24 74LS195

Commit message: more spice models and bugfixes ; more tests of io_controller - mostly keyboard
Parts:
- removed U12, U13, U14, U15, U16, U17, U23, U24: 74LS195, symbol 74xx:74LS195
- removed U19, U20, U21: 74LS377, symbol 74xx:74LS377
- added Uki1, Uki10, Uki11, Uki3, Uki4, Uki6, Uki7, Uki8, Uki9: 74LS195, Package_SO:SOIC-16_3.9x9.9mm_P1.27mm, symbol 74xx:74LS195
- added Uki13, Uki14, Uki15: 74LS377, Package_SO:SSOP-20_5.3x7.2mm_P0.65mm, symbol 74xx:74LS377
- added Uki5: 74LS08, symbol 74xx:74LS08
- Uki12: renamed from U18; footprint (none) -> Package_SO:SSOP-20_5.3x7.2mm_P0.65mm
- Uki2: renamed from U22; footprint (none) -> Package_SO:SOIC-16_3.9x9.9mm_P1.27mm
Connections:
- net GND: now also Uki2.6 (P2), Uki2.7 (P3), Uki1.8 (GND), Uki1.9 (~{PE}), Uki10.8 (GND), Uki11.8 (GND), Uki13.1 (~{E}), Uki13.10 (GND), Uki14.10 (GND), Uki15.1 (~{E}), Uki15.10 (GND), Uki3.4 (P0), Uki3.5 (P1), Uki3.6 (P2), Uki3.7 (P3), Uki4.4 (P0), Uki4.5 (P1), Uki4.6 (P2), Uki4.7 (P3), Uki4.8 (GND), Uki5.7 (GND), Uki6.8 (GND), Uki7.8 (GND), Uki8.8 (GND), Uki9.8 (GND); no longer Uki2.2 (J), Uki2.3 (~{K})
- net VCC: now also Uki1.1 (~{MR}), Uki1.16 (VCC), Uki1.2 (J), Uki1.3 (~{K}), Uki10.16 (VCC), Uki10.4 (P0), Uki10.5 (P1), Uki10.6 (P2), Uki10.7 (P3), Uki10.9 (~{PE}), Uki11.16 (VCC), Uki11.4 (P0), Uki11.5 (P1), Uki11.6 (P2), Uki11.7 (P3), Uki11.9 (~{PE}), Uki13.20 (VCC), Uki14.20 (VCC), Uki15.20 (VCC), Uki3.1 (~{MR}), Uki3.16 (VCC), Uki4.1 (~{MR}), Uki4.16 (VCC), Uki5.12, Uki5.13, Uki5.14 (VCC), Uki5.4, Uki5.5, Uki6.16 (VCC), Uki6.4 (P0), Uki6.5 (P1), Uki6.6 (P2), Uki6.7 (P3), Uki6.9 (~{PE}), Uki7.16 (VCC), Uki7.4 (P0), Uki7.5 (P1), Uki7.6 (P2), Uki7.7 (P3), Uki7.9 (~{PE}), Uki8.16 (VCC), Uki8.4 (P0), Uki8.5 (P1), Uki8.6 (P2), Uki8.7 (P3), Uki8.9 (~{PE}), Uki9.16 (VCC), Uki9.4 (P0), Uki9.5 (P1), Uki9.6 (P2), Uki9.7 (P3), Uki9.9 (~{PE}); no longer Uki2.6 (P2), Uki2.7 (P3)
- net clk: now also Uki1.10 (CP), Uki13.11 (CP), Uki14.11 (CP), Uki15.11 (CP)
- net lower0: now also Uki14.3 (D0), Uki8.14 (Q1)
- net lower1: now also Uki14.4 (D1), Uki8.15 (Q0)
- net lower2: now also Uki14.7 (D2), Uki7.12 (Q3), Uki8.2 (J), Uki8.3 (~{K})
- net lower3: now also Uki14.8 (D3), Uki7.13 (Q2)
- net lower4: now also Uki14.13 (D4), Uki7.14 (Q1)
- net lower5: now also Uki14.14 (D5), Uki7.15 (Q0)
- net lower6: now also Uki14.17 (D6), Uki6.12 (Q3), Uki7.2 (J), Uki7.3 (~{K})
- net lower7: now also Uki14.18 (D7), Uki6.13 (Q2)
- net lowerout0: now also Uki15.2 (Q0)
- net lowerout1: now also Uki15.5 (Q1)
- net lowerout2: now also Uki15.6 (Q2)
- net lowerout3: now also Uki15.9 (Q3)
- net lowerout4: now also Uki15.12 (Q4)
- net lowerout5: now also Uki15.15 (Q5)
- net lowerout6: now also Uki15.16 (Q6)
- net lowerout7: now also Uki15.19 (Q7)
- net ps2clk: now also Uki10.10 (CP), Uki11.10 (CP), Uki5.1, Uki6.10 (CP), Uki7.10 (CP), Uki8.10 (CP), Uki9.10 (CP); no longer Uki2.10 (CP)
- net ps2data: now also Uki6.2 (J), Uki6.3 (~{K})
- net rdy: now also Uki1.6 (P2), Uki4.12 (Q3)
- net upper0: now also Uki11.14 (Q1)
- net upper1: now also Uki11.15 (Q0)
- net upper2: now also Uki10.12 (Q3), Uki11.2 (J), Uki11.3 (~{K})
- net upper3: now also Uki10.13 (Q2)
- net upper4: now also Uki10.14 (Q1)
- net upper5: now also Uki10.15 (Q0)
- net upper6: now also Uki10.2 (J), Uki10.3 (~{K}), Uki9.12 (Q3)
- net upper7: now also Uki9.13 (Q2)
- net upperout0: now also Uki13.2 (Q0)
- net upperout1: now also Uki13.5 (Q1)
- net upperout2: now also Uki13.6 (Q2)
- net upperout3: now also Uki13.9 (Q3)
- net upperout4: now also Uki13.12 (Q4)
- net upperout5: now also Uki13.15 (Q5)
- net upperout6: now also Uki13.16 (Q6)
- net upperout7: now also Uki13.19 (Q7)
- net ~{rdy}: now also Uki14.1 (~{E}), Uki4.11 (~{Q3}); no longer Uki2.9 (~{PE})
- net at Uki2.12 (Q3): now also Uki3.2 (J), Uki3.3 (~{K})
- net at Uki12.12 (Q4): now also Uki13.13 (D4)
- net at Uki12.15 (Q5): now also Uki13.14 (D5)
- net at Uki12.16 (Q6): now also Uki13.17 (D6)
- net at Uki12.19 (Q7): now also Uki13.18 (D7)
- net at Uki12.2 (Q0): now also Uki13.3 (D0)
- net at Uki12.5 (Q1): now also Uki13.4 (D1)
- net at Uki12.6 (Q2): now also Uki13.7 (D2)
- net at Uki12.9 (Q3): now also Uki13.8 (D3)
- new net: Uki14.12 (Q4), Uki15.13 (D4)
- new net: Uki14.15 (Q5), Uki15.14 (D5)
- new net: Uki14.16 (Q6), Uki15.17 (D6)
- new net: Uki14.19 (Q7), Uki15.18 (D7)
- new net: Uki14.2 (Q0), Uki15.3 (D0)
- new net: Uki14.5 (Q1), Uki15.4 (D1)
- new net: Uki14.6 (Q2), Uki15.7 (D2)
- new net: Uki14.9 (Q3), Uki15.8 (D3)
- new net: Uki8.13 (Q2), Uki9.2 (J), Uki9.3 (~{K})
- new net: Uki3.12 (Q3), Uki4.2 (J), Uki4.3 (~{K})
- new net: Uki1.13 (Q2), Uki1.7 (P3)
- new net: Uki1.15 (Q0), Uki1.5 (P1)
- new net prerdy: Uki2.2 (J), Uki2.3 (~{K}), Uki4.13 (Q2)
- new net rdyclk: Uki2.10 (CP), Uki3.10 (CP), Uki4.10 (CP), Uki5.3
- new net rdyout: Uki1.12 (Q3)
- new net ~{rst_buf}: Uki1.14 (Q1), Uki2.9 (~{PE}), Uki3.9 (~{PE}), Uki4.9 (~{PE})
- new net ~{rst}: Uki1.4 (P0), Uki10.1 (~{MR}), Uki11.1 (~{MR}), Uki5.2, Uki6.1 (~{MR}), Uki7.1 (~{MR}), Uki8.1 (~{MR}), Uki9.1 (~{MR})
- no-connect marks 23 -> 25
Other:
- note added: "serves as both: 1. delay to rst signal, to properly time ~{PE} signal 2. delay to ouput ready, to sync with metastability fixers"
- note added: "the output is ready once every 11 pulses of PS2 clock once the PS2 cycles 11 times, registers are loaded with current contents simultaneously, the counter is reset and waits again for the input"
- note removed: "the output is ready once every 11 pulses of PS2 clock (verify) once the PS2 cycles 11 times, registers are loaded with current contents simultaneously, the counter is reset and waits again for the input"
- company: (none) -> AGH Logic Unit
- title: (none) -> Keyboard Input
- moved on the sheet: Uki2

Commit message: primarily keyboard decoder finish ; preliminary layout
Parts:
- removed unit 2 of Uki5
- removed unit 4 of Uki5
- added Cki1, Cki10, Cki11, Cki12, Cki13, Cki14, Cki15, Cki2, Cki3, Cki4, Cki5, Cki6, Cki7, Cki8, Cki9: 0.1u, Capacitor_SMD:C_0402_1005Metric, symbol Device:C
- Uki5: footprint (none) -> Package_SO:SOIC-14_3.9x8.7mm_P1.27mm
Connections:
- net GND: now also Uki3.8 (GND), Cki1.2, Cki10.2, Cki11.2, Cki12.2, Cki13.2, Cki14.2, Cki15.2, Cki2.2, Cki3.2, Cki4.2, Cki5.2, Cki6.2, Cki7.2, Cki8.2, Cki9.2
- net VCC: now also Cki1.1, Cki10.1, Cki11.1, Cki12.1, Cki13.1, Cki14.1, Cki15.1, Cki2.1, Cki3.1, Cki4.1, Cki5.1, Cki6.1, Cki7.1, Cki8.1, Cki9.1
- no-connect marks 25 -> 24
Other:
- moved on the sheet: Uki12, Uki13, Uki14, Uki15

Commit message: io controller update
Parts:
- Cki1, Cki10, Cki11, Cki12, Cki13, Cki14, Cki15, Cki2, Cki3, Cki4, Cki5, Cki6, Cki7, Cki8, Cki9: value 0.1u -> 100nF
- Uki1, Uki10, Uki11, Uki2, Uki3, Uki4, Uki6, Uki7, Uki8, Uki9: value 74LS195 -> 74195
- Uki12, Uki13, Uki14, Uki15: value 74LS377 -> 74377
- Uki5: value 74LS08 -> 7408; footprint Package_SO:SOIC-14_3.9x8.7mm_P1.27mm -> Package_SO:SO-14_3.9x8.65mm_P1.27mm
