File: PCB/Kicad/reg/_autosave-reg.kicad_pcb (KiCad board)
At the start: 2 copper layers, 172 parts, among them U1 7404, U10 74HCT574, U11 74HC245, U12 74HC245, U14 CD74HC4067M, U15 74HC245, U16 74HC245, U17 74HC245, U18 74HC245, U19 74HC245, U2 74AHC1G04, U20 74HC245, U21 74HC245, U22 74HC245, U23 74HCT574, U24 74HCT574, U25 74HCT574, U26 74HCT574, U27 74HCT574, U28 74HCT574, U29 74HCT574, U30 74HCT574, U31 74HCT574, U32 74HCT574, U33 74HCT574, U34 74HCT574, U35 74HCT574, U36 74HCT574, U37 74HCT574, U38 74HCT574, U39 74HCT574, U4 74AHC1G04, U40 74HCT574, U41 74HCT574, U42 74HCT574, U43 74HCT574, U44 74HCT574, U45 74HCT574, U46 74HCT574, U47 74HCT574, U48 74HCT574, U49 74HCT574, U5 74AHC1G04, U50 74HCT574, U51 74HCT574, U52 74HCT574, U53 74HC245, U54 74HC245, U55 74HC245, U56 74HC245, U57 74HC245, U58 74HC245, U59 74HC245, U6 74AHC1G04, U60 74HC245, U61 74HC245, U62 74HC245, U63 74HC245, U64 74HC245, U65 74HC245, U66 74HC245, U67 74HC245, U68 74HC245, U69 74HC245, U7 74HC245, U70 74HC245, U71 74HC245, U72 74HC245, U73 74HC245, U74 74HC245, U75 74HC245, U76 74HC245, U77 74HC245, U78 74HC245, U79 74HC245, U8 74HC245, U80 74HC245, U81 74HC245, U82 74HC245, U83 74HCT574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

Commit message: bus
Parts:
- added C83: C_Polarized, Capacitor_SMD:CP_Elec_4x3, F.Cu at (-24.1, 19.1)
- added C84: C_Polarized, Capacitor_SMD:CP_Elec_4x3, F.Cu at (-24.1, 24.9)
- added U1: 74LS10, Package_DIP:DIP-14_W7.62mm_SMDSocket_SmallPads, F.Cu at (-33.8, 25.9)
Connections:
- U10 pad 4: /16 bit register/in_10 -> /OUT10
- U11 pad 11: /16 bit buffor1/out_7 -> /OUT7
- U11 pad 12: /16 bit buffor1/out_6 -> /OUT6
- U11 pad 13: /16 bit buffor1/out_5 -> /OUT5
- U11 pad 14: /16 bit buffor1/out_4 -> /OUT4
- U11 pad 15: /16 bit buffor1/out_3 -> /OUT3
- U11 pad 16: /16 bit buffor1/out_2 -> /OUT2
- U11 pad 17: /16 bit buffor1/out_1 -> r1we
- U11 pad 18: /16 bit buffor1/out_0 -> /OUT0
- U11 pad 2: /16 bit buffor1/in_0 -> /IN0
- U11 pad 3: /16 bit buffor1/in_1 -> /IN1
- U11 pad 4: /16 bit buffor1/in_2 -> /IN2
- U11 pad 5: /16 bit buffor1/in_3 -> /IN3
- U11 pad 6: /16 bit buffor1/in_4 -> /IN4
- U11 pad 7: /16 bit buffor1/in_5 -> /IN5
- U11 pad 8: /16 bit buffor1/in_6 -> /IN6
- U11 pad 9: /16 bit buffor1/in_7 -> /IN7
- U12 pad 11: /16 bit buffor1/out_15 -> /OUT15
- U12 pad 12: /16 bit buffor1/out_14 -> /OUT14
- U12 pad 13: /16 bit buffor1/out_13 -> /OUT13
- U12 pad 14: /16 bit buffor1/out_12 -> /OUT12
- U12 pad 15: /16 bit buffor1/out_11 -> /OUT11
- U12 pad 16: /16 bit buffor1/out_10 -> /OUT10
- U12 pad 17: /16 bit buffor1/out_9 -> /OUT9
- U12 pad 18: /16 bit buffor1/out_8 -> /OUT8
- U12 pad 2: /16 bit buffor1/in_8 -> /IN8
- U12 pad 3: /16 bit buffor1/in_9 -> /IN9
- U12 pad 4: /16 bit buffor1/in_10 -> /IN10
- U12 pad 5: /16 bit buffor1/in_11 -> /IN11
- U12 pad 6: /16 bit buffor1/in_12 -> /IN12
- U12 pad 7: /16 bit buffor1/in_13 -> /IN13
- U12 pad 8: /16 bit buffor1/in_14 -> /IN14
- U12 pad 9: /16 bit buffor1/in_15 -> /IN15
- U15 pad 11: /16 bit buffor2/out_7 -> /OUT7
- U15 pad 12: /16 bit buffor2/out_6 -> /OUT6
- U15 pad 13: /16 bit buffor2/out_5 -> /OUT5
- U15 pad 14: /16 bit buffor2/out_4 -> /OUT4
- U15 pad 15: /16 bit buffor2/out_3 -> /OUT3
- U15 pad 16: /16 bit buffor2/out_2 -> /OUT2
- U15 pad 17: /16 bit buffor2/out_1 -> r1we
- U15 pad 18: /16 bit buffor2/out_0 -> /OUT0
- U15 pad 2: /16 bit buffor2/in_0 -> /IN0
- U15 pad 3: /16 bit buffor2/in_1 -> /IN1
- U15 pad 4: /16 bit buffor2/in_2 -> /IN2
- U15 pad 5: /16 bit buffor2/in_3 -> /IN3
- U15 pad 6: /16 bit buffor2/in_4 -> /IN4
- U15 pad 7: /16 bit buffor2/in_5 -> /IN5
- U15 pad 8: /16 bit buffor2/in_6 -> /IN6
- U15 pad 9: /16 bit buffor2/in_7 -> /IN7
- U16 pad 11: /16 bit buffor2/out_15 -> /OUT15
- U16 pad 12: /16 bit buffor2/out_14 -> /OUT14
- U16 pad 13: /16 bit buffor2/out_13 -> /OUT13
- U16 pad 14: /16 bit buffor2/out_12 -> /OUT12
- U16 pad 15: /16 bit buffor2/out_11 -> /OUT11
- U16 pad 16: /16 bit buffor2/out_10 -> /OUT10
- U16 pad 17: /16 bit buffor2/out_9 -> /OUT9
- U16 pad 18: /16 bit buffor2/out_8 -> /OUT8
- U16 pad 2: /16 bit buffor2/in_8 -> /IN8
- U16 pad 3: /16 bit buffor2/in_9 -> /IN9
- U16 pad 4: /16 bit buffor2/in_10 -> /IN10
- U16 pad 5: /16 bit buffor2/in_11 -> /IN11
- U16 pad 6: /16 bit buffor2/in_12 -> /IN12
- U16 pad 7: /16 bit buffor2/in_13 -> /IN13
- U16 pad 8: /16 bit buffor2/in_14 -> /IN14
- U16 pad 9: /16 bit buffor2/in_15 -> /IN15
- U17 pad 11: /16 bit buffor3/out_7 -> /OUT7
- U17 pad 12: /16 bit buffor3/out_6 -> /OUT6
- U17 pad 13: /16 bit buffor3/out_5 -> /OUT5
- U17 pad 14: /16 bit buffor3/out_4 -> /OUT4
- U17 pad 15: /16 bit buffor3/out_3 -> /OUT3
- U17 pad 16: /16 bit buffor3/out_2 -> /OUT2
- U17 pad 17: /16 bit buffor3/out_1 -> r1we
- U17 pad 18: /16 bit buffor3/out_0 -> /OUT0
- U17 pad 2: /16 bit buffor3/in_0 -> /IN0
- U17 pad 3: /16 bit buffor3/in_1 -> /IN1
- U17 pad 4: /16 bit buffor3/in_2 -> /IN2
- U17 pad 5: /16 bit buffor3/in_3 -> /IN3
- U17 pad 6: /16 bit buffor3/in_4 -> /IN4
- U17 pad 7: /16 bit buffor3/in_5 -> /IN5
- U17 pad 8: /16 bit buffor3/in_6 -> /IN6
- U17 pad 9: /16 bit buffor3/in_7 -> /IN7
- U18 pad 11: /16 bit buffor3/out_15 -> /OUT15
- U18 pad 12: /16 bit buffor3/out_14 -> /OUT14
- U18 pad 13: /16 bit buffor3/out_13 -> /OUT13
- U18 pad 14: /16 bit buffor3/out_12 -> /OUT12
- U18 pad 15: /16 bit buffor3/out_11 -> /OUT11
- U18 pad 16: /16 bit buffor3/out_10 -> /OUT10
- U18 pad 17: /16 bit buffor3/out_9 -> /OUT9
- U18 pad 18: /16 bit buffor3/out_8 -> /OUT8
- U18 pad 2: /16 bit buffor3/in_8 -> /IN8
- U18 pad 3: /16 bit buffor3/in_9 -> /IN9
- U18 pad 4: /16 bit buffor3/in_10 -> /IN10
- U18 pad 5: /16 bit buffor3/in_11 -> /IN11
- U18 pad 6: /16 bit buffor3/in_12 -> /IN12
- U18 pad 7: /16 bit buffor3/in_13 -> /IN13
- U18 pad 8: /16 bit buffor3/in_14 -> /IN14
- U18 pad 9: /16 bit buffor3/in_15 -> /IN15
- U19 pad 11: /16 bit buffor4/out_7 -> /OUT7
- U19 pad 12: /16 bit buffor4/out_6 -> /OUT6
- U19 pad 13: /16 bit buffor4/out_5 -> /OUT5
- U19 pad 14: /16 bit buffor4/out_4 -> /OUT4
- U19 pad 15: /16 bit buffor4/out_3 -> /OUT3
- U19 pad 16: /16 bit buffor4/out_2 -> /OUT2
- U19 pad 17: /16 bit buffor4/out_1 -> r1we
- U19 pad 18: /16 bit buffor4/out_0 -> /OUT0
- U19 pad 2: /16 bit buffor4/in_0 -> /OUT0
- U19 pad 3: /16 bit buffor4/in_1 -> r1we
- U19 pad 4: /16 bit buffor4/in_2 -> /OUT2
- U19 pad 5: /16 bit buffor4/in_3 -> /OUT3
- U19 pad 6: /16 bit buffor4/in_4 -> /OUT4
- U19 pad 7: /16 bit buffor4/in_5 -> /OUT5
- U19 pad 8: /16 bit buffor4/in_6 -> /OUT6
- U19 pad 9: /16 bit buffor4/in_7 -> /OUT7
- U20 pad 11: /16 bit buffor4/out_15 -> /OUT15
- U20 pad 12: /16 bit buffor4/out_14 -> /OUT14
- U20 pad 13: /16 bit buffor4/out_13 -> /OUT13
- U20 pad 14: /16 bit buffor4/out_12 -> /OUT12
- U20 pad 15: /16 bit buffor4/out_11 -> /OUT11
- U20 pad 16: /16 bit buffor4/out_10 -> /OUT10
- U20 pad 17: /16 bit buffor4/out_9 -> /OUT9
- U20 pad 18: /16 bit buffor4/out_8 -> /OUT8
- U20 pad 2: /16 bit buffor4/in_8 -> /OUT8
- U20 pad 3: /16 bit buffor4/in_9 -> /OUT9
- U20 pad 4: /16 bit buffor4/in_10 -> /OUT10
- U20 pad 5: /16 bit buffor4/in_11 -> /OUT11
- U20 pad 6: /16 bit buffor4/in_12 -> /OUT12
- U20 pad 7: /16 bit buffor4/in_13 -> /OUT13
- U20 pad 8: /16 bit buffor4/in_14 -> /OUT14
- U20 pad 9: /16 bit buffor4/in_15 -> /OUT15
- U21 pad 11: /16 bit buffor5/out_7 -> /OUT7
- U21 pad 12: /16 bit buffor5/out_6 -> /OUT6
- U21 pad 13: /16 bit buffor5/out_5 -> /OUT5
- U21 pad 14: /16 bit buffor5/out_4 -> /OUT4
- U21 pad 15: /16 bit buffor5/out_3 -> /OUT3
- U21 pad 16: /16 bit buffor5/out_2 -> /OUT2
- U21 pad 17: /16 bit buffor5/out_1 -> r1we
- U21 pad 18: /16 bit buffor5/out_0 -> /OUT0
- U21 pad 2: /16 bit buffor5/in_0 -> /IN0
- U21 pad 3: /16 bit buffor5/in_1 -> /IN1
- U21 pad 4: /16 bit buffor5/in_2 -> /IN2
- U21 pad 5: /16 bit buffor5/in_3 -> /IN3
- U21 pad 6: /16 bit buffor5/in_4 -> /IN4
- U21 pad 7: /16 bit buffor5/in_5 -> /IN5
- U21 pad 8: /16 bit buffor5/in_6 -> /IN6
- U21 pad 9: /16 bit buffor5/in_7 -> /IN7
- U22 pad 11: /16 bit buffor5/out_15 -> /OUT15
- U22 pad 12: /16 bit buffor5/out_14 -> /OUT14
- U22 pad 13: /16 bit buffor5/out_13 -> /OUT13
- U22 pad 14: /16 bit buffor5/out_12 -> /OUT12
- U22 pad 15: /16 bit buffor5/out_11 -> /OUT11
- U22 pad 16: /16 bit buffor5/out_10 -> /OUT10
- U22 pad 17: /16 bit buffor5/out_9 -> /OUT9
- U22 pad 18: /16 bit buffor5/out_8 -> /OUT8
- U22 pad 2: /16 bit buffor5/in_8 -> /IN8
- U22 pad 3: /16 bit buffor5/in_9 -> /IN9
- U22 pad 4: /16 bit buffor5/in_10 -> /IN10
- U22 pad 5: /16 bit buffor5/in_11 -> /IN11
- U22 pad 6: /16 bit buffor5/in_12 -> /IN12
- U22 pad 7: /16 bit buffor5/in_13 -> /IN13
- U22 pad 8: /16 bit buffor5/in_14 -> /IN14
- U22 pad 9: /16 bit buffor5/in_15 -> /IN15
- U23 pad 2: /16 bit register1/in_0 -> /OUT0
- U23 pad 3: /16 bit register1/in_1 -> r1we
- U23 pad 4: /16 bit register1/in_2 -> /OUT2
- U23 pad 5: /16 bit register1/in_3 -> /OUT3
- U23 pad 6: /16 bit register1/in_4 -> /OUT4
- U23 pad 7: /16 bit register1/in_5 -> /OUT5
- U23 pad 8: /16 bit register1/in_6 -> /OUT6
- U23 pad 9: /16 bit register1/in_7 -> /OUT7
- U24 pad 4: /16 bit register1/in_10 -> /OUT10
- U25 pad 2: /16 bit register2/in_0 -> /IN0
- U25 pad 3: /16 bit register2/in_1 -> /IN1
- U25 pad 4: /16 bit register2/in_2 -> /IN2
- U25 pad 5: /16 bit register2/in_3 -> /IN3
- U25 pad 6: /16 bit register2/in_4 -> /IN4
- U25 pad 7: /16 bit register2/in_5 -> /IN5
- U25 pad 8: /16 bit register2/in_6 -> /IN6
- U25 pad 9: /16 bit register2/in_7 -> /IN7
- U26 pad 4: /16 bit register2/in_10 -> /IN10
- U27 pad 2: /16 bit register3/in_0 -> /IN0
- U27 pad 3: /16 bit register3/in_1 -> /IN1
- U27 pad 4: /16 bit register3/in_2 -> /IN2
- U27 pad 5: /16 bit register3/in_3 -> /IN3
- U27 pad 6: /16 bit register3/in_4 -> /IN4
- U27 pad 7: /16 bit register3/in_5 -> /IN5
- U27 pad 8: /16 bit register3/in_6 -> /IN6
- U27 pad 9: /16 bit register3/in_7 -> /IN7
- U28 pad 4: /16 bit register3/in_10 -> /IN10
- U29 pad 2: /16 bit register4/in_0 -> /IN0
- U29 pad 3: /16 bit register4/in_1 -> /IN1
- U29 pad 4: /16 bit register4/in_2 -> /IN2
- U29 pad 5: /16 bit register4/in_3 -> /IN3
- U29 pad 6: /16 bit register4/in_4 -> /IN4
- U29 pad 7: /16 bit register4/in_5 -> /IN5
- U29 pad 8: /16 bit register4/in_6 -> /IN6
- U29 pad 9: /16 bit register4/in_7 -> /IN7
- U30 pad 4: /16 bit register4/in_10 -> /IN10
- U31 pad 2: /16 bit register5/in_0 -> /IN0
- U31 pad 3: /16 bit register5/in_1 -> /IN1
- U31 pad 4: /16 bit register5/in_2 -> /IN2
- U31 pad 5: /16 bit register5/in_3 -> /IN3
- U31 pad 6: /16 bit register5/in_4 -> /IN4
- U31 pad 7: /16 bit register5/in_5 -> /IN5
- U31 pad 8: /16 bit register5/in_6 -> /IN6
- U31 pad 9: /16 bit register5/in_7 -> /IN7
- U32 pad 4: /16 bit register5/in_10 -> /IN10
- U33 pad 2: /16 bit register6/in_0 -> /IN0
- U33 pad 3: /16 bit register6/in_1 -> /IN1
- U33 pad 4: /16 bit register6/in_2 -> /IN2
- U33 pad 5: /16 bit register6/in_3 -> /IN3
- U33 pad 6: /16 bit register6/in_4 -> /IN4
- U33 pad 7: /16 bit register6/in_5 -> /IN5
- U33 pad 8: /16 bit register6/in_6 -> /IN6
- U33 pad 9: /16 bit register6/in_7 -> /IN7
- U34 pad 4: /16 bit register6/in_10 -> /IN10
- U35 pad 2: /16 bit register7/in_0 -> /IN0
- U35 pad 3: /16 bit register7/in_1 -> /IN1
- U35 pad 4: /16 bit register7/in_2 -> /IN2
- U35 pad 5: /16 bit register7/in_3 -> /IN3
- U35 pad 6: /16 bit register7/in_4 -> /IN4
- U35 pad 7: /16 bit register7/in_5 -> /IN5
- U35 pad 8: /16 bit register7/in_6 -> /IN6
- U35 pad 9: /16 bit register7/in_7 -> /IN7
- U36 pad 4: /16 bit register7/in_10 -> /IN10
- U37 pad 2: /16 bit register8/in_0 -> /IN0
- U37 pad 3: /16 bit register8/in_1 -> /IN1
- U37 pad 4: /16 bit register8/in_2 -> /IN2
- U37 pad 5: /16 bit register8/in_3 -> /IN3
- U37 pad 6: /16 bit register8/in_4 -> /IN4
- U37 pad 7: /16 bit register8/in_5 -> /IN5
- U37 pad 8: /16 bit register8/in_6 -> /IN6
- U37 pad 9: /16 bit register8/in_7 -> /IN7
- U38 pad 4: /16 bit register8/in_10 -> /IN10
- U39 pad 2: /16 bit register9/in_0 -> /IN0
- U39 pad 3: /16 bit register9/in_1 -> /IN1
- U39 pad 4: /16 bit register9/in_2 -> /IN2
- U39 pad 5: /16 bit register9/in_3 -> /IN3
- U39 pad 6: /16 bit register9/in_4 -> /IN4
- U39 pad 7: /16 bit register9/in_5 -> /IN5
- U39 pad 8: /16 bit register9/in_6 -> /IN6
- U39 pad 9: /16 bit register9/in_7 -> /IN7
- U40 pad 4: /16 bit register9/in_10 -> /IN10
- U41 pad 2: /16 bit register10/in_0 -> /IN0
- U41 pad 3: /16 bit register10/in_1 -> /IN1
- U41 pad 4: /16 bit register10/in_2 -> /IN2
- U41 pad 5: /16 bit register10/in_3 -> /IN3
- U41 pad 6: /16 bit register10/in_4 -> /IN4
- U41 pad 7: /16 bit register10/in_5 -> /IN5
- U41 pad 8: /16 bit register10/in_6 -> /IN6
- U41 pad 9: /16 bit register10/in_7 -> /IN7
- U42 pad 4: /16 bit register10/in_10 -> /IN10
- U43 pad 2: /16 bit register11/in_0 -> /IN0
- U43 pad 3: /16 bit register11/in_1 -> /IN1
- U43 pad 4: /16 bit register11/in_2 -> /IN2
- U43 pad 5: /16 bit register11/in_3 -> /IN3
- U43 pad 6: /16 bit register11/in_4 -> /IN4
- U43 pad 7: /16 bit register11/in_5 -> /IN5
- U43 pad 8: /16 bit register11/in_6 -> /IN6
- U43 pad 9: /16 bit register11/in_7 -> /IN7
- U44 pad 4: /16 bit register11/in_10 -> /IN10
- U45 pad 2: /16 bit register12/in_0 -> /IN0
- U45 pad 3: /16 bit register12/in_1 -> /IN1
- U45 pad 4: /16 bit register12/in_2 -> /IN2
- U45 pad 5: /16 bit register12/in_3 -> /IN3
- U45 pad 6: /16 bit register12/in_4 -> /IN4
- U45 pad 7: /16 bit register12/in_5 -> /IN5
- U45 pad 8: /16 bit register12/in_6 -> /IN6
- U45 pad 9: /16 bit register12/in_7 -> /IN7
- U46 pad 4: /16 bit register12/in_10 -> /IN10
- U47 pad 2: /16 bit register13/in_0 -> /IN0
- U47 pad 3: /16 bit register13/in_1 -> /IN1
- U47 pad 4: /16 bit register13/in_2 -> /IN2
- U47 pad 5: /16 bit register13/in_3 -> /IN3
- U47 pad 6: /16 bit register13/in_4 -> /IN4
- U47 pad 7: /16 bit register13/in_5 -> /IN5
- U47 pad 8: /16 bit register13/in_6 -> /IN6
- U47 pad 9: /16 bit register13/in_7 -> /IN7
- U48 pad 4: /16 bit register13/in_10 -> /IN10
- U49 pad 2: /16 bit register14/in_0 -> /IN0
- U49 pad 3: /16 bit register14/in_1 -> /IN1
- U49 pad 4: /16 bit register14/in_2 -> /IN2
- U49 pad 5: /16 bit register14/in_3 -> /IN3
- U49 pad 6: /16 bit register14/in_4 -> /IN4
- U49 pad 7: /16 bit register14/in_5 -> /IN5
- U49 pad 8: /16 bit register14/in_6 -> /IN6
- U49 pad 9: /16 bit register14/in_7 -> /IN7
- U50 pad 4: /16 bit register14/in_10 -> /IN10
- U51 pad 2: /16 bit register15/in_0 -> /IN0
- U51 pad 3: /16 bit register15/in_1 -> /IN1
- U51 pad 4: /16 bit register15/in_2 -> /IN2
- U51 pad 5: /16 bit register15/in_3 -> /IN3
- U51 pad 6: /16 bit register15/in_4 -> /IN4
- U51 pad 7: /16 bit register15/in_5 -> /IN5
- U51 pad 8: /16 bit register15/in_6 -> /IN6
- U51 pad 9: /16 bit register15/in_7 -> /IN7
- U52 pad 4: /16 bit register15/in_10 -> /IN10
- U7 pad 11: /16 bit buffor/out_7 -> /OUT7
- U7 pad 12: /16 bit buffor/out_6 -> /OUT6
- U7 pad 13: /16 bit buffor/out_5 -> /OUT5
- U7 pad 14: /16 bit buffor/out_4 -> /OUT4
- U7 pad 15: /16 bit buffor/out_3 -> /OUT3
- U7 pad 16: /16 bit buffor/out_2 -> /OUT2
- U7 pad 17: /16 bit buffor/out_1 -> r1we
- U7 pad 18: /16 bit buffor/out_0 -> /OUT0
- U7 pad 2: /16 bit buffor/in_0 -> /IN0
- U7 pad 3: /16 bit buffor/in_1 -> /IN1
- U7 pad 4: /16 bit buffor/in_2 -> /IN2
- U7 pad 5: /16 bit buffor/in_3 -> /IN3
- U7 pad 6: /16 bit buffor/in_4 -> /IN4
- U7 pad 7: /16 bit buffor/in_5 -> /IN5
- U7 pad 8: /16 bit buffor/in_6 -> /IN6
- U7 pad 9: /16 bit buffor/in_7 -> /IN7
- U8 pad 11: /16 bit buffor/out_15 -> /OUT15
- U8 pad 12: /16 bit buffor/out_14 -> /OUT14
- U8 pad 13: /16 bit buffor/out_13 -> /OUT13
- U8 pad 14: /16 bit buffor/out_12 -> /OUT12
- U8 pad 15: /16 bit buffor/out_11 -> /OUT11
- U8 pad 16: /16 bit buffor/out_10 -> /OUT10
- U8 pad 17: /16 bit buffor/out_9 -> /OUT9
- U8 pad 18: /16 bit buffor/out_8 -> /OUT8
- U8 pad 2: /16 bit buffor/in_8 -> /IN8
- U8 pad 3: /16 bit buffor/in_9 -> /IN9
- U8 pad 4: /16 bit buffor/in_10 -> /IN10
- U8 pad 5: /16 bit buffor/in_11 -> /IN11
- U8 pad 6: /16 bit buffor/in_12 -> /IN12
- U8 pad 7: /16 bit buffor/in_13 -> /IN13
- U8 pad 8: /16 bit buffor/in_14 -> /IN14
- U8 pad 9: /16 bit buffor/in_15 -> /IN15
- U9 pad 12: /16 bit register/out_7 -> /OUT7
- U9 pad 13: /16 bit register/out_6 -> /OUT6
- U9 pad 14: /16 bit register/out_5 -> /OUT5
- U9 pad 15: /16 bit register/out_4 -> /OUT4
- U9 pad 16: /16 bit register/out_3 -> /OUT3
- U9 pad 17: /16 bit register/out_2 -> /OUT2
- U9 pad 18: /16 bit register/out_1 -> r1we
- U9 pad 19: /16 bit register/out_0 -> /OUT0
- U9 pad 2: /16 bit register/in_0 -> /OUT0
- U9 pad 3: /16 bit register/in_1 -> r1we
- U9 pad 4: /16 bit register/in_2 -> /OUT2
- U9 pad 5: /16 bit register/in_3 -> /OUT3
- U9 pad 6: /16 bit register/in_4 -> /OUT4
- U9 pad 7: /16 bit register/in_5 -> /OUT5
- U9 pad 8: /16 bit register/in_6 -> /OUT6
- U9 pad 9: /16 bit register/in_7 -> /OUT7
Routing:
- net /IN0: track 0.00 -> 66.7 mm
- net /IN2: track 0.00 -> 27.0 mm
- net /16 bit register15/in_2: track 27.0 -> 0.00 mm
- net /IN7: track 0.00 -> 5.85 mm
- net /16 bit register15/in_7: track 5.85 -> 0.00 mm
- net /IN6: track 0.00 -> 2.95 mm
- net /16 bit register15/in_6: track 2.95 -> 0.00 mm
