File: PCB/Kicad/reg/_autosave-running_and_8b.kicad_sch (KiCad schematic)
At the start: 4 parts, among them U91 74LS08, U92 74LS08

Commit message: VCC
Connections:
- net +5V renamed VCC
- net 0 renamed GND
