File: PCB/Kicad/reg/_autosave-reg.kicad_sch (KiCad schematic)
At the start: 7 parts, among them J1 Conn_02x10_Counter_Clockwise, J10 Conn_02x10_Counter_Clockwise, U1 74LS10, U2 4069, U85 74148

Commit message: VCC
Connections:
- net +5V: no longer C83.1, C84.1, U1.14 (VCC), U2.14 (VDD)
- net 0: no longer U85.8 (GND)
- net GND: now also J1.8 (Pin_8)
- net VCC: now reaches J1.7 (Pin_7)
- net VCC: now also C83.1, C84.1, U1.14 (VCC), U2.14 (VDD)
- no-connect marks 29 -> 27
Other:
- sheet 16 bit buffor10 ports: added GND, VCC; removed none
- sheet 16 bit buffor11 ports: added GND, VCC; removed none
- sheet 16 bit buffor12 ports: added GND, VCC; removed none
- sheet 16 bit buffor13 ports: added GND, VCC; removed none
- sheet 16 bit buffor14 ports: added GND, VCC; removed none
- sheet 16 bit buffor15 ports: added GND, VCC; removed none
- sheet 16 bit buffor16 ports: added GND, VCC; removed none
- sheet 16 bit buffor17 ports: added GND, VCC; removed none
- sheet 16 bit buffor18 ports: added GND, VCC; removed none
- sheet 16 bit buffor19 ports: added GND, VCC; removed none
- sheet 16 bit buffor2 ports: added GND, VCC; removed none
- sheet 16 bit buffor20 ports: added GND, VCC; removed none
- sheet 16 bit buffor22 ports: added GND, VCC; removed none
- sheet 16 bit buffor23 ports: added GND, VCC; removed none
- sheet 16 bit buffor24 ports: added GND, VCC; removed none
- sheet 16 bit buffor3 ports: added GND, VCC; removed none
- sheet 16 bit buffor4 ports: added GND, VCC; removed none
- sheet 16 bit buffor5 ports: added GND, VCC; removed none
- sheet 16 bit buffor6 ports: added GND, VCC; removed none
- sheet 16 bit buffor7 ports: added GND, VCC; removed none
- sheet 16 bit buffor8 ports: added GND, VCC; removed none
- sheet 16 bit buffor9 ports: added GND, VCC; removed none
- sheet 16 bit register10 ports: added GND, VCC; removed none
- sheet 16 bit register11 ports: added GND, VCC; removed none
- sheet 16 bit register12 ports: added GND, VCC; removed none
- sheet 16 bit register13 ports: added GND; removed none
- sheet 16 bit register14 ports: added GND, VCC; removed none
- sheet 16 bit register15 ports: added GND, VCC; removed none
- sheet 16 bit register17 ports: added GND, VCC; removed none
- sheet 16 bit register18 ports: added GND, VCC; removed none
- sheet 16 bit register19 ports: added GND, VCC; removed none
- sheet 16 bit register2 ports: added GND, VCC; removed none
- sheet 16 bit register3 ports: added GND, VCC; removed none
- sheet 16 bit register4 ports: added GND, VCC; removed none
- sheet 16 bit register5 ports: added GND, VCC; removed none
- sheet 16 bit register6 ports: added GND, VCC; removed none
- sheet 16 bit register7 ports: added GND, VCC; removed none
- sheet 16 bit register8 ports: added GND, VCC; removed none
- sheet 16 bit register9 ports: added GND, VCC; removed none
- sheet T74154 ports: added GND, VCC; removed none
- sheet T74155 ports: added GND, VCC; removed none
- sheet octal_and ports: added GND, VCC; removed none
- sheet running_and_8b ports: added GND, VCC; removed none

Commit message: everything_works
Connections:
- net +5V: now also C83.1, C84.1, U1.14 (VCC), U2.14 (VDD); no longer U85.16 (VCC)
- net GND: now also U85.8 (GND)
- net VCC: now also U85.16 (VCC); no longer C83.1, C84.1, U1.14 (VCC), U2.14 (VDD)
Other:
- sheet 16 bit register13 ports: added VCC; removed none
Changed lines of the file:
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@@
 	)
 	(junction
-		(at 29.21 39.37)
-		(diameter 0)
-		(color 0 0 0 0)
-	)
-	(junction
 		(at 58.42 57.15)
 		(diameter 0)
@@
 	)
 	(junction
-		(at 29.21 66.04)
-		(diameter 0)
-		(color 0 0 0 0)
-	)
-	(junction
 		(at 434.34 368.3)
 		(diameter 0)
@@
 	(wire
 		(pts
-			(xy 29.21 69.85) (xy 29.21 66.04)
-		)
-		(stroke
-			(width 0)
-			(type default)
-		)
-	)
-	(wire
-		(pts
 			(xy 439.42 622.3) (xy 439.42 628.65)
 		)
@@
 	(wire
 		(pts
-			(xy 19.05 66.04) (xy 29.21 66.04)
+			(xy 19.05 66.04) (xy 38.1 66.04)
 		)
 		(stroke
@@
 	(wire
 		(pts
-			(xy 38.1 39.37) (xy 59.69 39.37)
-		)
-		(stroke
-			(width 0)
-			(type default)
-		)
-	)
-	(wire
-		(pts
 			(xy 510.54 528.32) (xy 468.63 528.32)
 		)
@@
 	(wire
 		(pts
+			(xy 38.1 39.37) (xy 59.69 39.37)
+		)
+		(stroke
+			(width 0)
+			(type default)
+		)
+	)
+	(wire
+		(pts
 			(xy 510.54 455.93) (xy 468.63 455.93)
 		)
@@
 	(wire
 		(pts
-			(xy 29.21 66.04) (xy 38.1 66.04)
-		)
-		(stroke
-			(width 0)
-			(type default)
-		)
-	)
-	(wire
-		(pts
 			(xy 453.39 87.63) (xy 453.39 96.52)
 		)
@@
 	(wire
 		(pts
-			(xy 29.21 39.37) (xy 38.1 39.37)
+			(xy 19.05 39.37) (xy 38.1 39.37)
 		)
 		(stroke
@@
 	(wire
 		(pts
-			(xy 29.21 36.83) (xy 29.21 39.37)
-		)
-		(stroke
-			(width 0)
-			(type default)
-		)
-	)
-	(wire
-		(pts
 			(xy 541.02 62.23) (xy 549.91 62.23)
 		)
@@
 		)
 	)
-	(wire
-		(pts
-			(xy 19.05 39.37) (xy 29.21 39.37)
-		)
-		(stroke
-			(width 0)
-			(type default)
-		)
-	)
 	(bus
 		(pts
@@
 	)
 	(label "GND"
-		(at 29.21 69.85 270)
-		(effects
-			(font
-				(size 1.27 1.27)
-			)
-			(justify right bottom)
-		)
-	)
-	(label "GND"
 		(at 420.37 416.56 90)
 		(effects
@@
 		)
 	)
-	(label "VCC"
-		(at 29.21 36.83 90)
-		(effects
-			(font
-				(size 1.27 1.27)
-			)
-			(justify left bottom)
-		)
-	)
 	(label "OUT_7_13"
 		(at 537.21 144.78 270)
@@
 	)
 	(label "GND"
-		(at 529.59 88.9 270)
+		(at 525.78 85.09 270)
 		(effects
 			(font
@@
 		)
 	)
+	(label "VCC"
+		(at 525.78 48.26 90)
+		(effects
+			(font
+				(size 1.27 1.27)
+			)
+			(justify left bottom)
+		)
+	)
 	(label "GND"
 		(at 422.91 533.4 90)
@@
 	)
 	(symbol
+		(lib_id "power:GND")
+		(at 38.1 66.04 0)
+		(unit 1)
+		(exclude_from_sim no)
+		(in_bom yes)
+		(on_board yes)
+		(dnp no)
+		(fields_autoplaced yes)
+		(property "Reference" "#PWR02"
+			(at 38.1 72.39 0)
+			(effects
+				(font
+					(size 1.27 1.27)
+				)
+				(hide yes)
+			)
+		)
+		(property "Value" "GND"
+			(at 38.1 71.12 0)
+			(effects
+				(font
+					(size 1.27 1.27)
+				)
+			)
+		)
+		(property "Footprint" ""
+			(at 38.1 66.04 0)
+			(effects
+				(font
+					(size 1.27 1.27)
+				)
+				(hide yes)
+			)
+		)
+		(property "Datasheet" ""
+			(at 38.1 66.04 0)
+			(effects
+				(font
+					(size 1.27 1.27)
+				)
+				(hide yes)
+			)
+		)
+		(property "Description" "Power symbol creates a global label with name \"GND\" , ground"
+			(at 38.1 66.04 0)
+			(effects
+				(font
+					(size 1.27 1.27)
+				)
+				(hide yes)
+			)
+		)
+		(pin "1"
+		)
+		(instances
+			(project ""
+				(path "/e5ea2144-296a-4524-8c5b-c3f6342ff44f"
+					(reference "#PWR02")
+					(unit 1)
+				)
+			)
+		)
+	)
+	(symbol
 		(lib_id "Device:C_Polarized")
 		(at 74.93 53.34 0)
@@
 	)
 	(symbol
+		(lib_id "power:+5V")
+		(at 38.1 39.37 0)
+		(unit 1)
+		(exclude_from_sim no)
+		(in_bom yes)
+		(on_board yes)
+		(dnp no)
+		(fields_autoplaced yes)
+		(property "Reference" "#PWR01"
+			(at 38.1 43.18 0)
+			(effects
+				(font
+					(size 1.27 1.27)
+				)
+				(hide yes)
+			)
+		)
+		(property "Value" "+5V"
+			(at 38.1 34.29 0)
+			(effects
+				(font
+					(size 1.27 1.27)
+				)
+			)
+		)
+		(property "Footprint" ""
+			(at 38.1 39.37 0)
+			(effects
+				(font
+					(size 1.27 1.27)
+				)
+				(hide yes)
+			)
+		)
+		(property "Datasheet" ""
+			(at 38.1 39.37 0)
+			(effects
+				(font
+					(size 1.27 1.27)
+				)
+				(hide yes)
+			)
+		)
+		(property "Description" "Power symbol creates a global label with name \"+5V\""
+			(at 38.1 39.37 0)
+			(effects
+				(font
+					(size 1.27 1.27)
+				)
+				(hide yes)
+			)
+		)
+		(pin "1"
+		)
+		(instances
+			(project ""
+				(path "/e5ea2144-296a-4524-8c5b-c3f6342ff44f"
+					(reference "#PWR01")
+					(unit 1)
+				)
+			)
+		)
+	)
+	(symbol
 		(lib_id "74xx:74LS10")
 		(at 181.61 210.82 0)
@@
 	)
 	(symbol
-		(lib_id "power:+5V")
-		(at 525.78 48.26 0)
-		(unit 1)
-		(exclude_from_sim no)
-		(in_bom yes)
-		(on_board yes)
-		(dnp no)
-		(fields_autoplaced yes)
-		(property "Reference" "#PWR0121"
-			(at 525.78 52.07 0)
-			(effects
-				(font
-					(size 1.27 1.27)
-				)
-				(hide yes)
-			)
-		)
-		(property "Value" "+5V"
-			(at 525.78 43.18 0)
-			(effects
-				(font
-					(size 1.27 1.27)
-				)
-			)
-		)
-		(property "Footprint" ""
-			(at 525.78 48.26 0)
-			(effects
-				(font
-					(size 1.27 1.27)
-				)
-				(hide yes)
-			)
-		)
-		(property "Datasheet" ""
-			(at 525.78 48.26 0)
-			(effects
-				(font
-					(size 1.27 1.27)
-				)
-				(hide yes)
-			)
-		)
-		(property "Description" "Power symbol creates a global label with name \"+5V\""
-			(at 525.78 48.26 0)
-			(effects
-				(font
-					(size 1.27 1.27)
-				)
-				(hide yes)
-			)
-		)
-		(pin "1"
-		)
-		(instances
-			(project ""
-				(path "/e5ea2144-296a-4524-8c5b-c3f6342ff44f"
-					(reference "#PWR0121")
-					(unit 1)
-				)
-			)
-		)
-	)
-	(symbol
 		(lib_id "74xx:74LS10")
 		(at 168.91 252.73 0)
@@
 			(effects
 				(font
+					(size 1.27 1.27)
+				)
+				(justify right)
+			)
+		)
+		(pin "VCC" input
+			(at 420.37 609.6 90)
+			(effects
+				(font
