File: PCB/Kicad/reg/T74154.kicad_sch (KiCad schematic)
At the start: 4 parts, among them U13 74AHC1G02, U14 CD74HC4067M

Commit message: change_bus
Changed lines of the file:
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@@
-	(wire
-		(pts
-			(xy 52.07 52.07) (xy 82.55 52.07)
-		)
-		(stroke
-			(width 0)
-			(type default)
-		)
-	)
 	(wire
 		(pts
@@
 		)
 	)
+	(hierarchical_label "1"
+		(shape input)
+		(at 82.55 52.07 180)
+		(effects
+			(font
+				(size 1.27 1.27)
+			)
+			(justify right)
+		)
+	)
 	(hierarchical_label "out_8"
 		(shape output)
@@
 		)
 	)
-	(hierarchical_label "1"
-		(shape input)
-		(at 52.07 52.07 180)
-		(effects
-			(font
-				(size 1.27 1.27)
-			)
-			(justify right)
-		)
-	)
 	(hierarchical_label "out_10"
 		(shape output)
@@
 		)
 	)
+	(hierarchical_label "C"
+		(shape input)
+		(at 82.55 67.31 180)
+		(effects
+			(font
+				(size 1.27 1.27)
+			)
+			(justify right)
+		)
+	)
 	(hierarchical_label "out_2"
 		(shape output)
@@
 		)
 	)
+	(hierarchical_label "out_11"
+		(shape output)
+		(at 107.95 74.93 0)
+		(effects
+			(font
+				(size 1.27 1.27)
+			)
+			(justify left)
+		)
+	)
 	(hierarchical_label "D"
 		(shape input)
@@
 		)
 	)
+	(hierarchical_label "B"
+		(shape input)
+		(at 82.55 64.77 180)
+		(effects
+			(font
+				(size 1.27 1.27)
+			)
+			(justify right)
+		)
+	)
+	(hierarchical_label "out_7"
+		(shape output)
+		(at 107.95 64.77 0)
+		(effects
+			(font
+				(size 1.27 1.27)
+			)
+			(justify left)
+		)
+	)
+	(hierarchical_label "G1"
+		(shape input)
+		(at 33.02 99.06 180)
+		(effects
+			(font
+				(size 1.27 1.27)
+			)
+			(justify right)
+		)
+	)
 	(hierarchical_label "A"
 		(shape input)
@@
 		)
 	)
-	(hierarchical_label "out_11"
-		(shape output)
-		(at 107.95 74.93 0)
-		(effects
-			(font
-				(size 1.27 1.27)
-			)
-			(justify left)
-		)
-	)
-	(hierarchical_label "out_7"
-		(shape output)
-		(at 107.95 64.77 0)
-		(effects
-			(font
-				(size 1.27 1.27)
-			)
-			(justify left)
-		)
-	)
-	(hierarchical_label "G1"
-		(shape input)
-		(at 33.02 99.06 180)
-		(effects
-			(font
-				(size 1.27 1.27)
-			)
-			(justify right)
-		)
-	)
 	(hierarchical_label "out_0"
 		(shape output)
@@
 		)
 	)
-	(hierarchical_label "B"
-		(shape input)
-		(at 82.55 64.77 180)
-		(effects
-			(font
-				(size 1.27 1.27)
-			)
-			(justify right)
-		)
-	)
-	(hierarchical_label "C"
-		(shape input)
-		(at 82.55 67.31 180)
-		(effects
-			(font
-				(size 1.27 1.27)
-			)
-			(justify right)
-		)
-	)

Commit message: everything_works
Connections:
- net +5V renamed VCC
- net 0 renamed GND
Changed lines of the file:
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@@
-	)
-	(junction
-		(at 138.43 35.56)
-		(diameter 0)
-		(color 0 0 0 0)
 	)
 	(junction
@@
 	(wire
 		(pts
-			(xy 138.43 35.56) (xy 154.94 35.56)
+			(xy 134.62 35.56) (xy 154.94 35.56)
 		)
 		(stroke
@@
 	(wire
 		(pts
-			(xy 138.43 35.56) (xy 134.62 35.56)
-		)
-		(stroke
-			(width 0)
-			(type default)
-		)
-	)
-	(wire
-		(pts
 			(xy 134.62 45.72) (xy 138.43 45.72)
 		)
@@
 		)
 	)
+	(hierarchical_label "GND"
+		(shape output)
+		(at 138.43 48.26 270)
+		(effects
+			(font
+				(size 1.27 1.27)
+			)
+			(justify right)
+		)
+	)
 	(hierarchical_label "1"
 		(shape input)
@@
 		(shape output)
 		(at 107.95 57.15 0)
+		(effects
+			(font
+				(size 1.27 1.27)
+			)
+			(justify left)
+		)
+	)
+	(hierarchical_label "VCC"
+		(shape input)
+		(at 139.7 35.56 90)
 		(effects
 			(font
@@
 					(unit 1)
 				)
-			)
-		)
-	)
-	(symbol
-		(lib_id "power:+1V35")
-		(at 138.43 35.56 0)
-		(unit 1)
-		(exclude_from_sim no)
-		(in_bom yes)
-		(on_board yes)
-		(dnp no)
-		(fields_autoplaced yes)
-		(property "Reference" "#PWR015"
-			(at 138.43 39.37 0)
-			(effects
-				(font
-					(size 1.27 1.27)
-				)
-				(hide yes)
-			)
-		)
-		(property "Value" "+5V"
-			(at 138.43 30.48 0)
-			(effects
-				(font
-					(size 1.27 1.27)
-				)
-			)
-		)
-		(property "Footprint" ""
-			(at 138.43 35.56 0)
-			(effects
-				(font
-					(size 1.27 1.27)
-				)
-				(hide yes)
-			)
-		)
-		(property "Datasheet" ""
-			(at 138.43 35.56 0)
-			(effects
-				(font
-					(size 1.27 1.27)
-				)
-				(hide yes)
-			)
-		)
-		(property "Description" "Power symbol creates a global label with name \"+1V35\""
-			(at 138.43 35.56 0)
-			(effects
-				(font
-					(size 1.27 1.27)
-				)
-				(hide yes)
-			)
-		)
-		(pin "1"
-		)
-		(instances
-			(project "reg"
-				(path "/e5ea2144-296a-4524-8c5b-c3f6342ff44f/9e772c47-ba7c-4f5a-ad9a-0264023671f0"
-					(reference "#PWR015")
-					(unit 1)
-				)
-				(path "/e5ea2144-296a-4524-8c5b-c3f6342ff44f/e31facd4-6679-4b5c-a8ae-0d8e900d2b68"
-					(reference "#PWR0124")
-					(unit 1)
-				)
-			)
-		)
-	)
-	(symbol
-		(lib_id "Simulation_SPICE:0")
-		(at 138.43 48.26 0)
-		(unit 1)
-		(exclude_from_sim no)
-		(in_bom yes)
-		(on_board yes)
-		(dnp no)
-		(property "Reference" "#GND015"
-			(at 138.43 53.34 0)
-			(effects
-				(font
-					(size 1.27 1.27)
-				)
-				(hide yes)
-			)
-		)
-		(property "Value" "0"
-			(at 140.97 48.26 0)
-			(effects
-				(font
-					(size 1.27 1.27)
-				)
-			)
-		)
-		(property "Footprint" ""
-			(at 138.43 48.26 0)
-			(effects
-				(font
-					(size 1.27 1.27)
-				)
-				(hide yes)
-			)
-		)
-		(property "Datasheet" "https://ngspice.sourceforge.io/docs/ngspice-html-manual/manual.xhtml#subsec_Circuit_elements__device"
-			(at 138.43 58.42 0)
-			(effects
-				(font
-					(size 1.27 1.27)
-				)
-				(hide yes)
-			)
-		)
-		(property "Description" "0V reference potential for simulation"
-			(at 138.43 55.88 0)
-			(effects
-				(font
-					(size 1.27 1.27)
-				)
-				(hide yes)
-			)
-		)
-		(pin "1"
-		)
-		(instances
-			(project "reg"
-				(path "/e5ea2144-296a-4524-8c5b-c3f6342ff44f/9e772c47-ba7c-4f5a-ad9a-0264023671f0"
-					(reference "#GND015")
-					(unit 1)
-				)
-				(path "/e5ea2144-296a-4524-8c5b-c3f6342ff44f/e31facd4-6679-4b5c-a8ae-0d8e900d2b68"
-					(reference "#GND0124")
-					(unit 1)
-				)

Commit message: capacitor
Parts:
- removed U13: 74AHC1G02, symbol 74xGxx:74AHC1G02
- added U83: 4001, Package_DIP:DIP-14_W7.62mm_SMDSocket_SmallPads, symbol 4xxx:4001
- C7, C8: footprint Capacitor_SMD:CP_Elec_4x3 -> Capacitor_SMD:C_0402_1005Metric
Connections:
- net G1: now also U83.1
- net G2: now also U83.2
- net GND: now also U83.7 (VSS)
- net VCC: now also U83.14 (VDD)
- net at U14.15 (~{E}): now also U83.3
- no-connect marks 0 -> 9

Commit message: fix
Parts:
- removed U83: 4001, Package_DIP:DIP-14_W7.62mm_SMDSocket_SmallPads, symbol 4xxx:4001
- added U3: 74LS02, Package_DIP:DIP-14_W7.62mm_SMDSocket_SmallPads, symbol 74xx:74LS02
Connections:
- net G1: now also U3.2
- net G2: now also U3.3
- net GND: now also U3.7 (GND)
- net at U14.15 (~{E}): now also U3.1
- net VCC renamed +5V
- net +5V: now also U3.11, U3.12, U3.14 (VCC), U3.5, U3.6, U3.8, U3.9
- no-connect marks 9 -> 3
