File: PCB/Kicad/reg/reg.kicad_sch (KiCad schematic)
At the start: 7 parts, among them J1 Conn_02x10_Counter_Clockwise, J10 Conn_02x10_Counter_Clockwise, U1 74LS10, U2 4069, U85 74148

Commit message: everything_works
Connections:
- net +5V is gone; now on net VCC: C83.1, C84.1, U1.14 (VCC), U2.14 (VDD), U85.16 (VCC)
- net 0: no longer U85.8 (GND)
- net GND: now also J1.8 (Pin_8), U85.8 (GND)
- net VCC: now reaches J1.7 (Pin_7)
- no-connect marks 29 -> 27
Other:
- sheet 16 bit buffor10 ports: added GND, VCC; removed none
- sheet 16 bit buffor11 ports: added GND, VCC; removed none
- sheet 16 bit buffor12 ports: added GND, VCC; removed none
- sheet 16 bit buffor13 ports: added GND, VCC; removed none
- sheet 16 bit buffor14 ports: added GND, VCC; removed none
- sheet 16 bit buffor15 ports: added GND, VCC; removed none
- sheet 16 bit buffor16 ports: added GND, VCC; removed none
- sheet 16 bit buffor17 ports: added GND, VCC; removed none
- sheet 16 bit buffor18 ports: added GND, VCC; removed none
- sheet 16 bit buffor19 ports: added GND, VCC; removed none
- sheet 16 bit buffor2 ports: added GND, VCC; removed none
- sheet 16 bit buffor20 ports: added GND, VCC; removed none
- sheet 16 bit buffor22 ports: added GND, VCC; removed none
- sheet 16 bit buffor23 ports: added GND, VCC; removed none
- sheet 16 bit buffor24 ports: added GND, VCC; removed none
- sheet 16 bit buffor3 ports: added GND, VCC; removed none
- sheet 16 bit buffor4 ports: added GND, VCC; removed none
- sheet 16 bit buffor5 ports: added GND, VCC; removed none
- sheet 16 bit buffor6 ports: added GND, VCC; removed none
- sheet 16 bit buffor7 ports: added GND, VCC; removed none
- sheet 16 bit buffor8 ports: added GND, VCC; removed none
- sheet 16 bit buffor9 ports: added GND, VCC; removed none
- sheet 16 bit register10 ports: added GND, VCC; removed none
- sheet 16 bit register11 ports: added GND, VCC; removed none
- sheet 16 bit register12 ports: added GND, VCC; removed none
- sheet 16 bit register13 ports: added GND, VCC; removed none
- sheet 16 bit register14 ports: added GND, VCC; removed none
- sheet 16 bit register15 ports: added GND, VCC; removed none
- sheet 16 bit register17 ports: added GND, VCC; removed none
- sheet 16 bit register18 ports: added GND, VCC; removed none
- sheet 16 bit register19 ports: added GND, VCC; removed none
- sheet 16 bit register2 ports: added GND, VCC; removed none
- sheet 16 bit register3 ports: added GND, VCC; removed none
- sheet 16 bit register4 ports: added GND, VCC; removed none
- sheet 16 bit register5 ports: added GND, VCC; removed none
- sheet 16 bit register6 ports: added GND, VCC; removed none
- sheet 16 bit register7 ports: added GND, VCC; removed none
- sheet 16 bit register8 ports: added GND, VCC; removed none
- sheet 16 bit register9 ports: added GND, VCC; removed none
- sheet T74154 ports: added GND, VCC; removed none
- sheet T74155 ports: added GND, VCC; removed none
- sheet octal_and ports: added GND, VCC; removed none
- sheet running_and_8b ports: added GND, VCC; removed none

Commit message: capacitor
Parts:
- C83, C84: footprint Capacitor_SMD:CP_Elec_4x3 -> Capacitor_SMD:C_0402_1005Metric
- U2: footprint (none) -> Package_DIP:DIP-14_W7.62mm_SMDSocket_SmallPads
- U85: footprint (none) -> Package_DIP:DIP-16_W7.62mm_SMDSocket_SmallPads

Commit message: fix
Parts:
- removed U2: 4069, Package_DIP:DIP-14_W7.62mm_SMDSocket_SmallPads, symbol 4xxx:4069
- added J11, J12, J13, J14, J15, J16, J17, J2: Conn_02x10_Counter_Clockwise, Connector_PinHeader_2.54mm:PinHeader_2x10_P2.54mm_Horizontal, symbol Connector_Generic:Conn_02x10_Counter_Clockwise
- added U17: 74AHC04, Package_DIP:DIP-14_W7.62mm_SMDSocket_SmallPads, symbol 74xx:74AHC04
Connections:
- net VCC is gone; now on net +5V: C83.1, C84.1, J1.7 (Pin_7), U1.14 (VCC), U85.16 (VCC)
- net 16 bit register18/nWE: now also U17.4
- net GND: now also U85.5 (~{EI}), U17.7 (GND)
- net T74154/G1: now also U17.2
- net mask_restore: now also U17.9
- net mask_save: now also U17.11, U17.3
- net r1we: now also U17.13, U17.5
- net write_enable: now also U17.1
- net +5V: now reaches U1.3
- net +5V: now also U1.10, U1.11, U1.4, U1.5, U1.9, U17.14 (VCC)
- net at U1.1: now also U17.6
- net 0: no longer names the net of J1.18 (Pin_18)
- net 0: no longer U85.5 (~{EI})
- net 1: no longer names the net of J1.19 (Pin_19)
- new net 16 bit buffor23/n0E2: U17.12
- new net 16 bit buffor26/n0E2: U17.10
- new net 16 bit buffor3/n0E2: U17.8
- new net data0: J2.10 (Pin_10)
- new net data1: J2.9 (Pin_9)
- new net data10: J2.11 (Pin_11)
- new net data11: J2.12 (Pin_12)
- new net data12: J2.13 (Pin_13)
- new net data13: J2.14 (Pin_14)
- new net data14: J2.15 (Pin_15)
- new net data15: J2.16 (Pin_16)
- new net data2: J2.8 (Pin_8)
- new net data3: J2.7 (Pin_7)
- new net data4: J2.6 (Pin_6)
- new net data5: J2.5 (Pin_5)
- new net data6: J2.4 (Pin_4)
- new net data7: J2.3 (Pin_3)
- new net data8: J2.2 (Pin_2)
- new net data9: J2.1 (Pin_1)
- new net data_1_0: J11.10 (Pin_10)
- new net data_1_1: J11.9 (Pin_9)
- new net data_1_10: J11.11 (Pin_11)
- new net data_1_11: J11.12 (Pin_12)
- new net data_1_12: J11.13 (Pin_13)
- new net data_1_13: J11.14 (Pin_14)
- new net data_1_14: J11.15 (Pin_15)
- new net data_1_15: J11.16 (Pin_16)
- new net data_1_2: J11.8 (Pin_8)
- new net data_1_3: J11.7 (Pin_7)
- new net data_1_4: J11.6 (Pin_6)
- new net data_1_5: J11.5 (Pin_5)
- new net data_1_6: J11.4 (Pin_4)
- new net data_1_7: J11.3 (Pin_3)
- new net data_1_8: J11.2 (Pin_2)
- new net data_1_9: J11.1 (Pin_1)
- new net data_2_0: J12.10 (Pin_10)
- new net data_2_1: J12.9 (Pin_9)
- new net data_2_10: J12.11 (Pin_11)
- new net data_2_11: J12.12 (Pin_12)
- new net data_2_12: J12.13 (Pin_13)
- new net data_2_13: J12.14 (Pin_14)
- new net data_2_14: J12.15 (Pin_15)
- new net data_2_15: J12.16 (Pin_16)
- new net data_2_2: J12.8 (Pin_8)
- new net data_2_3: J12.7 (Pin_7)
- new net data_2_4: J12.6 (Pin_6)
- new net data_2_5: J12.5 (Pin_5)
- new net data_2_6: J12.4 (Pin_4)
- new net data_2_7: J12.3 (Pin_3)
- new net data_2_8: J12.2 (Pin_2)
- new net data_2_9: J12.1 (Pin_1)
- new net data_3_0: J13.10 (Pin_10)
- new net data_3_1: J13.9 (Pin_9)
- new net data_3_10: J13.11 (Pin_11)
- new net data_3_11: J13.12 (Pin_12)
- new net data_3_12: J13.13 (Pin_13)
- new net data_3_13: J13.14 (Pin_14)
- new net data_3_14: J13.15 (Pin_15)
- new net data_3_15: J13.16 (Pin_16)
- new net data_3_2: J13.8 (Pin_8)
- new net data_3_3: J13.7 (Pin_7)
- new net data_3_4: J13.6 (Pin_6)
- new net data_3_5: J13.5 (Pin_5)
- new net data_3_6: J13.4 (Pin_4)
- new net data_3_7: J13.3 (Pin_3)
- new net data_3_8: J13.2 (Pin_2)
- new net data_3_9: J13.1 (Pin_1)
- new net data_4_0: J14.10 (Pin_10)
- new net data_4_1: J14.9 (Pin_9)
- new net data_4_10: J14.11 (Pin_11)
- new net data_4_11: J14.12 (Pin_12)
- new net data_4_12: J14.13 (Pin_13)
- new net data_4_13: J14.14 (Pin_14)
- new net data_4_14: J14.15 (Pin_15)
- new net data_4_15: J14.16 (Pin_16)
- new net data_4_2: J14.8 (Pin_8)
- new net data_4_3: J14.7 (Pin_7)
- new net data_4_4: J14.6 (Pin_6)
- new net data_4_5: J14.5 (Pin_5)
- new net data_4_6: J14.4 (Pin_4)
- new net data_4_7: J14.3 (Pin_3)
- new net data_4_8: J14.2 (Pin_2)
- new net data_4_9: J14.1 (Pin_1)
- new net data_5_0: J15.10 (Pin_10)
- new net data_5_1: J15.9 (Pin_9)
- new net data_5_10: J15.11 (Pin_11)
- new net data_5_11: J15.12 (Pin_12)
- new net data_5_12: J15.13 (Pin_13)
- new net data_5_13: J15.14 (Pin_14)
- new net data_5_14: J15.15 (Pin_15)
- new net data_5_15: J15.16 (Pin_16)
- new net data_5_2: J15.8 (Pin_8)
- new net data_5_3: J15.7 (Pin_7)
- new net data_5_4: J15.6 (Pin_6)
- new net data_5_5: J15.5 (Pin_5)
- new net data_5_6: J15.4 (Pin_4)
- new net data_5_7: J15.3 (Pin_3)
- new net data_5_8: J15.2 (Pin_2)
- new net data_5_9: J15.1 (Pin_1)
- new net data_6_0: J16.10 (Pin_10)
- new net data_6_1: J16.9 (Pin_9)
- new net data_6_10: J16.11 (Pin_11)
- new net data_6_11: J16.12 (Pin_12)
- new net data_6_12: J16.13 (Pin_13)
- new net data_6_13: J16.14 (Pin_14)
- new net data_6_14: J16.15 (Pin_15)
- new net data_6_15: J16.16 (Pin_16)
- new net data_6_2: J16.8 (Pin_8)
- new net data_6_3: J16.7 (Pin_7)
- new net data_6_4: J16.6 (Pin_6)
- new net data_6_5: J16.5 (Pin_5)
- new net data_6_6: J16.4 (Pin_4)
- new net data_6_7: J16.3 (Pin_3)
- new net data_6_8: J16.2 (Pin_2)
- new net data_6_9: J16.1 (Pin_1)
- new net data_7_0: J17.10 (Pin_10)
- new net data_7_1: J17.9 (Pin_9)
- new net data_7_10: J17.11 (Pin_11)
- new net data_7_11: J17.12 (Pin_12)
- new net data_7_12: J17.13 (Pin_13)
- new net data_7_13: J17.14 (Pin_14)
- new net data_7_14: J17.15 (Pin_15)
- new net data_7_15: J17.16 (Pin_16)
- new net data_7_2: J17.8 (Pin_8)
- new net data_7_3: J17.7 (Pin_7)
- new net data_7_4: J17.6 (Pin_6)
- new net data_7_5: J17.5 (Pin_5)
- new net data_7_6: J17.4 (Pin_4)
- new net data_7_7: J17.3 (Pin_3)
- new net data_7_8: J17.2 (Pin_2)
- new net data_7_9: J17.1 (Pin_1)
- no-connect marks 27 -> 55
Other:
- removed sheet 0000
- removed sheet 16 bit buffor10
- removed sheet 16 bit buffor11
- removed sheet 16 bit buffor12
- removed sheet 16 bit buffor13
- removed sheet 16 bit buffor14
- removed sheet 16 bit buffor15
- removed sheet 16 bit buffor16
- removed sheet 16 bit buffor17
- removed sheet 16 bit buffor18
- removed sheet 16 bit buffor19
- removed sheet 16 bit buffor2
- removed sheet 16 bit buffor20
- removed sheet 16 bit buffor22
- removed sheet 16 bit buffor4
- removed sheet 16 bit buffor5
- removed sheet 16 bit buffor7
- removed sheet 16 bit buffor8
- removed sheet 16 bit buffor9
- removed sheet IO_bus[0..7]_IO_int[8..15]
- removed sheet data
- removed sheet data_1
- removed sheet mask_saved
- removed sheet mask_saved_1
- removed sheet r1_out
- removed sheet reg_out
- added sheet 16 bit buffor21 (untitled.kicad_sch)
- added sheet 16 bit buffor25 (untitled.kicad_sch)
- added sheet 16 bit buffor26 (untitled.kicad_sch)
- added sheet 16 bit buffor27 (untitled.kicad_sch)
- added sheet 16 bit buffor28 (untitled.kicad_sch)
- added sheet 16 bit buffor29 (untitled.kicad_sch)
- added sheet 16 bit buffor30 (untitled.kicad_sch)
- added sheet 16 bit buffor31 (untitled.kicad_sch)
- added sheet 16 bit buffor32 (untitled.kicad_sch)
- added sheet 16 bit buffor33 (untitled.kicad_sch)
- added sheet 16 bit buffor34 (untitled.kicad_sch)
- added sheet 16 bit buffor35 (untitled.kicad_sch)
- added sheet 16 bit buffor36 (untitled.kicad_sch)
- added sheet 16 bit buffor37 (untitled.kicad_sch)
- added sheet 16 bit buffor38 (untitled.kicad_sch)
- added sheet 16 bit buffor39 (untitled.kicad_sch)
- added sheet 16 bit buffor40 (untitled.kicad_sch)
- added sheet 16 bit buffor41 (untitled.kicad_sch)
- sheet 16 bit buffor23 ports: added none; removed GND, VCC
- sheet 16 bit buffor24 ports: added none; removed GND, VCC
- sheet 16 bit buffor3 ports: added none; removed GND, VCC
- sheet 16 bit buffor6 ports: added none; removed GND, VCC
- sheet 16 bit register10 ports: added none; removed GND, VCC
- sheet 16 bit register11 ports: added none; removed GND, VCC
- sheet 16 bit register12 ports: added none; removed GND, VCC
- sheet 16 bit register13 ports: added none; removed GND, VCC
- sheet 16 bit register14 ports: added none; removed GND, VCC
- sheet 16 bit register15 ports: added none; removed GND, VCC
- sheet 16 bit register17 ports: added none; removed GND, VCC
- sheet 16 bit register18 ports: added none; removed GND, VCC
- sheet 16 bit register19 ports: added none; removed GND, VCC
- sheet 16 bit register2 ports: added none; removed GND, VCC
- sheet 16 bit register3 ports: added none; removed GND, VCC
- sheet 16 bit register4 ports: added none; removed GND, VCC
- sheet 16 bit register5 ports: added none; removed GND, VCC
- sheet 16 bit register6 ports: added none; removed GND, VCC
- sheet 16 bit register7 ports: added none; removed GND, VCC
- sheet 16 bit register8 ports: added none; removed GND, VCC
- sheet 16 bit register9 ports: added none; removed GND, VCC
- sheet T74154 ports: added none; removed GND, VCC
- sheet T74155 ports: added none; removed GND, VCC
- sheet octal_and ports: added none; removed GND, VCC
- sheet running_and_8b ports: added none; removed GND, VCC
- moved on the sheet: U1B

Commit message: aaaaaaaaaaaaaaaaaaaaaaaaaaaaaaaaaaaaaaaaaaaa
Parts:
- removed J11, J2: Conn_02x10_Counter_Clockwise, Connector_PinHeader_2.54mm:PinHeader_2x10_P2.54mm_Horizontal, symbol Connector_Generic:Conn_02x10_Counter_Clockwise
- removed unit 3 of U1
- removed unit 1 of U17
- added U29, U30: CD74HC4067M, Package_SO:SOIC-24W_7.5x15.4mm_P1.27mm, symbol 74xx:CD74HC4067M
Connections:
- net +5V: now also U29.1 (COM), U29.15 (~{E}), U30.1 (COM), U30.15 (~{E})
- net OUT_1_10: now also U29.21 (I10)
- net OUT_1_11: now also U29.20 (I11)
- net OUT_1_12: now also U29.19 (I12)
- net OUT_1_13: now also U29.18 (I13)
- net OUT_1_14: now also U29.17 (I14)
- net OUT_1_15: now also U29.16 (I15)
- net OUT_1_2: now also U29.7 (I2)
- net OUT_1_3: now also U29.6 (I3)
- net OUT_1_4: now also U29.5 (I4)
- net OUT_1_5: now also U29.4 (I5)
- net OUT_1_6: now also U29.3 (I6)
- net OUT_1_7: now also U29.2 (I7)
- net OUT_1_8: now also U29.23 (I8)
- net OUT_1_9: now also U29.22 (I9)
- net OUT_7_0: now also U30.9 (I0)
- net OUT_7_1: now also U30.8 (I1)
- net OUT_7_10: now also U30.21 (I10)
- net OUT_7_11: now also U30.20 (I11)
- net OUT_7_12: now also U30.19 (I12)
- net OUT_7_13: now also U30.18 (I13)
- net OUT_7_14: now also U30.17 (I14)
- net OUT_7_15: now also U30.16 (I15)
- net OUT_7_2: now also U30.7 (I2)
- net OUT_7_3: now also U30.6 (I3)
- net OUT_7_4: now also U30.5 (I4)
- net OUT_7_5: now also U30.4 (I5)
- net OUT_7_6: now also U30.3 (I6)
- net OUT_7_7: now also U30.2 (I7)
- net OUT_7_8: now also U30.23 (I8)
- net OUT_7_9: now also U30.22 (I9)
- net a0: now also U30.10 (S0)
- net a1: now also U30.11 (S1)
- net a2: now also U30.14 (S2)
- net a3: now also U30.13 (S3)
- net r1we: now also U29.8 (I1)
- net write_enable: no longer J1.10 (Pin_10)
- net T74154/A: no longer names the net of J1.14 (Pin_14)
- net T74154/A: now also U29.10 (S0)
- net T74154/B: no longer names the net of J1.13 (Pin_13)
- net T74154/B: now also U29.11 (S1)
- net T74154/C: no longer names the net of J1.12 (Pin_12)
- net T74154/C: now also U29.14 (S2)
- net T74154/D: no longer names the net of J1.11 (Pin_11)
- net T74154/D: now also U29.13 (S3)
- no-connect marks 55 -> 46
Other:
- removed sheet T74154
- removed sheet T74155
- sheet 16 bit buffor21 ports: added none; removed nE1
- sheet 16 bit buffor23 ports: added none; removed nE1
- sheet 16 bit buffor24 ports: added none; removed nE1
- sheet 16 bit buffor25 ports: added none; removed nE1
- sheet 16 bit buffor26 ports: added none; removed nE1
- sheet 16 bit buffor27 ports: added none; removed nE1
- sheet 16 bit buffor28 ports: added none; removed nE1
- sheet 16 bit buffor29 ports: added none; removed nE1
- sheet 16 bit buffor3 ports: added none; removed nE1
- sheet 16 bit buffor30 ports: added none; removed nE1
- sheet 16 bit buffor31 ports: added none; removed nE1
- sheet 16 bit buffor32 ports: added none; removed nE1
- sheet 16 bit buffor33 ports: added none; removed nE1
- sheet 16 bit buffor34 ports: added none; removed nE1
- sheet 16 bit buffor35 ports: added none; removed nE1
- sheet 16 bit buffor36 ports: added none; removed nE1
- sheet 16 bit buffor37 ports: added none; removed nE1
- sheet 16 bit buffor38 ports: added none; removed nE1
- sheet 16 bit buffor39 ports: added none; removed nE1
- sheet 16 bit buffor40 ports: added none; removed nE1
- sheet 16 bit buffor41 ports: added none; removed nE1
- sheet 16 bit buffor6 ports: added none; removed nE1
- moved on the sheet: J1

Commit message: aaa
Parts:
- removed J14, J15, J16, J17: Conn_02x10_Counter_Clockwise, Connector_PinHeader_2.54mm:PinHeader_2x10_P2.54mm_Horizontal, symbol Connector_Generic:Conn_02x10_Counter_Clockwise
Connections:
- net r1we: no longer J1.15 (Pin_15)
- net data_2_0: no longer names the net of J12.10 (Pin_10)
- net data_2_1: no longer names the net of J12.9 (Pin_9)
- net data_2_10: no longer names the net of J12.11 (Pin_11)
- net data_2_11: no longer names the net of J12.12 (Pin_12)
- net data_2_12: no longer names the net of J12.13 (Pin_13)
- net data_2_13: no longer names the net of J12.14 (Pin_14)
- net data_2_14: no longer names the net of J12.15 (Pin_15)
- net data_2_15: no longer names the net of J12.16 (Pin_16)
- net data_2_2: no longer names the net of J12.8 (Pin_8)
- net data_2_3: no longer names the net of J12.7 (Pin_7)
- net data_2_4: no longer names the net of J12.6 (Pin_6)
- net data_2_5: no longer names the net of J12.5 (Pin_5)
- net data_2_6: no longer names the net of J12.4 (Pin_4)
- net data_2_7: no longer names the net of J12.3 (Pin_3)
- net data_2_8: no longer names the net of J12.2 (Pin_2)
- net data_2_9: no longer names the net of J12.1 (Pin_1)
- net write_enable: no longer names the net of J1.20 (Pin_20)
- no-connect marks 46 -> 26
Other:
- note removed: "set"
- moved on the sheet: U1B

Commit message: gggggggggggggggggggggggg
Parts:
- added U18: 74AHC04, Package_DIP:DIP-14_W7.62mm_SMDSocket_SmallPads, symbol 74xx:74AHC04
Connections:
- net +5V: no longer U29.1 (COM), U30.1 (COM)
- new net: U18.4, U29.1 (COM)
- new net write_enable: U18.3, U30.1 (COM)

Commit message: bombardino crocodilo
Parts:
- removed J1, J10: Conn_02x10_Counter_Clockwise, Connector_PinHeader_2.54mm:PinHeader_2x10_P2.54mm_Horizontal, symbol Connector_Generic:Conn_02x10_Counter_Clockwise
- removed U18: 74AHC04, Package_DIP:DIP-14_W7.62mm_SMDSocket_SmallPads, symbol 74xx:74AHC04
- added J14: Conn_02x10_Counter_Clockwise, Connector_PinHeader_2.54mm:PinHeader_2x10_P2.54mm_Horizontal, symbol Connector_Generic:Conn_02x10_Counter_Clockwise
- added R1288, R1289, R1290, R1291, R1292, R1293, R1294, R1295, R1296, R1297, R1298, R1299, R1300, R1301, R1302, R1303, R1304, R1305, R1306, R1307, R1308, R1309, R1310, R1311, R1312, R1313, R1314, R1315, R1316, R1317, R1318: 620, Resistor_SMD:R_0402_1005Metric_Pad0.72x0.64mm_HandSolder, symbol Device:R
- added unit 2 of U17
Connections:
- net a0 is gone; now on net ID_REG_SEL_0: U30.10 (S0)
- net a1 is gone; now on net ID_REG_SEL_1: U30.11 (S1)
- net a2 is gone; now on net ID_REG_SEL_2: U30.14 (S2)
- net a3 is gone; now on net ID_REG_SEL_3: U30.13 (S3)
- net data_3_0 is gone; now on net +5V: J13.10 (Pin_10)
- net data_3_10 is gone; now on net GND: J13.11 (Pin_11)
- net data_3_11 is gone; now on net mask_restore: J13.12 (Pin_12)
- net data_3_12 is gone; now on net mask_save: J13.13 (Pin_13)
- net data_3_13 is gone; now on net GND: J13.14 (Pin_14)
- net data_3_14 is gone; now on net INT: J13.15 (Pin_15)
- net data_3_15 is gone; now on net Interupt_ID_0: J13.16 (Pin_16)
- net data_3_9 is gone; now on net +5V: J13.1 (Pin_1)
- net +5V: now also J12.1 (Pin_1), J12.10 (Pin_10), U1.10, U1.11, U1.9, U29.24 (VCC), U30.24 (VCC), R1288.2, R1289.2, R1290.2, R1291.2, R1292.2, R1293.2, R1294.2, R1295.2, R1296.2, R1297.2, R1298.2, R1299.2, R1300.2, R1301.2, R1302.2, R1303.2, R1304.2, R1305.2, R1306.2, R1307.2, R1308.2, R1309.2, R1310.2, R1311.2, R1312.2, R1313.2, R1314.2, R1315.2, R1316.2, R1317.2, R1318.2
- net 16 bit register18/nWE: now also U17.2; no longer U17.4
- net GND: now also J12.11 (Pin_11), J12.14 (Pin_14), J12.17 (Pin_17), J12.20 (Pin_20), J13.17 (Pin_17), J13.20 (Pin_20), U29.12 (GND), U30.12 (GND), J14.11 (Pin_11), J14.19 (Pin_19), J14.4 (Pin_4), J14.7 (Pin_7)
- net OUT_1_10: now also R1309.1
- net OUT_1_11: now also R1308.1
- net OUT_1_12: now also R1307.1
- net OUT_1_13: now also R1306.1
- net OUT_1_14: now also R1305.1
- net OUT_1_15: now also R1304.1
- net OUT_1_2: now also R1317.1
- net OUT_1_3: now also R1316.1
- net OUT_1_4: now also R1315.1
- net OUT_1_5: now also R1314.1
- net OUT_1_6: now also R1313.1
- net OUT_1_7: now also R1312.1
- net OUT_1_8: now also R1311.1
- net OUT_1_9: now also R1310.1
- net OUT_7_0: now also R1303.1
- net OUT_7_1: now also R1302.1
- net OUT_7_10: now also R1293.1
- net OUT_7_11: now also R1292.1
- net OUT_7_12: now also R1291.1
- net OUT_7_13: now also R1290.1
- net OUT_7_14: now also R1289.1
- net OUT_7_15: now also R1288.1
- net OUT_7_2: now also R1301.1
- net OUT_7_3: now also R1300.1
- net OUT_7_4: now also R1299.1
- net OUT_7_5: now also R1298.1
- net OUT_7_6: now also R1297.1
- net OUT_7_7: now also R1296.1
- net OUT_7_8: now also R1295.1
- net OUT_7_9: now also R1294.1
- net busy: now also J12.18 (Pin_18)
- net clk: now also J12.19 (Pin_19)
- net mask_save: now also U17.1; no longer U17.3
- net r1we: now also R1318.1
- net write_enable: now also U17.3
- net Interupt_ID_0: now reaches U85.9 (~{S0})
- net Interupt_ID_1: now reaches U85.7 (~{S1})
- net Interupt_ID_1: now also J13.18 (Pin_18)
- net Interupt_ID_2: now reaches U85.6 (~{S2})
- net Interupt_ID_2: now also J13.19 (Pin_19)
- net INT: now reaches U85.14 (~{GS})
- net at U29.1 (COM): now also U17.4
- net ID_REG_SEL_0: now reaches U29.10 (S0)
- net ID_REG_SEL_0: now also J12.12 (Pin_12)
- net ID_REG_SEL_1: now reaches U29.11 (S1)
- net ID_REG_SEL_1: now also J12.13 (Pin_13)
- net ID_REG_SEL_3: now reaches U29.13 (S3)
- net ID_REG_SEL_3: now also J12.16 (Pin_16)
- net ID_REG_SEL_2: now reaches U29.14 (S2)
- net ID_REG_SEL_2: now also J12.15 (Pin_15)
- net data15: now reaches J12.2 (Pin_2)
- net data14: now reaches J12.3 (Pin_3)
- net data13: now reaches J12.4 (Pin_4)
- net data12: now reaches J12.5 (Pin_5)
- net data11: now reaches J12.6 (Pin_6)
- net data10: now reaches J12.7 (Pin_7)
- net data9: now reaches J12.8 (Pin_8)
- net data8: now reaches J12.9 (Pin_9)
- net data_3_1 renamed data0
- net data_3_2 renamed data1
- net data_3_3 renamed data2
- net data_3_4 renamed data3
- net data_3_5 renamed data4
- net data_3_6 renamed data5
- net data_3_7 renamed data6
- net data_3_8 renamed data7
- new net IO0: J14.10 (Pin_10)
- new net IO1: J14.9 (Pin_9)
- new net IO10: J14.14 (Pin_14)
- new net IO11: J14.15 (Pin_15)
- new net IO12: J14.16 (Pin_16)
- new net IO13: J14.17 (Pin_17)
- new net IO14: J14.18 (Pin_18)
- new net IO15: J14.20 (Pin_20)
- new net IO2: J14.8 (Pin_8)
- new net IO3: J14.6 (Pin_6)
- new net IO4: J14.5 (Pin_5)
- new net IO5: J14.3 (Pin_3)
- new net IO6: J14.2 (Pin_2)
- new net IO7: J14.1 (Pin_1)
- new net IO8: J14.12 (Pin_12)
- new net IO9: J14.13 (Pin_13)
- no-connect marks 26 -> 4
Other:
- note removed: "int"
- note removed: "int_id"
- moved on the sheet: J12
