File: PCB/Kicad/reg/reg.kicad_sch (KiCad schematic)
At the start: 41 parts, among them J12 Conn_02x10_Counter_Clockwise, J13 Conn_02x10_Counter_Clockwise, J14 Conn_02x10_Counter_Clockwise, U1 74LS10, U17 74AHC04, U29 CD74HC4067M, U30 CD74HC4067M, U85 74148

Commit message: unify schematic
Parts:
- removed C83, C84: C_Polarized, Capacitor_SMD:C_0402_1005Metric, symbol Device:C_Polarized
- removed J12, J13, J14: Conn_02x10_Counter_Clockwise, Connector_PinHeader_2.54mm:PinHeader_2x10_P2.54mm_Horizontal, symbol Connector_Generic:Conn_02x10_Counter_Clockwise
- removed U1: 74LS10, Package_DIP:DIP-14_W7.62mm_SMDSocket_SmallPads, symbol 74xx:74LS10
- added C1, C10, C7, C8, C9: 100nF, Capacitor_SMD:C_0402_1005Metric, symbol Device:C
- added D1: green, Diode_SMD:D_0603_1608Metric, symbol Device:LED
- added Dd1, Dd2, Dd3, Dd4, Dd5, Dd6, Dd7: yellow, LED_SMD:LED_0603_1608Metric, symbol Device:LED
- added H1, H2, H3, H4: MountingHole_Pad, MountingHole:MountingHole_2.2mm_M2_DIN965_Pad, symbol Mechanical:MountingHole_Pad
- added J4, J5, J6: Conn_02x10_Odd_Even, Connector_PinHeader_2.54mm:PinHeader_2x10_P2.54mm_Horizontal, symbol Connector_Generic:Conn_02x10_Odd_Even
- added R1, Rd1, Rd2, Rd3, Rd4, Rd5, Rd6, Rd7: 680, Resistor_SMD:R_0402_1005Metric, symbol Device:R
- added U4: 7400, Package_SO:SO-14_3.9x8.65mm_P1.27mm, symbol 74xx:74HC00
- R1288, R1289, R1290, R1291, R1292, R1293, R1294, R1295, R1296, R1297, R1298, R1299, R1300, R1301, R1302, R1303, R1304, R1305, R1306, R1307, R1308, R1309, R1310, R1311, R1312, R1313, R1314, R1315, R1316, R1317, R1318: value 620 -> 10k; footprint Resistor_SMD:R_0402_1005Metric_Pad0.72x0.64mm_HandSolder -> Resistor_SMD:R_0402_1005Metric
- U17: value 74AHC04 -> 7404; footprint Package_DIP:DIP-14_W7.62mm_SMDSocket_SmallPads -> Package_SO:SO-14_3.9x8.65mm_P1.27mm
- U29, U30: value CD74HC4067M -> 744067; footprint Package_SO:SOIC-24W_7.5x15.4mm_P1.27mm -> Package_SO:TSSOP-24_4.4x7.8mm_P0.65mm
- U85: footprint Package_DIP:DIP-16_W7.62mm_SMDSocket_SmallPads -> Package_SO:SOIC-16_3.9x9.9mm_P1.27mm
Connections:
- net +5V: now also U17.5, C1.1, C10.1, C7.1, C8.1, C9.1, D1.2 (A), J5.1 (Pin_1), J5.19 (Pin_19), J6.1 (Pin_1), J6.19 (Pin_19), U4.14 (VCC)
- net 16 bit register17/nWE: now also U4.8
- net GND: now also C1.2, C10.2, C7.2, C8.2, C9.2, H1.1, H2.1, H3.1, H4.1, J4.13 (Pin_13), J4.14 (Pin_14), J4.7 (Pin_7), J4.8 (Pin_8), J5.14 (Pin_14), J5.2 (Pin_2), J5.20 (Pin_20), J5.8 (Pin_8), J6.14 (Pin_14), J6.2 (Pin_2), J6.20 (Pin_20), J6.8 (Pin_8), R1.2, Rd1.2, Rd2.2, Rd3.2, Rd4.2, Rd5.2, Rd6.2, Rd7.2, U4.7 (GND)
- net ID_REG_SEL_0: now also Dd6.2 (A), J6.4 (Pin_4)
- net ID_REG_SEL_1: now also Dd5.2 (A), J6.6 (Pin_6)
- net ID_REG_SEL_2: now also Dd4.2 (A), J6.10 (Pin_10)
- net ID_REG_SEL_3: now also Dd3.2 (A), J6.12 (Pin_12)
- net INT: now also J5.10 (Pin_10)
- net IO0: now also J4.1 (Pin_1)
- net IO1: now also J4.3 (Pin_3)
- net IO10: now also J4.6 (Pin_6)
- net IO11: now also J4.10 (Pin_10)
- net IO12: now also J4.12 (Pin_12)
- net IO13: now also J4.16 (Pin_16)
- net IO14: now also J4.18 (Pin_18)
- net IO15: now also J4.20 (Pin_20)
- net IO2: now also J4.5 (Pin_5)
- net IO3: now also J4.9 (Pin_9)
- net IO4: now also J4.11 (Pin_11)
- net IO5: now also J4.15 (Pin_15)
- net IO6: now also J4.17 (Pin_17)
- net IO7: now also J4.19 (Pin_19)
- net IO8: now also J4.2 (Pin_2)
- net IO9: now also J4.4 (Pin_4)
- net Interupt_ID_0: now also J5.12 (Pin_12)
- net Interupt_ID_1: now also J5.16 (Pin_16)
- net Interupt_ID_2: now also J5.18 (Pin_18)
- net clk: now also J6.18 (Pin_18)
- net data0: now also J5.3 (Pin_3)
- net data1: now also J5.5 (Pin_5)
- net data10: now also J6.7 (Pin_7)
- net data11: now also J6.9 (Pin_9)
- net data12: now also J6.11 (Pin_11)
- net data13: now also J6.13 (Pin_13)
- net data14: now also J6.15 (Pin_15)
- net data15: now also J6.17 (Pin_17)
- net data2: now also J5.7 (Pin_7)
- net data3: now also J5.9 (Pin_9)
- net data4: now also J5.11 (Pin_11)
- net data5: now also J5.13 (Pin_13)
- net data6: now also J5.15 (Pin_15)
- net data7: now also J5.17 (Pin_17)
- net data8: now also J6.3 (Pin_3)
- net data9: now also J6.5 (Pin_5)
- net mask_restore: now also Dd2.2 (A), J5.4 (Pin_4), U4.2
- net mask_save: now also Dd1.2 (A), J5.6 (Pin_6), U4.1
- net r1we: now also U4.12, U4.13; no longer U17.5
- net write_enable: now also Dd7.2 (A), J6.16 (Pin_16)
- new net: Dd3.1 (K), Rd3.1
- new net: Dd5.1 (K), Rd5.1
- new net: D1.1 (K), R1.1
- new net: U4.3, U4.4, U4.5
- new net: U4.10, U4.6
- new net: U4.11, U4.9
- new net: Dd6.1 (K), Rd6.1
- new net: Dd2.1 (K), Rd2.1
- new net: Dd4.1 (K), Rd4.1
- new net: Dd1.1 (K), Rd1.1
- new net: Dd7.1 (K), Rd7.1
- no-connect marks 4 -> 3
Other:
- sheet octal_and renamed octal_nand
- note added: "power LED"
- moved on the sheet: U17C, U17G
