File: PCB/Kicad/reg/rejest_16_bitowy.kicad_sch (KiCad schematic)
At the start: 4 parts, among them U10 74HCT574, U9 74HCT574

Commit message: samll fix and new problems
Connections:
- net OUT15: now reaches U10.12 (Q7)
- net OUT14: now reaches U10.13 (Q6)
- net OUT13: now reaches U10.14 (Q5)
- net OUT12: now reaches U10.15 (Q4)
- net OUT11: now reaches U10.16 (Q3)
- net OUT10: now reaches U10.17 (Q2)
- net OUT9: now reaches U10.18 (Q1)
- net OUT8: now reaches U10.19 (Q0)
- net IN_1_8: now reaches U10.2 (D0)
- net IN_1_9: now reaches U10.3 (D1)
- net IN_1_11: now reaches U10.5 (D3)
- net IN_1_12: now reaches U10.6 (D4)
- net IN_1_13: now reaches U10.7 (D5)
- net IN_1_14: now reaches U10.8 (D6)
- net IN_1_15: now reaches U10.9 (D7)
- net in_0 renamed IN_1_0
- net in_1 renamed IN_1_1
- net in_10 renamed IN_1_10
- net in_2 renamed IN_1_2
- net in_3 renamed IN_1_3
- net in_4 renamed IN_1_4
- net in_5 renamed IN_1_5
- net in_6 renamed IN_1_6
- net in_7 renamed IN_1_7
- net out_0 renamed OUT0
- net out_1 renamed OUT1
- net out_2 renamed OUT2
- net out_3 renamed OUT3
- net out_4 renamed OUT4
- net out_5 renamed OUT5
- net out_6 renamed OUT6
- net out_7 renamed OUT7
Other:
- moved on the sheet: U10

Commit message: everything_works
Connections:
- net +5V renamed VCC
- net 0 renamed GND

Commit message: capacitor
Parts:
- C3, C4: footprint Capacitor_SMD:CP_Elec_4x3 -> Capacitor_SMD:C_0402_1005Metric
Changed lines of the file:
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@@
 			)
 		)
-		(property "Footprint" "Capacitor_SMD:CP_Elec_4x3"
+		(property "Footprint" "Capacitor_SMD:C_0402_1005Metric"
 			(at 55.5752 29.21 0)
 			(effects
@@
 			)
 		)
-		(property "Footprint" "Capacitor_SMD:CP_Elec_4x3"
+		(property "Footprint" "Capacitor_SMD:C_0402_1005Metric"
 			(at 75.8952 29.21 0)
 			(effects

Commit message: fix
Parts:
- removed U10, U9: 74HCT574, Package_DIP:DIP-20_W7.62mm_SMDSocket_SmallPads, symbol 74xx:74HCT574
- added U13, U19: 74AHCT374, Package_DIP:DIP-20_W7.62mm_SMDSocket_SmallPads, symbol 74xx:74AHCT374
Connections:
- net GND: now also U13.10 (GND), U19.10 (GND)
- net IN_1_0: now also U13.3 (D0)
- net IN_1_1: now also U13.4 (D1)
- net IN_1_10: now also U19.7 (D2)
- net IN_1_11: now also U19.8 (D3)
- net IN_1_12: now also U19.13 (D4)
- net IN_1_13: now also U19.14 (D5)
- net IN_1_14: now also U19.17 (D6)
- net IN_1_15: now also U19.18 (D7)
- net IN_1_2: now also U13.7 (D2)
- net IN_1_3: now also U13.8 (D3)
- net IN_1_4: now also U13.13 (D4)
- net IN_1_5: now also U13.14 (D5)
- net IN_1_6: now also U13.17 (D6)
- net IN_1_7: now also U13.18 (D7)
- net IN_1_8: now also U19.3 (D0)
- net IN_1_9: now also U19.4 (D1)
- net OUT0: now also U13.2 (O0)
- net OUT1: now also U13.5 (O1)
- net OUT10: now also U19.6 (O2)
- net OUT11: now also U19.9 (O3)
- net OUT12: now also U19.12 (O4)
- net OUT13: now also U19.15 (O5)
- net OUT14: now also U19.16 (O6)
- net OUT15: now also U19.19 (O7)
- net OUT2: now also U13.6 (O2)
- net OUT3: now also U13.9 (O3)
- net OUT4: now also U13.12 (O4)
- net OUT5: now also U13.15 (O5)
- net OUT6: now also U13.16 (O6)
- net OUT7: now also U13.19 (O7)
- net OUT8: now also U19.2 (O0)
- net OUT9: now also U19.5 (O1)
- net clk: now also U13.11 (Cp), U19.11 (Cp)
- net nWE: now also U13.1 (OE), U19.1 (OE)
- net VCC renamed +5V
- net +5V: now also U13.20 (VCC), U19.20 (VCC)

Commit message: aaaaaaaaaaaaaaaaaaaaaaaaaaaaaaaaaaaaaaaaaaaa
Parts:
- added D705, D706, D707, D708, D709, D710, D711, D712, D713, D714, D715, D716, D717, D718, D719, D720, D721, D722, D723, D724, D725, D726, D727, D728, D729, D730, D731, D732, D733, D734, D735, D736: LED, LED_SMD:LED_0603_1608Metric_Pad1.05x0.95mm_HandSolder, symbol Device:LED
- added R705, R706, R707, R708, R709, R710, R711, R712, R713, R714, R715, R716, R717, R718, R719, R720, R721, R722, R723, R724, R725, R726, R727, R728, R729, R730, R731, R732, R733, R734, R735, R736: 620, Resistor_SMD:R_0402_1005Metric_Pad0.72x0.64mm_HandSolder, symbol Device:R
Connections:
- net GND: now also R705.2, R706.2, R707.2, R708.2, R709.2, R710.2, R711.2, R712.2, R713.2, R714.2, R715.2, R716.2, R717.2, R718.2, R719.2, R720.2, R721.2, R722.2, R723.2, R724.2, R725.2, R726.2, R727.2, R728.2, R729.2, R730.2, R731.2, R732.2, R733.2, R734.2, R735.2, R736.2
- net IN_1_0: now also D706.2 (A)
- net IN_1_1: now also D708.2 (A)
- net IN_1_10: now also D726.2 (A)
- net IN_1_11: now also D728.2 (A)
- net IN_1_12: now also D730.2 (A)
- net IN_1_13: now also D732.2 (A)
- net IN_1_14: now also D734.2 (A)
- net IN_1_15: now also D736.2 (A)
- net IN_1_2: now also D710.2 (A)
- net IN_1_3: now also D712.2 (A)
- net IN_1_4: now also D714.2 (A)
- net IN_1_5: now also D716.2 (A)
- net IN_1_6: now also D718.2 (A)
- net IN_1_7: now also D720.2 (A)
- net IN_1_8: now also D722.2 (A)
- net IN_1_9: now also D724.2 (A)
- net OUT0: now also D705.2 (A)
- net OUT1: now also D707.2 (A)
- net OUT10: now also D725.2 (A)
- net OUT11: now also D727.2 (A)
- net OUT12: now also D729.2 (A)
- net OUT13: now also D731.2 (A)
- net OUT14: now also D733.2 (A)
- net OUT15: now also D735.2 (A)
- net OUT2: now also D709.2 (A)
- net OUT3: now also D711.2 (A)
- net OUT4: now also D713.2 (A)
- net OUT5: now also D715.2 (A)
- net OUT6: now also D717.2 (A)
- net OUT7: now also D719.2 (A)
- net OUT8: now also D721.2 (A)
- net OUT9: now also D723.2 (A)
- new net: D727.1 (K), R727.1
- new net: D705.1 (K), R705.1
- new net: D734.1 (K), R734.1
- new net: D720.1 (K), R720.1
- new net: D733.1 (K), R733.1
- new net: D713.1 (K), R713.1
- new net: D729.1 (K), R729.1
- new net: D716.1 (K), R716.1
- new net: D728.1 (K), R728.1
- new net: D717.1 (K), R717.1
- new net: D722.1 (K), R722.1
- new net: D731.1 (K), R731.1
- new net: D706.1 (K), R706.1
- new net: D715.1 (K), R715.1
- new net: D719.1 (K), R719.1
- new net: D710.1 (K), R710.1
- new net: D732.1 (K), R732.1
- new net: D725.1 (K), R725.1
- new net: D735.1 (K), R735.1
- new net: D726.1 (K), R726.1
- new net: D712.1 (K), R712.1
- new net: D724.1 (K), R724.1
- new net: D709.1 (K), R709.1
- new net: D714.1 (K), R714.1
- new net: D708.1 (K), R708.1
- new net: D730.1 (K), R730.1
- new net: D736.1 (K), R736.1
- new net: D718.1 (K), R718.1
- new net: D711.1 (K), R711.1
- new net: D707.1 (K), R707.1
- new net: D721.1 (K), R721.1
- new net: D723.1 (K), R723.1

Commit message: bombardino crocodilo
Parts:
- added D1271: LED, LED_SMD:LED_0603_1608Metric_Pad1.05x0.95mm_HandSolder, symbol Device:LED
- added R1271: 620, Resistor_SMD:R_0402_1005Metric_Pad0.72x0.64mm_HandSolder, symbol Device:R
Connections:
- net +5V: now also D1271.2 (A)
- net GND: now also R1271.2
- new net: D1271.1 (K), R1271.1

Commit message: unify schematic
Parts:
- removed C3, C4: C_Polarized, Capacitor_SMD:C_0402_1005Metric, symbol Device:C_Polarized
- removed D1271: LED, LED_SMD:LED_0603_1608Metric_Pad1.05x0.95mm_HandSolder, symbol Device:LED
- removed R1271: 620, Resistor_SMD:R_0402_1005Metric_Pad0.72x0.64mm_HandSolder, symbol Device:R
- removed U13, U19: 74AHCT374, Package_DIP:DIP-20_W7.62mm_SMDSocket_SmallPads, symbol 74xx:74AHCT374
- added C15, C3: 100nF, Capacitor_SMD:C_0402_1005Metric, symbol Device:C
- added U1, U19: 74377, Package_SO:SSOP-20_5.3x7.2mm_P0.65mm, symbol 74xx:74LS377
- D705, D706, D707, D708, D709, D710, D711, D712, D713, D714, D715, D716, D717, D718, D719, D720, D721, D722, D723, D724, D725, D726, D727, D728, D729, D730, D731, D732, D733, D734, D735, D736: value LED -> red; footprint LED_SMD:LED_0603_1608Metric_Pad1.05x0.95mm_HandSolder -> LED_SMD:LED_0603_1608Metric
- R705, R706, R707, R708, R709, R710, R711, R712, R713, R714, R715, R716, R717, R718, R719, R720, R721, R722, R723, R724, R725, R726, R727, R728, R729, R730, R731, R732, R733, R734, R735, R736: value 620 -> 680; footprint Resistor_SMD:R_0402_1005Metric_Pad0.72x0.64mm_HandSolder -> Resistor_SMD:R_0402_1005Metric
Connections:
- net +5V: now also U1.20 (VCC), U19.20 (VCC)
- net GND: now also C15.2, C3.2, U1.10 (GND), U19.10 (GND)
- net IN_1_0: now also U1.3 (D0)
- net IN_1_1: now also U1.4 (D1)
- net IN_1_10: now also U19.7 (D2)
- net IN_1_11: now also U19.8 (D3)
- net IN_1_12: now also U19.13 (D4)
- net IN_1_13: now also U19.14 (D5)
- net IN_1_14: now also U19.17 (D6)
- net IN_1_15: now also U19.18 (D7)
- net IN_1_2: now also U1.7 (D2)
- net IN_1_3: now also U1.8 (D3)
- net IN_1_4: now also U1.13 (D4)
- net IN_1_5: now also U1.14 (D5)
- net IN_1_6: now also U1.17 (D6)
- net IN_1_7: now also U1.18 (D7)
- net IN_1_8: now also U19.3 (D0)
- net IN_1_9: now also U19.4 (D1)
- net OUT0: now also U1.2 (Q0)
- net OUT1: now also U1.5 (Q1)
- net OUT10: now also U19.6 (Q2)
- net OUT11: now also U19.9 (Q3)
- net OUT12: now also U19.12 (Q4)
- net OUT13: now also U19.15 (Q5)
- net OUT14: now also U19.16 (Q6)
- net OUT15: now also U19.19 (Q7)
- net OUT2: now also U1.6 (Q2)
- net OUT3: now also U1.9 (Q3)
- net OUT4: now also U1.12 (Q4)
- net OUT5: now also U1.15 (Q5)
- net OUT6: now also U1.16 (Q6)
- net OUT7: now also U1.19 (Q7)
- net OUT8: now also U19.2 (Q0)
- net OUT9: now also U19.5 (Q1)
- net clk: now also U1.11 (CP), U19.11 (CP)
- net nWE: now also U1.1 (~{E}), U19.1 (~{E})
- new net VCC: C15.1, C3.1
