File: PCB/Kicad/reg/octal_and.kicad_sch (KiCad schematic)
At the start: 2 parts, among them U89 74LS08, U90 74LS08

Commit message: everything_works
Parts:
- added C87, C88: C_Polarized, Capacitor_SMD:CP_Elec_4x3, symbol Device:C_Polarized
Connections:
- net +5V renamed VCC
- net VCC: now also C87.1, C88.1
- net 0 renamed GND
- net GND: now also C87.2, C88.2
Changed lines of the file:
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@@
 	(paper "A4")
 	(junction
-		(at 46.99 22.86)
+		(at 55.88 48.26)
 		(diameter 0)
 		(color 0 0 0 0)
 	)
 	(junction
-		(at 45.72 48.26)
+		(at 57.15 22.86)
 		(diameter 0)
 		(color 0 0 0 0)
 	)
-	(wire
-		(pts
-			(xy 36.83 48.26) (xy 45.72 48.26)
+	(junction
+		(at 78.74 22.86)
+		(diameter 0)
+		(color 0 0 0 0)
+	)
+	(junction
+		(at 85.09 33.02)
+		(diameter 0)
+		(color 0 0 0 0)
+	)
+	(wire
+		(pts
+			(xy 36.83 48.26) (xy 55.88 48.26)
+		)
+		(stroke
+			(width 0)
+			(type default)
+		)
+	)
+	(wire
+		(pts
+			(xy 85.09 33.02) (xy 99.06 33.02)
 		)
 		(stroke
@@
 	(wire
 		(pts
-			(xy 45.72 48.26) (xy 57.15 48.26)
+			(xy 85.09 33.02) (xy 85.09 49.53)
 		)
 		(stroke
@@
 	(wire
 		(pts
+			(xy 78.74 33.02) (xy 85.09 33.02)
+		)
+		(stroke
+			(width 0)
+			(type default)
+		)
+	)
+	(wire
+		(pts
 			(xy 149.86 31.75) (xy 149.86 35.56)
 		)
@@
 	(wire
 		(pts
+			(xy 99.06 25.4) (xy 99.06 22.86)
+		)
+		(stroke
+			(width 0)
+			(type default)
+		)
+	)
+	(wire
+		(pts
 			(xy 144.78 31.75) (xy 144.78 35.56)
 		)
@@
 	(wire
 		(pts
+			(xy 55.88 48.26) (xy 57.15 48.26)
+		)
+		(stroke
+			(width 0)
+			(type default)
+		)
+	)
+	(wire
+		(pts
+			(xy 78.74 22.86) (xy 99.06 22.86)
+		)
+		(stroke
+			(width 0)
+			(type default)
+		)
+	)
+	(wire
+		(pts
 			(xy 97.79 60.96) (xy 97.79 66.04)
 		)
@@
 	(wire
 		(pts
+			(xy 55.88 48.26) (xy 55.88 49.53)
+		)
+		(stroke
+			(width 0)
+			(type default)
+		)
+	)
+	(wire
+		(pts
 			(xy 147.32 55.88) (xy 147.32 50.8)
 		)
@@
 	(wire
 		(pts
+			(xy 57.15 22.86) (xy 78.74 22.86)
+		)
+		(stroke
+			(width 0)
+			(type default)
+		)
+	)
+	(wire
+		(pts
 			(xy 135.89 31.75) (xy 135.89 35.56)
 		)
@@
 	(wire
 		(pts
-			(xy 36.83 22.86) (xy 46.99 22.86)
+			(xy 78.74 22.86) (xy 78.74 25.4)
 		)
 		(stroke
@@
 	(wire
 		(pts
-			(xy 45.72 48.26) (xy 45.72 53.34)
+			(xy 85.09 49.53) (xy 55.88 49.53)
 		)
 		(stroke
@@
 	(wire
 		(pts
-			(xy 46.99 22.86) (xy 57.15 22.86)
+			(xy 36.83 22.86) (xy 57.15 22.86)
 		)
 		(stroke
@@
 		)
 	)
+	(hierarchical_label "GND"
+		(shape output)
+		(at 50.8 48.26 270)
+		(effects
+			(font
+				(size 1.27 1.27)
+			)
+			(justify right)
+		)
+	)
 	(hierarchical_label "in_8"
 		(shape input)
@@
 		(shape input)
 		(at 149.86 31.75 90)
+		(effects
+			(font
+				(size 1.27 1.27)
+			)
+			(justify left)
+		)
+	)
+	(hierarchical_label "VCC"
+		(shape input)
+		(at 52.07 22.86 90)
 		(effects
 			(font
@@
 			)
 			(justify left)
+		)
+	)
+	(symbol
+		(lib_id "Device:C_Polarized")
+		(at 99.06 29.21 0)
+		(unit 1)
+		(exclude_from_sim no)
+		(in_bom yes)
+		(on_board yes)
+		(dnp no)
+		(fields_autoplaced yes)
+		(property "Reference" "C88"
+			(at 102.87 27.0509 0)
+			(effects
+				(font
+					(size 1.27 1.27)
+				)
+				(justify left)
+			)
+		)
+		(property "Value" "C_Polarized"
+			(at 102.87 29.5909 0)
+			(effects
+				(font
+					(size 1.27 1.27)
+				)
+				(justify left)
+			)
+		)
+		(property "Footprint" "Capacitor_SMD:CP_Elec_4x3"
+			(at 100.0252 33.02 0)
+			(effects
+				(font
+					(size 1.27 1.27)
+				)
+				(hide yes)
+			)
+		)
+		(property "Datasheet" "~"
+			(at 99.06 29.21 0)
+			(effects
+				(font
+					(size 1.27 1.27)
+				)
+				(hide yes)
+			)
+		)
+		(property "Description" "Polarized capacitor"
+			(at 99.06 29.21 0)
+			(effects
+				(font
+					(size 1.27 1.27)
+				)
+				(hide yes)
+			)
+		)
+		(pin "1"
+		)
+		(pin "2"
+		)
+		(instances
+			(project "reg"
+				(path "/e5ea2144-296a-4524-8c5b-c3f6342ff44f/131ca02f-eb01-47a4-a14c-0da3c0e51fc2"
+					(reference "C88")
+					(unit 1)
+				)
+			)
 		)
 	)
@@
 	)
 	(symbol
-		(lib_id "Simulation_SPICE:0")
-		(at 45.72 53.34 0)
-		(unit 1)
-		(exclude_from_sim no)
-		(in_bom yes)
-		(on_board yes)
-		(dnp no)
-		(property "Reference" "#GND0125"
-			(at 45.72 58.42 0)
-			(effects
-				(font
-					(size 1.27 1.27)
-				)
-				(hide yes)
-			)
-		)
-		(property "Value" "0"
-			(at 48.514 51.562 0)
-			(effects
-				(font
-					(size 1.27 1.27)
-				)
-			)
-		)
-		(property "Footprint" ""
-			(at 45.72 53.34 0)
-			(effects
-				(font
-					(size 1.27 1.27)
-				)
-				(hide yes)
-			)
-		)
-		(property "Datasheet" "https://ngspice.sourceforge.io/docs/ngspice-html-manual/manual.xhtml#subsec_Circuit_elements__device"
-			(at 45.72 63.5 0)
-			(effects
-				(font
-					(size 1.27 1.27)
-				)
-				(hide yes)
-			)
-		)
-		(property "Description" "0V reference potential for simulation"
-			(at 45.72 60.96 0)
-			(effects
-				(font
-					(size 1.27 1.27)
-				)
-				(hide yes)
-			)
-		)
-		(pin "1"
-		)
-		(instances
-			(project ""
-				(path "/e5ea2144-296a-4524-8c5b-c3f6342ff44f/131ca02f-eb01-47a4-a14c-0da3c0e51fc2"
-					(reference "#GND0125")
-					(unit 1)
-				)
-			)
-		)
-	)
-	(symbol
 		(lib_id "74xx:74LS08")
 		(at 133.35 43.18 270)
@@
 	)
 	(symbol
-		(lib_id "power:+1V35")
-		(at 46.99 22.86 0)
+		(lib_id "Device:C_Polarized")
+		(at 78.74 29.21 0)
 		(unit 1)
 		(exclude_from_sim no)
@@
 		(dnp no)
 		(fields_autoplaced yes)
-		(property "Reference" "#PWR0125"
-			(at 46.99 26.67 0)
-			(effects
-				(font
-					(size 1.27 1.27)
-				)
-				(hide yes)
-			)
-		)
-		(property "Value" "+5V"
-			(at 46.99 17.78 0)
-			(effects
-				(font
-					(size 1.27 1.27)
-				)
-			)
-		)
-		(property "Footprint" ""
-			(at 46.99 22.86 0)
-			(effects
-				(font
-					(size 1.27 1.27)
-				)
-				(hide yes)
-			)
-		)
-		(property "Datasheet" ""
-			(at 46.99 22.86 0)
-			(effects
-				(font
-					(size 1.27 1.27)
-				)
-				(hide yes)
-			)
-		)
-		(property "Description" "Power symbol creates a global label with name \"+1V35\""
-			(at 46.99 22.86 0)
+		(property "Reference" "C87"
+			(at 82.55 27.0509 0)
+			(effects
+				(font
+					(size 1.27 1.27)
+				)
+				(justify left)
+			)
+		)
+		(property "Value" "C_Polarized"
+			(at 82.55 29.5909 0)
+			(effects
+				(font
+					(size 1.27 1.27)
+				)
+				(justify left)
+			)
+		)
+		(property "Footprint" "Capacitor_SMD:CP_Elec_4x3"
+			(at 79.7052 33.02 0)
+			(effects
+				(font
+					(size 1.27 1.27)
+				)
+				(hide yes)
+			)
+		)
+		(property "Datasheet" "~"
+			(at 78.74 29.21 0)
+			(effects
+				(font
+					(size 1.27 1.27)
+				)
+				(hide yes)
+			)
+		)
+		(property "Description" "Polarized capacitor"
+			(at 78.74 29.21 0)
 			(effects
 				(font
@@
 		(pin "1"
 		)
+		(pin "2"
+		)
 		(instances
-			(project ""
+			(project "reg"
 				(path "/e5ea2144-296a-4524-8c5b-c3f6342ff44f/131ca02f-eb01-47a4-a14c-0da3c0e51fc2"
-					(reference "#PWR0125")
+					(reference "C87")
 					(unit 1)
 				)

Commit message: capacitor
Parts:
- C87, C88: footprint Capacitor_SMD:CP_Elec_4x3 -> Capacitor_SMD:C_0402_1005Metric
Changed lines of the file:
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@@
 			)
 		)
-		(property "Footprint" "Capacitor_SMD:CP_Elec_4x3"
+		(property "Footprint" "Capacitor_SMD:C_0402_1005Metric"
 			(at 100.0252 33.02 0)
 			(effects
@@
 			)
 		)
-		(property "Footprint" "Capacitor_SMD:CP_Elec_4x3"
+		(property "Footprint" "Capacitor_SMD:C_0402_1005Metric"
 			(at 79.7052 33.02 0)
 			(effects

Commit message: fix
Connections:
- net VCC renamed +5V

Commit message: aaaaaaaaaaaaaaaaaaaaaaaaaaaaaaaaaaaaaaaaaaaa
Parts:
- removed U89: 74LS08, Package_DIP:DIP-14_W7.62mm_SMDSocket_SmallPads, symbol 74xx:74LS08
- removed U90: 74LS08, Package_DIP:DIP-20_W7.62mm_SMDSocket_SmallPads, symbol 74xx:74LS08
- added U2, U3: 74HC00, Package_DIP:DIP-14_W7.62mm_SMDSocket_SmallPads, symbol 74xx:74HC00
Connections:
- net +5V: now also U2.14 (VCC), U3.14 (VCC)
- net GND: now also U2.7 (GND), U3.7 (GND)
- net in_0: now also U2.12
- net in_1: now also U2.13
- net in_10: now also U3.9
- net in_11: now also U3.10
- net in_12: now also U3.4
- net in_13: now also U3.5
- net in_14: now also U3.1
- net in_15: now also U3.2
- net in_2: now also U2.9
- net in_3: now also U2.10
- net in_4: now also U2.4
- net in_5: now also U2.5
- net in_6: now also U2.1
- net in_7: now also U2.2
- net in_8: now also U3.12
- net in_9: now also U3.13
- net out_0: now also U2.11
- net out_1: now also U2.8
- net out_2: now also U2.6
- net out_3: now also U2.3
- net out_4: now also U3.11
- net out_5: now also U3.8
- net out_6: now also U3.6
- net out_7: now also U3.3

Commit message: unify schematic
Parts:
- removed C87, C88: C_Polarized, Capacitor_SMD:C_0402_1005Metric, symbol Device:C_Polarized
- added C13, C14: 100nF, Capacitor_SMD:C_0402_1005Metric, symbol Device:C
- U2, U3: value 74HC00 -> 7400; footprint Package_DIP:DIP-14_W7.62mm_SMDSocket_SmallPads -> Package_SO:SO-14_3.9x8.65mm_P1.27mm
Connections:
- net GND: now also C13.2, C14.2
- new net VCC: C13.1, C14.1
Other:
- moved on the sheet: U2E, U3E

Commit message: layout_1
Other:
- company: (none) -> AGH Logic Unit
Changed lines of the file:
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@@
 	(generator_version "10.0")
 	(paper "A4")
+	(title_block
+		(company "AGH Logic Unit")
+		(comment 1 "author: Jan Pieprzycki")
+	)
 	(wire
 		(pts
