File: PCB/Kicad/reg/running_and_8b.kicad_sch (KiCad schematic)
At the start: 4 parts, among them U91 74LS08, U92 74LS08

Commit message: capacitor
Parts:
- C85, C86: footprint Capacitor_SMD:CP_Elec_4x3 -> Capacitor_SMD:C_0402_1005Metric
Changed lines of the file:
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@@
 			)
 		)
-		(property "Footprint" "Capacitor_SMD:CP_Elec_4x3"
+		(property "Footprint" "Capacitor_SMD:C_0402_1005Metric"
 			(at 113.9952 39.37 0)
 			(effects
@@
 			)
 		)
-		(property "Footprint" "Capacitor_SMD:CP_Elec_4x3"
+		(property "Footprint" "Capacitor_SMD:C_0402_1005Metric"
 			(at 93.6752 39.37 0)
 			(effects

Commit message: fix
Connections:
- net VCC is gone; now on net +5V: C85.1, C86.1, U91.14 (VCC), U92.14 (VCC)
- net +5V: now reaches U92.12
- net +5V: now also U92.13
- no-connect marks 3 -> 1
Other:
- moved on the sheet: U92D

Commit message: unify schematic
Parts:
- removed C85, C86: C_Polarized, Capacitor_SMD:C_0402_1005Metric, symbol Device:C_Polarized
- U91: value 74LS08 -> 7408; footprint Package_DIP:DIP-14_W7.62mm_SMDSocket_SmallPads -> Package_SO:SO-14_3.9x8.65mm_P1.27mm
- U92: value 74LS08 -> 7408; footprint Package_DIP:DIP-20_W7.62mm_SMDSocket_SmallPads -> Package_SO:SO-14_3.9x8.65mm_P1.27mm
Other:
- moved on the sheet: U91E, U92E

Commit message: layout_1
Other:
- company: (none) -> AGH Logic Unit
Changed lines of the file:
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@@
 	(generator_version "10.0")
 	(paper "A4")
+	(title_block
+		(company "AGH Logic Unit")
+		(comment 1 "author: Jan Pieprzycki")
+	)
 	(junction
 		(at 140.97 144.78)
