File: PCB/Kicad/reg/untitled.kicad_sch (KiCad schematic)
At the start: 4 parts, among them U7 74HC245, U8 74HC245

Commit message: capacitor
Parts:
- C1, C2: footprint Capacitor_SMD:CP_Elec_4x3 -> Capacitor_SMD:C_0402_1005Metric
Changed lines of the file:
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@@
 			)
 		)
-		(property "Footprint" "Capacitor_SMD:CP_Elec_4x3"
+		(property "Footprint" "Capacitor_SMD:C_0402_1005Metric"
 			(at 150.8252 36.83 0)
 			(effects
@@
 			)
 		)
-		(property "Footprint" "Capacitor_SMD:CP_Elec_4x3"
+		(property "Footprint" "Capacitor_SMD:C_0402_1005Metric"
 			(at 130.5052 36.83 0)
 			(effects

Commit message: fix
Connections:
- net VCC renamed +5V

Commit message: aaaaaaaaaaaaaaaaaaaaaaaaaaaaaaaaaaaaaaaaaaaa
Parts:
- added D1, D111, D133, D155, D177, D199, D221, D23, D243, D265, D287, D309, D331, D353, D375, D397, D419, D441, D45, D463, D485, D507, D529, D551, D573, D595, D617, D639, D661, D67, D683, D89: LED, LED_SMD:LED_0603_1608Metric_Pad1.05x0.95mm_HandSolder, symbol Device:LED
- added R1, R111, R133, R155, R177, R199, R221, R23, R243, R265, R287, R309, R331, R353, R375, R397, R419, R441, R45, R463, R485, R507, R529, R551, R573, R595, R617, R639, R661, R67, R683, R89: 620, Resistor_SMD:R_0402_1005Metric_Pad0.72x0.64mm_HandSolder, symbol Device:R
Connections:
- net nE1 is gone; now on net +5V: U7.1 (A->B), U8.1 (A->B)
- net GND: now also R1.2, R111.2, R133.2, R155.2, R177.2, R199.2, R221.2, R23.2, R243.2, R265.2, R287.2, R309.2, R331.2, R353.2, R375.2, R397.2, R419.2, R441.2, R45.2, R463.2, R485.2, R507.2, R529.2, R551.2, R573.2, R595.2, R617.2, R639.2, R661.2, R67.2, R683.2, R89.2
- net IN_1_0: now also D1.2 (A)
- net IN_1_1: now also D23.2 (A)
- net IN_1_10: now also D221.2 (A)
- net IN_1_11: now also D243.2 (A)
- net IN_1_12: now also D265.2 (A)
- net IN_1_13: now also D287.2 (A)
- net IN_1_14: now also D309.2 (A)
- net IN_1_15: now also D331.2 (A)
- net IN_1_2: now also D45.2 (A)
- net IN_1_3: now also D67.2 (A)
- net IN_1_4: now also D89.2 (A)
- net IN_1_5: now also D111.2 (A)
- net IN_1_6: now also D133.2 (A)
- net IN_1_7: now also D155.2 (A)
- net IN_1_8: now also D177.2 (A)
- net IN_1_9: now also D199.2 (A)
- net OUT0: now also D353.2 (A)
- net OUT1: now also D375.2 (A)
- net OUT10: now also D573.2 (A)
- net OUT11: now also D595.2 (A)
- net OUT12: now also D617.2 (A)
- net OUT13: now also D639.2 (A)
- net OUT14: now also D661.2 (A)
- net OUT15: now also D683.2 (A)
- net OUT2: now also D397.2 (A)
- net OUT3: now also D419.2 (A)
- net OUT4: now also D441.2 (A)
- net OUT5: now also D463.2 (A)
- net OUT6: now also D485.2 (A)
- net OUT7: now also D507.2 (A)
- net OUT8: now also D529.2 (A)
- net OUT9: now also D551.2 (A)
- new net: D375.1 (K), R375.1
- new net: D441.1 (K), R441.1
- new net: D133.1 (K), R133.1
- new net: D683.1 (K), R683.1
- new net: D463.1 (K), R463.1
- new net: D573.1 (K), R573.1
- new net: D551.1 (K), R551.1
- new net: D309.1 (K), R309.1
- new net: D199.1 (K), R199.1
- new net: D23.1 (K), R23.1
- new net: D331.1 (K), R331.1
- new net: D265.1 (K), R265.1
- new net: D397.1 (K), R397.1
- new net: D617.1 (K), R617.1
- new net: D485.1 (K), R485.1
- new net: D111.1 (K), R111.1
- new net: D353.1 (K), R353.1
- new net: D507.1 (K), R507.1
- new net: D639.1 (K), R639.1
- new net: D419.1 (K), R419.1
- new net: D155.1 (K), R155.1
- new net: D1.1 (K), R1.1
- new net: D89.1 (K), R89.1
- new net: D45.1 (K), R45.1
- new net: D661.1 (K), R661.1
- new net: D243.1 (K), R243.1
- new net: D177.1 (K), R177.1
- new net: D287.1 (K), R287.1
- new net: D221.1 (K), R221.1
- new net: D67.1 (K), R67.1
- new net: D529.1 (K), R529.1
- new net: D595.1 (K), R595.1
Other:
- moved on the sheet: C1, C2, U7, U8

Commit message: bombardino crocodilo
Parts:
- added D1249: LED, LED_SMD:LED_0603_1608Metric_Pad1.05x0.95mm_HandSolder, symbol Device:LED
- added R1249: 620, Resistor_SMD:R_0402_1005Metric_Pad0.72x0.64mm_HandSolder, symbol Device:R
Connections:
- net +5V: now also D1249.2 (A)
- net GND: now also R1249.2
- new net: D1249.1 (K), R1249.1

Commit message: unify schematic
Parts:
- removed C1, C2: C_Polarized, Capacitor_SMD:C_0402_1005Metric, symbol Device:C_Polarized
- removed D1, D111, D1249, D133, D155, D177, D199, D221, D23, D243, D265, D287, D309, D331, D353, D375, D397, D419, D441, D45, D463, D485, D507, D529, D551, D573, D595, D617, D639, D661, D67, D683, D89: LED, LED_SMD:LED_0603_1608Metric_Pad1.05x0.95mm_HandSolder, symbol Device:LED
- removed R1, R111, R1249, R133, R155, R177, R199, R221, R23, R243, R265, R287, R309, R331, R353, R375, R397, R419, R441, R45, R463, R485, R507, R529, R551, R573, R595, R617, R639, R661, R67, R683, R89: 620, Resistor_SMD:R_0402_1005Metric_Pad0.72x0.64mm_HandSolder, symbol Device:R
- added C47, C5: 100nF, Capacitor_SMD:C_0402_1005Metric, symbol Device:C
- U7, U8: value 74HC245 -> 74245; footprint Package_DIP:DIP-20_W7.62mm_SMDSocket_SmallPads -> Package_SO:TSSOP-20_4.4x6.5mm_P0.65mm
Connections:
- net GND: now also C47.2, C5.2
- new net VCC: C47.1, C5.1

Commit message: layout_1
Other:
- company: (none) -> AGH Logic Unit
Changed lines of the file:
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@@
 	(generator_version "10.0")
 	(paper "A4")
+	(title_block
+		(company "AGH Logic Unit")
+		(comment 1 "author: Jan Pieprzycki")
+	)
 	(junction
 		(at 91.44 78.74)
