File: PCB/Kicad/reg/reg.kicad_pcb (KiCad board)
At the start: 6 copper layers, 200 x 150 mm, 770 parts, among them J4 Conn_02x10_Odd_Even, J5 Conn_02x10_Odd_Even, J6 Conn_02x10_Odd_Even, U1 74377, U10 74245, U107 74245, U108 74245, U109 74245, U11 74245, U110 74245, U111 74245, U112 74245, U113 74245, U114 74245, U115 74245, U116 74245, U117 74245, U118 74245, U119 74245, U12 74245, U120 74245, U121 74245, U122 74245, U123 74245, U124 74245, U125 74245, U126 74245, U127 74245, U128 74245, U129 74245, U130 74245, U131 74245, U132 74245, U133 74245, U134 74245, U135 74245, U136 74245, U14 74377, U15 74245, U16 74245, U17 7404, U18 74377, U19 74377, U2 7400, U20 74377, U21 74245, U22 74245, U23 74377, U24 74377, U25 74377, U26 74377, U27 74377, U28 74377, U29 744067, U3 7400, U30 744067, U31 74377, U32 74377, U33 74377, U34 74377, U35 74377, U36 74377, U37 74377, U38 74377, U39 74377, U4 7400, U40 74377, U41 74377, U42 74377, U43 74377, U44 74377, U45 74377, U46 74377, U47 74377, U48 74377, U49 74377, U5 74245, U50 74377, U51 74377, U52 74377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

Commit message: layout_1
Parts:
- removed D1001, D1003, D1005, D1007, D1009, D1011, D1013, D1015, D1017, D1019, D1021, D1023, D1025, D1027, D1029, D1031, D1033, D1035, D1037, D1039, D1041, D1043, D1045, D1047, D1049, D1051, D1053, D1055, D1057, D1059, D1061, D1063, D1065, D1067, D1069, D1071, D1073, D1075, D1077, D1079, D1081, D1083, D1085, D1087, D1089, D1091, D1093, D1095, D1097, D1099, D1101, D1103, D1105, D1107, D1109, D1111, D1113, D1115, D1117, D1119, D1121, D1123, D1125, D1127, D1129, D1131, D1133, D1135, D1137, D1139, D1141, D1143, D1145, D1147, D1149, D1151, D1153, D1155, D1157, D1159, D1161, D1163, D1165, D1167, D1169, D1171, D1173, D1175, D1177, D1179, D1181, D1183, D1185, D1187, D1189, D1191, D1193, D1195, D1197, D1199, D1201, D1203, D1205, D1207, D1209, D1211, D1213, D1215, D1217, D1219, D1221, D1223, D1225, D1227, D1229, D1231, D1233, D1235, D1237, D1239, D1241, D1243, D1245, D1247, D705, D707, D709, D711, D713, D715, D717, D719, D721, D723, D725, D727, D729, D731, D733, D735, D737, D739, D741, D743, D745, D747, D749, D751, D753, D755, D757, D759, D761, D763, D765, D767, D769, D771, D773, D775, D777, D779, D781, D783, D785, D787, D789, D791, D793, D795, D797, D799, D801, D803, D805, D807, D809, D811, D813, D815, D817, D819, D821, D823, D825, D827, D829, D831, D833, D835, D837, D839, D841, D843, D845, D847, D849, D851, D853, D855, D857, D859, D861, D863, D865, D867, D869, D871, D873, D875, D877, D879, D881, D883, D885, D887, D889, D891, D893, D895, D897, D899, D901, D903, D905, D907, D909, D911, D913, D915, D917, D919, D921, D923, D925, D927, D929, D931, D933, D935, D937, D939, D941, D943, D945, D947, D949, D951, D953, D955, D957, D959, D961, D963, D965, D967, D969, D971, D973, D975, D977, D979, D981, D983, D985, D987, D989, D991, D993, D995, D997, D999: red, LED_SMD:LED_0603_1608Metric
- removed R1001, R1003, R1005, R1007, R1009, R1011, R1013, R1015, R1017, R1019, R1021, R1023, R1025, R1027, R1029, R1031, R1033, R1035, R1037, R1039, R1041, R1043, R1045, R1047, R1049, R1051, R1053, R1055, R1057, R1059, R1061, R1063, R1065, R1067, R1069, R1071, R1073, R1075, R1077, R1079, R1081, R1083, R1085, R1087, R1089, R1091, R1093, R1095, R1097, R1099, R1101, R1103, R1105, R1107, R1109, R1111, R1113, R1115, R1117, R1119, R1121, R1123, R1125, R1127, R1129, R1131, R1133, R1135, R1137, R1139, R1141, R1143, R1145, R1147, R1149, R1151, R1153, R1155, R1157, R1159, R1161, R1163, R1165, R1167, R1169, R1171, R1173, R1175, R1177, R1179, R1181, R1183, R1185, R1187, R1189, R1191, R1193, R1195, R1197, R1199, R1201, R1203, R1205, R1207, R1209, R1211, R1213, R1215, R1217, R1219, R1221, R1223, R1225, R1227, R1229, R1231, R1233, R1235, R1237, R1239, R1241, R1243, R1245, R1247, R705, R707, R709, R711, R713, R715, R717, R719, R721, R723, R725, R727, R729, R731, R733, R735, R737, R739, R741, R743, R745, R747, R749, R751, R753, R755, R757, R759, R761, R763, R765, R767, R769, R771, R773, R775, R777, R779, R781, R783, R785, R787, R789, R791, R793, R795, R797, R799, R801, R803, R805, R807, R809, R811, R813, R815, R817, R819, R821, R823, R825, R827, R829, R831, R833, R835, R837, R839, R841, R843, R845, R847, R849, R851, R853, R855, R857, R859, R861, R863, R865, R867, R869, R871, R873, R875, R877, R879, R881, R883, R885, R887, R889, R891, R893, R895, R897, R899, R901, R903, R905, R907, R909, R911, R913, R915, R917, R919, R921, R923, R925, R927, R929, R931, R933, R935, R937, R939, R941, R943, R945, R947, R949, R951, R953, R955, R957, R959, R961, R963, R965, R967, R969, R971, R973, R975, R977, R979, R981, R983, R985, R987, R989, R991, R993, R995, R997, R999: 680, Resistor_SMD:R_0402_1005Metric
- moved U52 609.4 mm to (37.7, 653.1), turned to 90 degrees
- moved C43 605.9 mm to (24.4, 653.1), turned to -90 degrees
- moved U48 605.3 mm to (37.7, 640.1), turned to 90 degrees
- moved C44 590.5 mm to (17.4, 638.1), turned to -90 degrees
- moved U46 552.5 mm to (37.7, 576.6), turned to 90 degrees
- moved U43 549.0 mm to (37.6, 564.4), turned to 90 degrees
- moved U134 539.1 mm to (49.9, 603.6)
- moved C38 535.4 mm to (22.4, 565.6)
- moved C37 535.4 mm to (22.4, 563.6)
- moved U133 533.9 mm to (49.4, 590.1)
- moved U135 531.2 mm to (49.9, 653.3)
- moved U49 531.1 mm to (37.4, 603.1), turned to 90 degrees
- moved U44 526.4 mm to (37.7, 589.6), turned to 90 degrees
- moved C79 524.6 mm to (59.3, 578.4)
- moved C80 524.6 mm to (59.3, 580.3)
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Routing:
- net /16 bit buffor41/IN_1_7: track 0.00 -> 25.5 mm
- net /16 bit buffor37/IN_1_15: track 0.00 -> 24.2 mm
- net /16 bit buffor38/IN_1_7: track 0.00 -> 24.2 mm
- net /16 bit buffor37/IN_1_7: track 0.00 -> 24.2 mm
- net /16 bit buffor36/IN_1_7: track 0.00 -> 24.2 mm
- net /data7: track 0.00 -> 24.2 mm
- net /16 bit buffor40/IN_1_15: track 0.00 -> 24.2 mm
- net /16 bit buffor38/IN_1_15: track 0.00 -> 24.2 mm
- net /16 bit buffor39/IN_1_7: track 0.00 -> 24.2 mm
- net /16 bit buffor39/IN_1_15: track 0.00 -> 24.1 mm
- net /16 bit buffor41/IN_1_15: track 0.00 -> 23.6 mm
- net /16 bit buffor41/IN_1_6: track 0.00 -> 21.7 mm
- net /16 bit buffor37/IN_1_6: track 0.00 -> 20.6 mm
- net /16 bit buffor36/IN_1_6: track 0.00 -> 20.6 mm
- net /16 bit buffor37/IN_1_14: track 0.00 -> 20.6 mm
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
Commit message: changes
Parts:
- moved U36 22.9 mm to (38.0, 525.7), turned to 90 degrees
- moved U44 13.7 mm to (38.2, 603.2)
- moved U49 13.4 mm to (37.7, 589.7)
- moved U45 13.2 mm to (38.0, 538.3)
- moved U41 13.2 mm to (37.9, 512.6)
- moved U40 13.1 mm to (38.1, 551.5)
- moved U43 12.4 mm to (37.6, 576.8)
- moved U38 12.4 mm to (45.6, 493.6), turned to 90 degrees
- moved U46 12.2 mm to (37.6, 564.4)
- moved U125 12.2 mm to (49.4, 513.0)
Routing:
- net /16 bit buffor36/IN_1_15: track 0.00 -> 24.2 mm
- net /data7: track 24.2 -> 0.00 mm
- net /16 bit buffor40/IN_1_7: track 0.00 -> 24.2 mm
- net /16 bit buffor36/IN_1_7: track 24.2 -> 48.3 mm
- net /16 bit buffor36/IN_1_14: track 0.00 -> 20.6 mm
- net /16 bit buffor40/IN_1_6: track 0.00 -> 20.6 mm
- net /16 bit buffor36/IN_1_6: track 20.6 -> 41.2 mm
- net /16 bit buffor36/IN_1_13: track 0.00 -> 18.3 mm
- net /data5: track 18.3 -> 0.00 mm
- net /16 bit buffor36/IN_1_5: track 18.3 -> 36.6 mm
- net /16 bit buffor36/IN_1_12: track 0.00 -> 14.6 mm
- net /clk: track 14.6 -> 0.00 mm
- net /16 bit buffor40/IN_1_4: track 0.00 -> 14.6 mm
- net /16 bit buffor36/IN_1_4: track 14.6 -> 29.2 mm
- net /16 bit buffor36/IN_1_8: track 0.00 -> 13.9 mm
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
Commit message: changes_1
Parts:
- moved D1 154.7 mm to (35.0, 115.2), turned to 180 degrees
- moved R1 148.7 mm to (38.6, 115.2)
- moved Rd7 67.9 mm to (37.2, 86.8)
- moved Rd3 54.4 mm to (37.2, 92.6)
- moved Dd7 53.5 mm to (33.4, 86.8), turned to 180 degrees
- moved Rd4 52.3 mm to (37.2, 96.8)
- moved Rd5 50.7 mm to (37.2, 100.4)
- moved Rd6 49.4 mm to (37.2, 103.8)
- moved Dd3 37.3 mm to (33.4, 92.6), turned to 180 degrees
- moved Dd4 35.7 mm to (33.4, 96.8), turned to 180 degrees
- moved Dd5 34.7 mm to (33.4, 100.4), turned to 180 degrees
- moved Dd6 33.9 mm to (33.4, 103.8), turned to 180 degrees
- moved U82 26.3 mm to (52.1, 218.4)
- moved Rd1 24.7 mm to (38.6, 119.6)
- moved U123 24.4 mm to (49.7, 499.4)
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Routing:
- net /16 bit buffor33/IN_1_15: track 0.00 -> 24.2 mm
- net /16 bit buffor29/IN_1_15: track 0.00 -> 24.2 mm
- net /16 bit buffor32/IN_1_7: track 0.00 -> 24.2 mm
- net /16 bit buffor28/IN_1_15: track 0.00 -> 24.2 mm
- net /16 bit buffor35/IN_1_7: track 0.00 -> 24.2 mm
- net /16 bit buffor35/IN_1_15: track 0.43 -> 24.6 mm
- net /16 bit buffor31/IN_1_15: track 0.00 -> 24.2 mm
- net /r1_out7: track 0.00 -> 24.2 mm
- net /OUT_5_7: track 0.00 -> 24.2 mm
- net /16 bit buffor30/IN_1_15: track 0.00 -> 24.2 mm
- net /16 bit buffor32/IN_1_15: track 0.00 -> 24.2 mm
- net /r1_out15: track 0.00 -> 24.2 mm
- net /16 bit buffor34/IN_1_7: track 0.00 -> 24.2 mm
- net /16 bit buffor34/IN_1_15: track 0.00 -> 24.2 mm
- net /16 bit buffor33/IN_1_7: track 0.00 -> 24.2 mm
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Other:
- board text added: "ID_REG_SEL_0"
- board text added: "ID_REG_SEL_1"
- board text added: "ID_REG_SEL_2"
- board text added: "ID_REG_SEL_3"
- board text added: "VCC"
- board text added: "mask_restore"
- board text added: "mask_save"
- board text added: "write_enable"

Commit message: changes_2
Parts:
- moved U134 551.1 mm to (209.5, 76.1)
- moved U44 551.1 mm to (197.8, 75.8)
- moved U49 545.2 mm to (173.8, 61.7)
- moved U133 545.2 mm to (185.5, 62.1)
- moved U136 533.3 mm to (209.5, 131.9)
- moved U48 533.3 mm to (197.7, 131.4)
- moved U132 532.0 mm to (137.7, 103.9)
- moved U47 532.0 mm to (125.6, 103.7)
- moved U131 523.5 mm to (209.5, 118.2)
- moved U50 523.5 mm to (197.7, 117.6)
- moved U135 505.4 mm to (161.7, 160.4)
- moved U52 505.4 mm to (149.5, 160.2)
- moved U38 465.5 mm to (197.8, 61.6)
- moved U123 465.5 mm to (209.5, 62.2)
- moved U128 454.6 mm to (185.5, 118.1)
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Routing:
- net /ID_REG_SEL_0: track 3.99 -> 5.64 mm

Commit message: changes_3
Parts:
- moved R1310 123.3 mm to (158.1, 38.2)
- moved R1309 122.0 mm to (158.1, 40.2)
- moved R1308 121.0 mm to (158.2, 42.2)
- moved R1307 120.0 mm to (158.1, 44.2)
- moved R1306 119.1 mm to (158.1, 46.2)
- moved R1305 118.4 mm to (158.1, 48.2)
- moved R1304 117.8 mm to (158.1, 50.2)
- moved R1311 117.2 mm to (158.2, 36.1)
- moved U29 117.0 mm to (148.4, 43.2)
- moved R1312 99.0 mm to (138.7, 36.2), turned to 180 degrees
- moved R1313 99.0 mm to (138.7, 38.2), turned to 180 degrees
- moved R1314 99.0 mm to (138.7, 40.2), turned to 180 degrees
- moved R1315 99.0 mm to (138.7, 42.2), turned to 180 degrees
- moved R1316 98.9 mm to (138.7, 44.2), turned to 180 degrees
- moved R1317 98.9 mm to (138.7, 46.2), turned to 180 degrees
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Routing:
- net /OUT_7_15: track 0.00 -> 98.8 mm, vias 0 -> 3
- net /OUT_7_14: track 0.00 -> 86.5 mm, vias 0 -> 3
- net /OUT_7_13: track 0.00 -> 47.5 mm, vias 0 -> 3
- net /mask_save: track 3.61 -> 12.9 mm
- net /OUT_1_15: track 0.00 -> 8.56 mm
- net /OUT_7_0: track 0.00 -> 8.45 mm, vias 0 -> 1
- net /OUT_1_8: track 0.00 -> 8.11 mm
- net /OUT_1_7: track 0.00 -> 8.01 mm
- net /OUT_1_14: track 0.00 -> 8.00 mm
- net /OUT_7_7: track 0.00 -> 7.92 mm, vias 0 -> 1
- net /OUT_7_1: track 0.00 -> 7.89 mm, vias 0 -> 1
- net /write_enable: track 3.83 -> 11.7 mm
- net /OUT_1_9: track 0.00 -> 7.47 mm
- net /OUT_1_6: track 0.00 -> 7.45 mm
- net /OUT_1_13: track 0.00 -> 7.45 mm
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