File: PCB/Kicad/memory_controller/ADDER.kicad_sch (KiCad schematic)
At the start: 8 parts, among them U10 4b_fulladder__CD74HC283M96, U7 4b_fulladder__CD74HC283M96, U8 4b_fulladder__CD74HC283M96, U9 4b_fulladder__CD74HC283M96

Commit message: pcb init
Parts:
- C10, C7, C8, C9: footprint (none) -> Capacitor_SMD:C_0402_1005Metric
Changed lines of the file:
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@@
 			)
 		)
-		(property "Footprint" ""
+		(property "Footprint" "Capacitor_SMD:C_0402_1005Metric"
 			(at 161.5948 168.91 0)
 			(effects
@@
 			)
 		)
-		(property "Footprint" ""
+		(property "Footprint" "Capacitor_SMD:C_0402_1005Metric"
 			(at 84.1248 74.93 0)
 			(effects
@@
 			)
 		)
-		(property "Footprint" ""
+		(property "Footprint" "Capacitor_SMD:C_0402_1005Metric"
 			(at 85.3948 168.91 0)
 			(effects
@@
 			)
 		)
-		(property "Footprint" ""
+		(property "Footprint" "Capacitor_SMD:C_0402_1005Metric"
 			(at 169.2148 76.2 0)
 			(effects

Commit message: memory controller schematic update
Parts:
- U10, U7, U8, U9: value 4b_fulladder__CD74HC283M96 -> 74283; footprint mALUch_lib:CD_SOIC127P600X175-16N -> Package_SO:SOIC-16_3.9x9.9mm_P1.27mm
