File: PCB/Kicad/memory_controller/RAM_AS7C1026B.kicad_sch (KiCad schematic)
At the start: 2 parts, among them U27 AS7C1026B-10TCN

Commit message: memory controler fix
Parts:
- removed U27: AS7C1026B-10TCN, symbol mALUch_lib:RAM_AS7C1026B-10TCN
- added U13: AS7C1026B-10TCN, symbol mALUch_lib:RAM__AS7C1026B-10TCN
Connections:
- net A0: now also U13.5 (A0)
- net A1: now also U13.4 (A1)
- net A10: now also U13.25 (A10)
- net A11: now also U13.24 (A11)
- net A12: now also U13.21 (A12)
- net A13: now also U13.20 (A13)
- net A14: now also U13.19 (A14)
- net A15: now also U13.18 (A15)
- net A2: now also U13.3 (A2)
- net A3: now also U13.2 (A3)
- net A4: now also U13.1 (A4)
- net A5: now also U13.44 (A5)
- net A6: now also U13.43 (A6)
- net A7: now also U13.42 (A7)
- net A8: now also U13.27 (A8)
- net A9: now also U13.26 (A9)
- net GND: now also U13.12 (GND1), U13.34 (GND2), U13.39 (~{LB}), U13.40 (~{UB}), U13.6 (~{CE})
- net IO0: now also U13.7 (I/O0)
- net IO1: now also U13.8 (I/O1)
- net IO10: now also U13.31 (I/O10)
- net IO11: now also U13.32 (I/O11)
- net IO12: now also U13.35 (I/O12)
- net IO13: now also U13.36 (I/O13)
- net IO14: now also U13.37 (I/O14)
- net IO15: now also U13.38 (I/O15)
- net IO2: now also U13.9 (I/O2)
- net IO3: now also U13.10 (I/O3)
- net IO4: now also U13.13 (I/O4)
- net IO5: now also U13.14 (I/O5)
- net IO6: now also U13.15 (I/O6)
- net IO7: now also U13.16 (I/O7)
- net IO8: now also U13.29 (I/O8)
- net IO9: now also U13.30 (I/O9)
- net VCC: now also U13.11 (VCC1), U13.33 (VCC2)
- net ~{OE}: now also U13.41 (~{OE})
- net ~{WE}: now also U13.17 (~{WE})
Changed lines of the file:
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@@
 	)
 	(symbol
-		(lib_id "mALUch_lib:RAM_AS7C1026B-10TCN")
-		(at 149.86 96.52 0)
+		(lib_id "mALUch_lib:RAM__AS7C1026B-10TCN")
+		(at 149.86 97.79 0)
 		(unit 1)
 		(exclude_from_sim no)
@@
 		(dnp no)
 		(fields_autoplaced yes)
-		(property "Reference" "U27"
+		(property "Reference" "U13"
 			(at 153.2733 58.42 0)
 			(effects
@@
 		)
 		(property "Footprint" ""
-			(at 149.86 78.74 0)
+			(at 149.86 97.79 0)
 			(effects
 				(font
@@
 		)
 		(property "Datasheet" "https://www.tme.eu/Document/46d32e262fd3d2b42e2a04fb336a9d9b/AS7C1026B.pdf"
-			(at 145.034 158.242 0)
+			(at 149.86 43.18 0)
 			(effects
 				(font
@@
 		)
 		(property "Description" ""
-			(at 149.86 78.74 0)
+			(at 149.86 97.79 0)
 			(effects
 				(font
@@
 		)
 		(property "TME" "https://www.tme.eu/pl/details/as7c1026b-10tcn/pamieci-sram-rownolegle/alliance-memory/"
-			(at 150.622 155.448 0)
+			(at 149.86 43.18 0)
 			(effects
 				(font
@@
 			)
 		)
+		(pin "42"
+		)
+		(pin "22"
+		)
+		(pin "17"
+		)
+		(pin "18"
+		)
+		(pin "33"
+		)
+		(pin "39"
+		)
+		(pin "4"
+		)
+		(pin "21"
+		)
+		(pin "2"
+		)
+		(pin "44"
+		)
 		(pin "43"
+		)
+		(pin "27"
+		)
+		(pin "26"
 		)
 		(pin "25"
 		)
-		(pin "20"
-		)
-		(pin "3"
-		)
-		(pin "2"
-		)
-		(pin "5"
-		)
-		(pin "4"
-		)
-		(pin "44"
-		)
-		(pin "42"
-		)
-		(pin "26"
-		)
-		(pin "1"
-		)
-		(pin "27"
-		)
 		(pin "24"
-		)
-		(pin "21"
-		)
-		(pin "18"
 		)
 		(pin "19"
@@
 		(pin "6"
 		)
-		(pin "17"
-		)
-		(pin "39"
-		)
 		(pin "40"
 		)
 		(pin "41"
 		)
-		(pin "22"
+		(pin "1"
+		)
+		(pin "3"
+		)
+		(pin "5"
+		)
+		(pin "20"
 		)
 		(pin "23"
 		)
+		(pin "11"
+		)
+		(pin "12"
+		)
 		(pin "28"
 		)
-		(pin "33"
+		(pin "7"
+		)
+		(pin "34"
 		)
 		(pin "9"
@@
 		(pin "10"
 		)
-		(pin "12"
-		)
-		(pin "14"
-		)
-		(pin "34"
+		(pin "13"
 		)
 		(pin "8"
 		)
-		(pin "29"
-		)
-		(pin "30"
-		)
-		(pin "31"
-		)
-		(pin "37"
+		(pin "14"
 		)
 		(pin "15"
@@
 		(pin "16"
 		)
+		(pin "29"
+		)
+		(pin "31"
+		)
 		(pin "32"
 		)
-		(pin "13"
+		(pin "30"
+		)
+		(pin "36"
 		)
 		(pin "35"
 		)
-		(pin "11"
-		)
-		(pin "7"
-		)
-		(pin "36"
+		(pin "37"
 		)
 		(pin "38"
@@
 			(project ""
 				(path "/dccec861-b967-466c-843e-d6d1ad6064ce/65198342-3b70-4e1d-8493-7cbe3d0407e3"
-					(reference "U27")
+					(reference "U13")
 					(unit 1)
 				)

Commit message: kicad fix
Parts:
- renumbered C27 to C25, U13 to U25
Changed lines of the file:
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@@
 		(dnp no)
 		(fields_autoplaced yes)
-		(property "Reference" "U13"
+		(property "Reference" "U25"
 			(at 153.2733 58.42 0)
 			(effects
@@
 			(project ""
 				(path "/dccec861-b967-466c-843e-d6d1ad6064ce/65198342-3b70-4e1d-8493-7cbe3d0407e3"
-					(reference "U13")
+					(reference "U25")
 					(unit 1)
 				)
@@
 		(dnp no)
 		(fields_autoplaced yes)
-		(property "Reference" "#PWR0138"
+		(property "Reference" "#PWR0128"
 			(at 149.86 62.23 0)
 			(effects
@@
 			(project ""
 				(path "/dccec861-b967-466c-843e-d6d1ad6064ce/65198342-3b70-4e1d-8493-7cbe3d0407e3"
-					(reference "#PWR0138")
+					(reference "#PWR0128")
 					(unit 1)
 				)
@@
 		(dnp no)
 		(fields_autoplaced yes)
-		(property "Reference" "#PWR0135"
+		(property "Reference" "#PWR0125"
 			(at 125.73 113.03 0)
 			(effects
@@
 			(project "memory_controller"
 				(path "/dccec861-b967-466c-843e-d6d1ad6064ce/65198342-3b70-4e1d-8493-7cbe3d0407e3"
-					(reference "#PWR0135")
+					(reference "#PWR0125")
 					(unit 1)
 				)
@@
 		(dnp no)
 		(fields_autoplaced yes)
-		(property "Reference" "#PWR0136"
+		(property "Reference" "#PWR0126"
 			(at 137.16 49.53 0)
 			(effects
@@
 			(project "memory_controller"
 				(path "/dccec861-b967-466c-843e-d6d1ad6064ce/65198342-3b70-4e1d-8493-7cbe3d0407e3"
-					(reference "#PWR0136")
+					(reference "#PWR0126")
 					(unit 1)
 				)
@@
 		(dnp no)
 		(fields_autoplaced yes)
-		(property "Reference" "#PWR0137"
+		(property "Reference" "#PWR0127"
 			(at 137.16 59.69 0)
 			(effects
@@
 			(project "memory_controller"
 				(path "/dccec861-b967-466c-843e-d6d1ad6064ce/65198342-3b70-4e1d-8493-7cbe3d0407e3"
-					(reference "#PWR0137")
+					(reference "#PWR0127")
 					(unit 1)
 				)
@@
 		(dnp no)
 		(fields_autoplaced yes)
-		(property "Reference" "#PWR0139"
+		(property "Reference" "#PWR0129"
 			(at 149.86 146.05 0)
 			(effects
@@
 			(project ""
 				(path "/dccec861-b967-466c-843e-d6d1ad6064ce/65198342-3b70-4e1d-8493-7cbe3d0407e3"
-					(reference "#PWR0139")
+					(reference "#PWR0129")
 					(unit 1)
 				)
@@
 		(dnp no)
 		(fields_autoplaced yes)
-		(property "Reference" "C27"
+		(property "Reference" "C25"
 			(at 140.97 48.2599 0)
 			(effects
@@
 			(project "memory_controller"
 				(path "/dccec861-b967-466c-843e-d6d1ad6064ce/65198342-3b70-4e1d-8493-7cbe3d0407e3"
-					(reference "C27")
-					(unit 1)
-				)
+					(reference "C25")
+					(unit 1)
+				)

Commit message: pcb init
Parts:
- C25: footprint (none) -> Capacitor_SMD:C_0402_1005Metric
- U25: footprint (none) -> Package_SO:TSOP-II-44_10.16x18.41mm_P0.8mm
Changed lines of the file:
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@@
 			)
 		)
-		(property "Footprint" ""
+		(property "Footprint" "Package_SO:TSOP-II-44_10.16x18.41mm_P0.8mm"
 			(at 149.86 97.79 0)
 			(effects
@@
 			)
 		)
-		(property "Footprint" ""
+		(property "Footprint" "Capacitor_SMD:C_0402_1005Metric"
 			(at 136.1948 45.72 0)
 			(effects

Commit message: names
Other:
- title: (none) -> RAM AS7C1026B
Changed lines of the file:
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@@
 	(generator_version "9.0")
 	(paper "A4")
+	(title_block
+		(title "RAM AS7C1026B")
+		(comment 1 "review: Hubert Wójcik")
+		(comment 2 "author: Maciej Rogoz")
+	)
 	(junction
 		(at 149.86 58.42)
