File: PCB/Kicad/alu/LAYER2.kicad_sch (KiCad schematic)
At the start: 4 parts, among them U33 74LS257, U34 74LS257, U35 74LS257, U36 74LS257

Commit message: UPDATE
Parts:
- added C30, C31, C32, C33: 10n, symbol Device:C
Connections:
- net GND: now also U36.13 (I1c), C30.2, C31.2, C32.2, C33.2
- net Lin1: no longer U33.3 (I1a)
- net Lin10: now also U35.3 (I1a); no longer U35.6 (I1b)
- net Lin11: now also U35.6 (I1b); no longer U35.13 (I1c)
- net Lin12: now also U35.13 (I1c); no longer U35.10 (I1d)
- net Lin13: now also U35.10 (I1d); no longer U36.3 (I1a)
- net Lin14: now also U36.3 (I1a); no longer U36.6 (I1b)
- net Lin15: now also U36.6 (I1b); no longer U36.13 (I1c)
- net Lin2: now also U33.3 (I1a); no longer U33.6 (I1b)
- net Lin3: now also U33.6 (I1b); no longer U33.13 (I1c)
- net Lin4: now also U33.13 (I1c); no longer U33.10 (I1d)
- net Lin5: now also U33.10 (I1d); no longer U34.3 (I1a)
- net Lin6: now also U34.3 (I1a); no longer U34.6 (I1b)
- net Lin7: now also U34.6 (I1b); no longer U34.13 (I1c)
- net Lin8: now also U34.13 (I1c); no longer U34.10 (I1d)
- net Lin9: now also U34.10 (I1d); no longer U35.3 (I1a)
- net Lout0: no longer U36.4 (Za)
- net Lout1: no longer U36.7 (Zb)
- net Lout2: no longer U36.12 (Zc)
- net Lout3: no longer U36.9 (Zd)
- net VCC: now also C30.1, C31.1, C32.1, C33.1
- new net Lout12: U36.4 (Za)
- new net Lout13: U36.7 (Zb)
- new net Lout14: U36.12 (Zc)
- new net Lout15: U36.9 (Zd)

Commit message: LEDs added
REGISTER.kicad_sch LEDs added to both REG_A and REG_B
Parts:
- renumbered C33 to C34, C30 to C35, C31 to C36, C32 to C37, U33 to U34, U34 to U35, U35 to U36, U36 to U37
Changed lines of the file:
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@@
 		(dnp no)
 		(fields_autoplaced yes)
-		(property "Reference" "#PWR073"
+		(property "Reference" "#PWR0150"
 			(at 161.29 109.22 0)
 			(effects
@@
 			(project "alu"
 				(path "/2f66781e-a1af-4159-bccc-5b52a490afb6/80a1dfcd-7697-4d3a-b862-6f8977c64ed2/1e85d2b8-1084-42d0-b5ce-c4d5d7f3b84e"
-					(reference "#PWR073")
+					(reference "#PWR0150")
 					(unit 1)
 				)
@@
 		(dnp no)
 		(fields_autoplaced yes)
-		(property "Reference" "U36"
+		(property "Reference" "U37"
 			(at 163.4333 107.95 0)
 			(effects
@@
 			(project "alu"
 				(path "/2f66781e-a1af-4159-bccc-5b52a490afb6/80a1dfcd-7697-4d3a-b862-6f8977c64ed2/1e85d2b8-1084-42d0-b5ce-c4d5d7f3b84e"
-					(reference "U36")
+					(reference "U37")
 					(unit 1)
 				)
@@
 		(dnp no)
 		(fields_autoplaced yes)
-		(property "Reference" "#PWR0185"
+		(property "Reference" "#PWR0144"
 			(at 140.97 139.7 0)
 			(effects
@@
 			(project "alu"
 				(path "/2f66781e-a1af-4159-bccc-5b52a490afb6/80a1dfcd-7697-4d3a-b862-6f8977c64ed2/1e85d2b8-1084-42d0-b5ce-c4d5d7f3b84e"
-					(reference "#PWR0185")
+					(reference "#PWR0144")
 					(unit 1)
 				)
@@
 		(dnp no)
 		(fields_autoplaced yes)
-		(property "Reference" "#PWR0241"
+		(property "Reference" "#PWR0142"
 			(at 137.16 120.65 0)
 			(effects
@@
 			(project "alu"
 				(path "/2f66781e-a1af-4159-bccc-5b52a490afb6/80a1dfcd-7697-4d3a-b862-6f8977c64ed2/1e85d2b8-1084-42d0-b5ce-c4d5d7f3b84e"
-					(reference "#PWR0241")
+					(reference "#PWR0142")
 					(unit 1)
 				)
@@
 		(dnp no)
 		(fields_autoplaced yes)
-		(property "Reference" "U34"
+		(property "Reference" "U35"
 			(at 112.6333 107.95 0)
 			(effects
@@
 			(project "alu"
 				(path "/2f66781e-a1af-4159-bccc-5b52a490afb6/80a1dfcd-7697-4d3a-b862-6f8977c64ed2/1e85d2b8-1084-42d0-b5ce-c4d5d7f3b84e"
-					(reference "U34")
+					(reference "U35")
 					(unit 1)
 				)
@@
 		(dnp no)
 		(fields_autoplaced yes)
-		(property "Reference" "#PWR081"
+		(property "Reference" "#PWR0147"
 			(at 148.59 154.94 0)
 			(effects
@@
 			(project "alu"
 				(path "/2f66781e-a1af-4159-bccc-5b52a490afb6/80a1dfcd-7697-4d3a-b862-6f8977c64ed2/1e85d2b8-1084-42d0-b5ce-c4d5d7f3b84e"
-					(reference "#PWR081")
+					(reference "#PWR0147")
 					(unit 1)
 				)
@@
 		(dnp no)
 		(fields_autoplaced yes)
-		(property "Reference" "#PWR064"
+		(property "Reference" "#PWR0139"
 			(at 110.49 91.44 0)
 			(effects
@@
 			(project "alu"
 				(path "/2f66781e-a1af-4159-bccc-5b52a490afb6/80a1dfcd-7697-4d3a-b862-6f8977c64ed2/1e85d2b8-1084-42d0-b5ce-c4d5d7f3b84e"
-					(reference "#PWR064")
+					(reference "#PWR0139")
 					(unit 1)
 				)
@@
 		(dnp no)
 		(fields_autoplaced yes)
-		(property "Reference" "#PWR087"
+		(property "Reference" "#PWR0145"
 			(at 143.51 147.32 0)
 			(effects
@@
 			(project ""
 				(path "/2f66781e-a1af-4159-bccc-5b52a490afb6/80a1dfcd-7697-4d3a-b862-6f8977c64ed2/1e85d2b8-1084-42d0-b5ce-c4d5d7f3b84e"
-					(reference "#PWR087")
+					(reference "#PWR0145")
 					(unit 1)
 				)
@@
 		(dnp no)
 		(fields_autoplaced yes)
-		(property "Reference" "#PWR082"
+		(property "Reference" "#PWR0146"
 			(at 148.59 83.82 0)
 			(effects
@@
 			(project "alu"
 				(path "/2f66781e-a1af-4159-bccc-5b52a490afb6/80a1dfcd-7697-4d3a-b862-6f8977c64ed2/1e85d2b8-1084-42d0-b5ce-c4d5d7f3b84e"
-					(reference "#PWR082")
+					(reference "#PWR0146")
 					(unit 1)
 				)
@@
 		(dnp no)
 		(fields_autoplaced yes)
-		(property "Reference" "#PWR066"
+		(property "Reference" "#PWR0151"
 			(at 161.29 162.56 0)
 			(effects
@@
 			(project "alu"
 				(path "/2f66781e-a1af-4159-bccc-5b52a490afb6/80a1dfcd-7697-4d3a-b862-6f8977c64ed2/1e85d2b8-1084-42d0-b5ce-c4d5d7f3b84e"
-					(reference "#PWR066")
+					(reference "#PWR0151")
 					(unit 1)
 				)
@@
 		(dnp no)
 		(fields_autoplaced yes)
-		(property "Reference" "#PWR0240"
+		(property "Reference" "#PWR0135"
 			(at 87.63 120.65 0)
 			(effects
@@
 			(project "alu"
 				(path "/2f66781e-a1af-4159-bccc-5b52a490afb6/80a1dfcd-7697-4d3a-b862-6f8977c64ed2/1e85d2b8-1084-42d0-b5ce-c4d5d7f3b84e"
-					(reference "#PWR0240")
+					(reference "#PWR0135")
 					(unit 1)
 				)
@@
 		(dnp no)
 		(fields_autoplaced yes)
-		(property "Reference" "C32"
+		(property "Reference" "C37"
 			(at 142.24 38.0999 0)
 			(effects
@@
 			(project "alu"
 				(path "/2f66781e-a1af-4159-bccc-5b52a490afb6/80a1dfcd-7697-4d3a-b862-6f8977c64ed2/1e85d2b8-1084-42d0-b5ce-c4d5d7f3b84e"
-					(reference "C32")
+					(reference "C37")
 					(unit 1)
 				)
@@
 		(dnp no)
 		(fields_autoplaced yes)
-		(property "Reference" "U35"
+		(property "Reference" "U36"
 			(at 163.4333 36.83 0)
 			(effects
@@
 			(project "alu"
 				(path "/2f66781e-a1af-4159-bccc-5b52a490afb6/80a1dfcd-7697-4d3a-b862-6f8977c64ed2/1e85d2b8-1084-42d0-b5ce-c4d5d7f3b84e"
-					(reference "U35")
+					(reference "U36")
 					(unit 1)
 				)
@@
 		(dnp no)
 		(fields_autoplaced yes)
-		(property "Reference" "C30"
+		(property "Reference" "C35"
 			(at 91.44 109.2199 0)
 			(effects
@@
 			(project "alu"
 				(path "/2f66781e-a1af-4159-bccc-5b52a490afb6/80a1dfcd-7697-4d3a-b862-6f8977c64ed2/1e85d2b8-1084-42d0-b5ce-c4d5d7f3b84e"
-					(reference "C30")
+					(reference "C35")
 					(unit 1)
 				)
@@
 		(dnp no)
 		(fields_autoplaced yes)
-		(property "Reference" "#PWR072"
+		(property "Reference" "#PWR0140"
 			(at 110.49 109.22 0)
 			(effects
@@
 			(project "alu"
 				(path "/2f66781e-a1af-4159-bccc-5b52a490afb6/80a1dfcd-7697-4d3a-b862-6f8977c64ed2/1e85d2b8-1084-42d0-b5ce-c4d5d7f3b84e"
-					(reference "#PWR072")
+					(reference "#PWR0140")
 					(unit 1)
 				)
@@
 		(dnp no)
 		(fields_autoplaced yes)
-		(property "Reference" "#PWR080"
+		(property "Reference" "#PWR0137"
 			(at 97.79 154.94 0)
 			(effects
@@
 			(project "alu"
 				(path "/2f66781e-a1af-4159-bccc-5b52a490afb6/80a1dfcd-7697-4d3a-b862-6f8977c64ed2/1e85d2b8-1084-42d0-b5ce-c4d5d7f3b84e"
-					(reference "#PWR080")
+					(reference "#PWR0137")
 					(unit 1)
 				)
@@
 		(dnp no)
 		(fields_autoplaced yes)
-		(property "Reference" "#PWR074"
+		(property "Reference" "#PWR0138"
 			(at 110.49 38.1 0)
 			(effects
@@
 			(project "alu"
 				(path "/2f66781e-a1af-4159-bccc-5b52a490afb6/80a1dfcd-7697-4d3a-b862-6f8977c64ed2/1e85d2b8-1084-42d0-b5ce-c4d5d7f3b84e"
-					(reference "#PWR074")
+					(reference "#PWR0138")
 					(unit 1)
 				)
@@
 		(dnp no)
 		(fields_autoplaced yes)
-		(property "Reference" "#PWR075"
+		(property "Reference" "#PWR0148"
 			(at 161.29 38.1 0)
 			(effects
@@
 			(project "alu"
 				(path "/2f66781e-a1af-4159-bccc-5b52a490afb6/80a1dfcd-7697-4d3a-b862-6f8977c64ed2/1e85d2b8-1084-42d0-b5ce-c4d5d7f3b84e"
-					(reference "#PWR075")
+					(reference "#PWR0148")
 					(unit 1)
 				)
@@
 		(dnp no)
 		(fields_autoplaced yes)
-		(property "Reference" "U33"
+		(property "Reference" "U34"
 			(at 112.6333 36.83 0)
 			(effects
@@
 			(project "alu"
 				(path "/2f66781e-a1af-4159-bccc-5b52a490afb6/80a1dfcd-7697-4d3a-b862-6f8977c64ed2/1e85d2b8-1084-42d0-b5ce-c4d5d7f3b84e"
-					(reference "U33")
+					(reference "U34")
 					(unit 1)
 				)
@@
 		(dnp no)
 		(fields_autoplaced yes)
-		(property "Reference" "#PWR0242"
+		(property "Reference" "#PWR0143"
 			(at 138.43 49.53 0)
 			(effects
@@
 			(project "alu"
 				(path "/2f66781e-a1af-4159-bccc-5b52a490afb6/80a1dfcd-7697-4d3a-b862-6f8977c64ed2/1e85d2b8-1084-42d0-b5ce-c4d5d7f3b84e"
-					(reference "#PWR0242")
+					(reference "#PWR0143")
 					(unit 1)
 				)
@@
 		(dnp no)
 		(fields_autoplaced yes)
-		(property "Reference" "#PWR065"
+		(property "Reference" "#PWR0149"
 			(at 161.29 91.44 0)
 			(effects
@@
 			(project "alu"
 				(path "/2f66781e-a1af-4159-bccc-5b52a490afb6/80a1dfcd-7697-4d3a-b862-6f8977c64ed2/1e85d2b8-1084-42d0-b5ce-c4d5d7f3b84e"
-					(reference "#PWR065")
+					(reference "#PWR0149")
 					(unit 1)
 				)
@@
 		(dnp no)
 		(fields_autoplaced yes)
-		(property "Reference" "C33"
+		(property "Reference" "C34"
 			(at 91.44 38.0999 0)
 			(effects
@@
 			(project "alu"
 				(path "/2f66781e-a1af-4159-bccc-5b52a490afb6/80a1dfcd-7697-4d3a-b862-6f8977c64ed2/1e85d2b8-1084-42d0-b5ce-c4d5d7f3b84e"
-					(reference "C33")
+					(reference "C34")
 					(unit 1)
 				)
@@
 		(dnp no)
 		(fields_autoplaced yes)
-		(property "Reference" "#PWR0243"
+		(property "Reference" "#PWR0134"
 			(at 87.63 49.53 0)
 			(effects
@@
 			(project "alu"
 				(path "/2f66781e-a1af-4159-bccc-5b52a490afb6/80a1dfcd-7697-4d3a-b862-6f8977c64ed2/1e85d2b8-1084-42d0-b5ce-c4d5d7f3b84e"
-					(reference "#PWR0243")
+					(reference "#PWR0134")
 					(unit 1)
 				)
@@
 		(dnp no)
 		(fields_autoplaced yes)
-		(property "Reference" "#PWR067"
+		(property "Reference" "#PWR0141"
 			(at 110.49 162.56 0)
 			(effects
@@
 			(project "alu"
 				(path "/2f66781e-a1af-4159-bccc-5b52a490afb6/80a1dfcd-7697-4d3a-b862-6f8977c64ed2/1e85d2b8-1084-42d0-b5ce-c4d5d7f3b84e"
-					(reference "#PWR067")
+					(reference "#PWR0141")
 					(unit 1)
 				)
@@
 		(dnp no)
 		(fields_autoplaced yes)
-		(property "Reference" "#PWR083"
+		(property "Reference" "#PWR0136"
 			(at 97.79 83.82 0)
 			(effects
@@
 			(project "alu"
 				(path "/2f66781e-a1af-4159-bccc-5b52a490afb6/80a1dfcd-7697-4d3a-b862-6f8977c64ed2/1e85d2b8-1084-42d0-b5ce-c4d5d7f3b84e"
-					(reference "#PWR083")
+					(reference "#PWR0136")
 					(unit 1)
 				)
@@
 		(dnp no)
 		(fields_autoplaced yes)
-		(property "Reference" "C31"
+		(property "Reference" "C36"
 			(at 140.97 109.2199 0)
 			(effects
@@
 			(project "alu"
 				(path "/2f66781e-a1af-4159-bccc-5b52a490afb6/80a1dfcd-7697-4d3a-b862-6f8977c64ed2/1e85d2b8-1084-42d0-b5ce-c4d5d7f3b84e"
-					(reference "C31")
-					(unit 1)
-				)
+					(reference "C36")
+					(unit 1)
+				)

Commit message: Footprints, PCB update
Added footprints to all components, updated the PCB with the schematic
Parts:
- C34, C35, C36, C37: footprint (none) -> Capacitor_SMD:C_0603_1608Metric
- U34, U35, U36, U37: footprint (none) -> Package_SO:SOIC-16_3.9x9.9mm_P1.27mm
Changed lines of the file:
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@@
 			)
 		)
-		(property "Footprint" ""
+		(property "Footprint" "Package_SO:SOIC-16_3.9x9.9mm_P1.27mm"
 			(at 161.29 130.81 0)
 			(effects
@@
 			)
 		)
-		(property "Footprint" ""
+		(property "Footprint" "Package_SO:SOIC-16_3.9x9.9mm_P1.27mm"
 			(at 110.49 130.81 0)
 			(effects
@@
 			)
 		)
-		(property "Footprint" ""
+		(property "Footprint" "Capacitor_SMD:C_0603_1608Metric"
 			(at 139.3952 43.18 0)
 			(effects
@@
 			)
 		)
-		(property "Footprint" ""
+		(property "Footprint" "Package_SO:SOIC-16_3.9x9.9mm_P1.27mm"
 			(at 161.29 59.69 0)
 			(effects
@@
 			)
 		)
-		(property "Footprint" ""
+		(property "Footprint" "Capacitor_SMD:C_0603_1608Metric"
 			(at 88.5952 114.3 0)
 			(effects
@@
 			)
 		)
-		(property "Footprint" ""
+		(property "Footprint" "Package_SO:SOIC-16_3.9x9.9mm_P1.27mm"
 			(at 110.49 59.69 0)
 			(effects
@@
 			)
 		)
-		(property "Footprint" ""
+		(property "Footprint" "Capacitor_SMD:C_0603_1608Metric"
 			(at 88.5952 43.18 0)
 			(effects
@@
 			)
 		)
-		(property "Footprint" ""
+		(property "Footprint" "Capacitor_SMD:C_0603_1608Metric"
 			(at 138.1252 114.3 0)
 			(effects

Commit message: ALU Pcb update
Parts:
- C34, C35, C36, C37: value 10n -> 100nF; footprint Capacitor_SMD:C_0603_1608Metric -> Capacitor_SMD:C_0402_1005Metric
- U34, U35, U36, U37: value 74LS257 -> 74257
