File: PCB/Kicad/alu/REGISTER.kicad_sch (KiCad schematic)
At the start: 2 parts, among them U49 74LS377, U50 74LS377

Commit message: Update
Other:
- note removed: "Takie coś?"
Changed lines of the file:
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@@
 	(generator_version "9.0")
 	(paper "A4")
-	(text "Takie coś?\n"
-		(exclude_from_sim no)
-		(at 116.332 103.378 0)
-		(effects
-			(font
-				(size 5.08 5.08)
-			)
-		)
-	)
 	(no_connect
 		(at 20.32 30.48)

Commit message: UPDATE
Parts:
- renumbered U49 to U57
Changed lines of the file:
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@@
+					(unit 1)
+				)
+				(path "/2f66781e-a1af-4159-bccc-5b52a490afb6/9a179709-3864-45fb-ba1b-bb4e75fdee37"
+					(reference "#PWR0147")
 					(unit 1)
 				)
@@
 		(dnp no)
 		(fields_autoplaced yes)
-		(property "Reference" "U49"
+		(property "Reference" "U57"
 			(at 79.6133 45.72 0)
 			(effects
@@
 			(project ""
 				(path "/2f66781e-a1af-4159-bccc-5b52a490afb6/3c4c5033-bd2a-4f85-be2a-cffc4fb60939"
-					(reference "U49")
+					(reference "U57")
+					(unit 1)
+				)
+				(path "/2f66781e-a1af-4159-bccc-5b52a490afb6/9a179709-3864-45fb-ba1b-bb4e75fdee37"
+					(reference "U57")
 					(unit 1)
 				)
@@
 		(dnp no)
 		(fields_autoplaced yes)
-		(property "Reference" "#PWR0127"
+		(property "Reference" "#PWR0145"
 			(at 77.47 92.71 0)
 			(effects
@@
 			(project ""
 				(path "/2f66781e-a1af-4159-bccc-5b52a490afb6/3c4c5033-bd2a-4f85-be2a-cffc4fb60939"
-					(reference "#PWR0127")
+					(reference "#PWR0145")
+					(unit 1)
+				)
+				(path "/2f66781e-a1af-4159-bccc-5b52a490afb6/9a179709-3864-45fb-ba1b-bb4e75fdee37"
+					(reference "#PWR0145")
 					(unit 1)
 				)
@@
 					(unit 1)
 				)
+				(path "/2f66781e-a1af-4159-bccc-5b52a490afb6/9a179709-3864-45fb-ba1b-bb4e75fdee37"
+					(reference "#PWR0146")
+					(unit 1)
+				)
 			)
 		)
@@
 		(dnp no)
 		(fields_autoplaced yes)
-		(property "Reference" "#PWR0126"
+		(property "Reference" "#PWR0144"
 			(at 77.47 49.53 0)
 			(effects
@@
 			(project ""
 				(path "/2f66781e-a1af-4159-bccc-5b52a490afb6/3c4c5033-bd2a-4f85-be2a-cffc4fb60939"
-					(reference "#PWR0126")
+					(reference "#PWR0144")
+					(unit 1)
+				)
+				(path "/2f66781e-a1af-4159-bccc-5b52a490afb6/9a179709-3864-45fb-ba1b-bb4e75fdee37"
+					(reference "#PWR0144")
 					(unit 1)
 				)
@@
 					(unit 1)
 				)
+				(path "/2f66781e-a1af-4159-bccc-5b52a490afb6/9a179709-3864-45fb-ba1b-bb4e75fdee37"
+					(reference "U58")
+					(unit 1)
+				)

Commit message: UPDATE
Parts:
- added C46, C48: 10n, symbol Device:C
- renumbered U57 to U75
Connections:
- net GND: now also C46.2, C48.2
- net VCC: now also C46.1, C48.1

Commit message: LEDs added
REGISTER.kicad_sch LEDs added to both REG_A and REG_B
Parts:
- added D10, D11, D12, D13, D14, D15, D16, D17, D18, D19, D20, D21, D6, D7, D8, D9: red, LED_SMD:LED_0603_1608Metric, symbol Device:LED
- added R10, R11, R12, R13, R14, R15, R16, R17, R18, R19, R20, R21, R6, R7, R8, R9: 680, Resistor_SMD:R_0402_1005Metric, symbol Device:R
- renumbered C46 to C50, C48 to C51, U75 to U50, U50 to U51
Connections:
- net GND: now also R10.2, R11.2, R12.2, R13.2, R14.2, R15.2, R16.2, R17.2, R18.2, R19.2, R20.2, R21.2, R6.2, R7.2, R8.2, R9.2
- net REG_OUT0: now also D6.2 (A)
- net REG_OUT1: now also D8.2 (A)
- net REG_OUT10: now also D11.2 (A)
- net REG_OUT11: now also D13.2 (A)
- net REG_OUT12: now also D15.2 (A)
- net REG_OUT13: now also D17.2 (A)
- net REG_OUT14: now also D19.2 (A)
- net REG_OUT15: now also D21.2 (A)
- net REG_OUT2: now also D10.2 (A)
- net REG_OUT3: now also D12.2 (A)
- net REG_OUT4: now also D14.2 (A)
- net REG_OUT5: now also D16.2 (A)
- net REG_OUT6: now also D18.2 (A)
- net REG_OUT7: now also D20.2 (A)
- net REG_OUT8: now also D7.2 (A)
- net REG_OUT9: now also D9.2 (A)
- new net: D11.1 (K), R11.1
- new net: D10.1 (K), R10.1
- new net: D15.1 (K), R15.1
- new net: D18.1 (K), R18.1
- new net: D21.1 (K), R21.1
- new net: D17.1 (K), R17.1
- new net: D13.1 (K), R13.1
- new net: D16.1 (K), R16.1
- new net: D12.1 (K), R12.1
- new net: D6.1 (K), R6.1
- new net: D20.1 (K), R20.1
- new net: D14.1 (K), R14.1
- new net: D7.1 (K), R7.1
- new net: D19.1 (K), R19.1
- new net: D8.1 (K), R8.1
- new net: D9.1 (K), R9.1

Commit message: Footprints, PCB update
Added footprints to all components, updated the PCB with the schematic
Parts:
- C50, C51: footprint (none) -> Capacitor_SMD:C_0603_1608Metric
- U50, U51: footprint (none) -> Package_SO:SOIC-20W_7.5x12.8mm_P1.27mm
Changed lines of the file:
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@@
 			)
 		)
-		(property "Footprint" ""
+		(property "Footprint" "Package_SO:SOIC-20W_7.5x12.8mm_P1.27mm"
 			(at 77.47 66.04 0)
 			(effects
@@
 			)
 		)
-		(property "Footprint" ""
+		(property "Footprint" "Capacitor_SMD:C_0603_1608Metric"
 			(at 117.8052 44.45 0)
 			(effects
@@
 			)
 		)
-		(property "Footprint" ""
+		(property "Footprint" "Capacitor_SMD:C_0603_1608Metric"
 			(at 68.2752 44.45 0)
 			(effects
@@
 			)
 		)
-		(property "Footprint" ""
+		(property "Footprint" "Package_SO:SOIC-20W_7.5x12.8mm_P1.27mm"
 			(at 127 66.04 0)
 			(effects

Commit message: ALU Pcb update
Parts:
- C50, C51: value 10n -> 100nF; footprint Capacitor_SMD:C_0603_1608Metric -> Capacitor_SMD:C_0402_1005Metric
- U50, U51: value 74LS377 -> 74377; footprint Package_SO:SOIC-20W_7.5x12.8mm_P1.27mm -> Package_SO:SSOP-20_5.3x7.2mm_P0.65mm
