File: PCB/Kicad/alu/REV2.kicad_sch (KiCad schematic)
At the start: 4 parts, among them U45 74LS257, U46 74LS257, U47 74LS257, U48 74LS257

Commit message: UPDATE
Parts:
- added C42, C43, C44, C45: 10n, symbol Device:C
Connections:
- net GND: now also C42.2, C43.2, C44.2, C45.2
- net VCC: now also C42.1, C43.1, C44.1, C45.1

Commit message: LEDs added
REGISTER.kicad_sch LEDs added to both REG_A and REG_B
Parts:
- renumbered C43 to C46, C42 to C47, C45 to C48, C44 to C49, U45 to U46, U46 to U47, U47 to U48, U48 to U49
Changed lines of the file:
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@@
 		(dnp no)
 		(fields_autoplaced yes)
-		(property "Reference" "#PWR0255"
+		(property "Reference" "#PWR0204"
 			(at 148.59 113.03 0)
 			(effects
@@
 			(project "alu"
 				(path "/2f66781e-a1af-4159-bccc-5b52a490afb6/80a1dfcd-7697-4d3a-b862-6f8977c64ed2/d589d6f2-03b4-410e-8081-b53488f96cb4"
-					(reference "#PWR0255")
+					(reference "#PWR0204")
 					(unit 1)
 				)
@@
 		(dnp no)
 		(fields_autoplaced yes)
-		(property "Reference" "#PWR0114"
+		(property "Reference" "#PWR0198"
 			(at 87.63 87.63 0)
 			(effects
@@
 			(project "alu"
 				(path "/2f66781e-a1af-4159-bccc-5b52a490afb6/80a1dfcd-7697-4d3a-b862-6f8977c64ed2/d589d6f2-03b4-410e-8081-b53488f96cb4"
-					(reference "#PWR0114")
+					(reference "#PWR0198")
 					(unit 1)
 				)
@@
 		(dnp no)
 		(fields_autoplaced yes)
-		(property "Reference" "U46"
+		(property "Reference" "U47"
 			(at 106.2833 101.6 0)
 			(effects
@@
 			(project "alu"
 				(path "/2f66781e-a1af-4159-bccc-5b52a490afb6/80a1dfcd-7697-4d3a-b862-6f8977c64ed2/d589d6f2-03b4-410e-8081-b53488f96cb4"
-					(reference "U46")
+					(reference "U47")
 					(unit 1)
 				)
@@
 		(dnp no)
 		(fields_autoplaced yes)
-		(property "Reference" "#PWR0253"
+		(property "Reference" "#PWR0196"
 			(at 81.28 49.53 0)
 			(effects
@@
 			(project "alu"
 				(path "/2f66781e-a1af-4159-bccc-5b52a490afb6/80a1dfcd-7697-4d3a-b862-6f8977c64ed2/d589d6f2-03b4-410e-8081-b53488f96cb4"
-					(reference "#PWR0253")
+					(reference "#PWR0196")
 					(unit 1)
 				)
@@
 		(dnp no)
 		(fields_autoplaced yes)
-		(property "Reference" "#PWR0116"
+		(property "Reference" "#PWR0200"
 			(at 104.14 38.1 0)
 			(effects
@@
 			(project "alu"
 				(path "/2f66781e-a1af-4159-bccc-5b52a490afb6/80a1dfcd-7697-4d3a-b862-6f8977c64ed2/d589d6f2-03b4-410e-8081-b53488f96cb4"
-					(reference "#PWR0116")
+					(reference "#PWR0200")
 					(unit 1)
 				)
@@
 		(dnp no)
 		(fields_autoplaced yes)
-		(property "Reference" "C45"
+		(property "Reference" "C48"
 			(at 152.4 101.5999 0)
 			(effects
@@
 			(project "alu"
 				(path "/2f66781e-a1af-4159-bccc-5b52a490afb6/80a1dfcd-7697-4d3a-b862-6f8977c64ed2/d589d6f2-03b4-410e-8081-b53488f96cb4"
-					(reference "C45")
+					(reference "C48")
 					(unit 1)
 				)
@@
 		(dnp no)
 		(fields_autoplaced yes)
-		(property "Reference" "C43"
+		(property "Reference" "C46"
 			(at 85.09 38.0999 0)
 			(effects
@@
 			(project "alu"
 				(path "/2f66781e-a1af-4159-bccc-5b52a490afb6/80a1dfcd-7697-4d3a-b862-6f8977c64ed2/d589d6f2-03b4-410e-8081-b53488f96cb4"
-					(reference "C43")
+					(reference "C46")
 					(unit 1)
 				)
@@
 		(dnp no)
 		(fields_autoplaced yes)
-		(property "Reference" "C42"
+		(property "Reference" "C47"
 			(at 85.09 102.8699 0)
 			(effects
@@
 			(project "alu"
 				(path "/2f66781e-a1af-4159-bccc-5b52a490afb6/80a1dfcd-7697-4d3a-b862-6f8977c64ed2/d589d6f2-03b4-410e-8081-b53488f96cb4"
-					(reference "C42")
+					(reference "C47")
 					(unit 1)
 				)
@@
 		(dnp no)
 		(fields_autoplaced yes)
-		(property "Reference" "#PWR0124"
+		(property "Reference" "#PWR0210"
 			(at 172.72 101.6 0)
 			(effects
@@
 			(project "alu"
 				(path "/2f66781e-a1af-4159-bccc-5b52a490afb6/80a1dfcd-7697-4d3a-b862-6f8977c64ed2/d589d6f2-03b4-410e-8081-b53488f96cb4"
-					(reference "#PWR0124")
+					(reference "#PWR0210")
 					(unit 1)
 				)
@@
 		(dnp no)
 		(fields_autoplaced yes)
-		(property "Reference" "#PWR0118"
+		(property "Reference" "#PWR0202"
 			(at 104.14 102.87 0)
 			(effects
@@
 			(project "alu"
 				(path "/2f66781e-a1af-4159-bccc-5b52a490afb6/80a1dfcd-7697-4d3a-b862-6f8977c64ed2/d589d6f2-03b4-410e-8081-b53488f96cb4"
-					(reference "#PWR0118")
+					(reference "#PWR0202")
 					(unit 1)
 				)
@@
 		(dnp no)
 		(fields_autoplaced yes)
-		(property "Reference" "#PWR0125"
+		(property "Reference" "#PWR0211"
 			(at 172.72 154.94 0)
 			(effects
@@
 			(project "alu"
 				(path "/2f66781e-a1af-4159-bccc-5b52a490afb6/80a1dfcd-7697-4d3a-b862-6f8977c64ed2/d589d6f2-03b4-410e-8081-b53488f96cb4"
-					(reference "#PWR0125")
+					(reference "#PWR0211")
 					(unit 1)
 				)
@@
 		(dnp no)
 		(fields_autoplaced yes)
-		(property "Reference" "#PWR0119"
+		(property "Reference" "#PWR0203"
 			(at 104.14 156.21 0)
 			(effects
@@
 			(project "alu"
 				(path "/2f66781e-a1af-4159-bccc-5b52a490afb6/80a1dfcd-7697-4d3a-b862-6f8977c64ed2/d589d6f2-03b4-410e-8081-b53488f96cb4"
-					(reference "#PWR0119")
+					(reference "#PWR0203")
 					(unit 1)
 				)
@@
 		(dnp no)
 		(fields_autoplaced yes)
-		(property "Reference" "U48"
+		(property "Reference" "U49"
 			(at 174.8633 100.33 0)
 			(effects
@@
 			(project "alu"
 				(path "/2f66781e-a1af-4159-bccc-5b52a490afb6/80a1dfcd-7697-4d3a-b862-6f8977c64ed2/d589d6f2-03b4-410e-8081-b53488f96cb4"
-					(reference "U48")
+					(reference "U49")
 					(unit 1)
 				)
@@
 		(dnp no)
 		(fields_autoplaced yes)
-		(property "Reference" "#PWR0254"
+		(property "Reference" "#PWR0205"
 			(at 149.86 49.53 0)
 			(effects
@@
 			(project "alu"
 				(path "/2f66781e-a1af-4159-bccc-5b52a490afb6/80a1dfcd-7697-4d3a-b862-6f8977c64ed2/d589d6f2-03b4-410e-8081-b53488f96cb4"
-					(reference "#PWR0254")
+					(reference "#PWR0205")
 					(unit 1)
 				)
@@
 		(dnp no)
 		(fields_autoplaced yes)
-		(property "Reference" "#PWR0115"
+		(property "Reference" "#PWR0199"
 			(at 87.63 152.4 0)
 			(effects
@@
 			(project "alu"
 				(path "/2f66781e-a1af-4159-bccc-5b52a490afb6/80a1dfcd-7697-4d3a-b862-6f8977c64ed2/d589d6f2-03b4-410e-8081-b53488f96cb4"
-					(reference "#PWR0115")
+					(reference "#PWR0199")
 					(unit 1)
 				)
@@
 		(dnp no)
 		(fields_autoplaced yes)
-		(property "Reference" "#PWR0252"
+		(property "Reference" "#PWR0197"
 			(at 81.28 114.3 0)
 			(effects
@@
 			(project "alu"
 				(path "/2f66781e-a1af-4159-bccc-5b52a490afb6/80a1dfcd-7697-4d3a-b862-6f8977c64ed2/d589d6f2-03b4-410e-8081-b53488f96cb4"
-					(reference "#PWR0252")
+					(reference "#PWR0197")
 					(unit 1)
 				)
@@
 		(dnp no)
 		(fields_autoplaced yes)
-		(property "Reference" "#PWR0121"
+		(property "Reference" "#PWR0207"
 			(at 156.21 151.13 0)
 			(effects
@@
 			(project "alu"
 				(path "/2f66781e-a1af-4159-bccc-5b52a490afb6/80a1dfcd-7697-4d3a-b862-6f8977c64ed2/d589d6f2-03b4-410e-8081-b53488f96cb4"
-					(reference "#PWR0121")
+					(reference "#PWR0207")
 					(unit 1)
 				)
@@
 		(dnp no)
 		(fields_autoplaced yes)
-		(property "Reference" "U45"
+		(property "Reference" "U46"
 			(at 106.2833 36.83 0)
 			(effects
@@
 			(project "alu"
 				(path "/2f66781e-a1af-4159-bccc-5b52a490afb6/80a1dfcd-7697-4d3a-b862-6f8977c64ed2/d589d6f2-03b4-410e-8081-b53488f96cb4"
-					(reference "U45")
+					(reference "U46")
 					(unit 1)
 				)
@@
 		(dnp no)
 		(fields_autoplaced yes)
-		(property "Reference" "#PWR0123"
+		(property "Reference" "#PWR0209"
 			(at 172.72 91.44 0)
 			(effects
@@
 			(project "alu"
 				(path "/2f66781e-a1af-4159-bccc-5b52a490afb6/80a1dfcd-7697-4d3a-b862-6f8977c64ed2/d589d6f2-03b4-410e-8081-b53488f96cb4"
-					(reference "#PWR0123")
+					(reference "#PWR0209")
 					(unit 1)
 				)
@@
 		(dnp no)
 		(fields_autoplaced yes)
-		(property "Reference" "C44"
+		(property "Reference" "C49"
 			(at 153.67 38.0999 0)
 			(effects
@@
 			(project "alu"
 				(path "/2f66781e-a1af-4159-bccc-5b52a490afb6/80a1dfcd-7697-4d3a-b862-6f8977c64ed2/d589d6f2-03b4-410e-8081-b53488f96cb4"
-					(reference "C44")
+					(reference "C49")
 					(unit 1)
 				)
@@
 		(dnp no)
 		(fields_autoplaced yes)
-		(property "Reference" "#PWR0120"
+		(property "Reference" "#PWR0206"
 			(at 156.21 87.63 0)
 			(effects
@@
 			(project "alu"
 				(path "/2f66781e-a1af-4159-bccc-5b52a490afb6/80a1dfcd-7697-4d3a-b862-6f8977c64ed2/d589d6f2-03b4-410e-8081-b53488f96cb4"
-					(reference "#PWR0120")
+					(reference "#PWR0206")
 					(unit 1)
 				)
@@
 		(dnp no)
 		(fields_autoplaced yes)
-		(property "Reference" "#PWR0122"
+		(property "Reference" "#PWR0208"
 			(at 172.72 38.1 0)
 			(effects
@@
 			(project "alu"
 				(path "/2f66781e-a1af-4159-bccc-5b52a490afb6/80a1dfcd-7697-4d3a-b862-6f8977c64ed2/d589d6f2-03b4-410e-8081-b53488f96cb4"
-					(reference "#PWR0122")
+					(reference "#PWR0208")
 					(unit 1)
 				)
@@
 		(dnp no)
 		(fields_autoplaced yes)
-		(property "Reference" "U47"
+		(property "Reference" "U48"
 			(at 174.8633 36.83 0)
 			(effects
@@
 			(project "alu"
 				(path "/2f66781e-a1af-4159-bccc-5b52a490afb6/80a1dfcd-7697-4d3a-b862-6f8977c64ed2/d589d6f2-03b4-410e-8081-b53488f96cb4"
-					(reference "U47")
+					(reference "U48")
 					(unit 1)
 				)
@@
 		(dnp no)
 		(fields_autoplaced yes)
-		(property "Reference" "#PWR0117"
+		(property "Reference" "#PWR0201"
 			(at 104.14 91.44 0)
 			(effects
@@
 			(project "alu"
 				(path "/2f66781e-a1af-4159-bccc-5b52a490afb6/80a1dfcd-7697-4d3a-b862-6f8977c64ed2/d589d6f2-03b4-410e-8081-b53488f96cb4"
-					(reference "#PWR0117")
-					(unit 1)
-				)
+					(reference "#PWR0201")
+					(unit 1)
+				)

Commit message: Footprints, PCB update
Added footprints to all components, updated the PCB with the schematic
Parts:
- C46, C47, C48, C49: footprint (none) -> Capacitor_SMD:C_0603_1608Metric
- U46, U47, U48, U49: footprint (none) -> Package_SO:SOIC-16_3.9x9.9mm_P1.27mm
Changed lines of the file:
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@@
 			)
 		)
-		(property "Footprint" ""
+		(property "Footprint" "Package_SO:SOIC-16_3.9x9.9mm_P1.27mm"
 			(at 104.14 124.46 0)
 			(effects
@@
 			)
 		)
-		(property "Footprint" ""
+		(property "Footprint" "Capacitor_SMD:C_0603_1608Metric"
 			(at 149.5552 106.68 0)
 			(effects
@@
 			)
 		)
-		(property "Footprint" ""
+		(property "Footprint" "Capacitor_SMD:C_0603_1608Metric"
 			(at 82.2452 43.18 0)
 			(effects
@@
 			)
 		)
-		(property "Footprint" ""
+		(property "Footprint" "Capacitor_SMD:C_0603_1608Metric"
 			(at 82.2452 107.95 0)
 			(effects
@@
 			)
 		)
-		(property "Footprint" ""
+		(property "Footprint" "Package_SO:SOIC-16_3.9x9.9mm_P1.27mm"
 			(at 172.72 123.19 0)
 			(effects
@@
 			)
 		)
-		(property "Footprint" ""
+		(property "Footprint" "Package_SO:SOIC-16_3.9x9.9mm_P1.27mm"
 			(at 104.14 59.69 0)
 			(effects
@@
 			)
 		)
-		(property "Footprint" ""
+		(property "Footprint" "Capacitor_SMD:C_0603_1608Metric"
 			(at 150.8252 43.18 0)
 			(effects
@@
 			)
 		)
-		(property "Footprint" ""
+		(property "Footprint" "Package_SO:SOIC-16_3.9x9.9mm_P1.27mm"
 			(at 172.72 59.69 0)
 			(effects

Commit message: ALU Pcb update
Parts:
- C46, C47, C48, C49: value 10n -> 100nF; footprint Capacitor_SMD:C_0603_1608Metric -> Capacitor_SMD:C_0402_1005Metric
- U46, U47, U48, U49: value 74LS257 -> 74257
