File: PCB/Kicad/alu/alu.kicad_pcb (KiCad board)
At the start: 2 copper layers, 226 parts, among them J1 Conn_02x10_Odd_Even, J2 Conn_02x10_Odd_Even, U1 74LS08, U10 74LS08, U11 74LS86, U12 74LS86, U13 74LS86, U14 74LS86, U15 74LS04, U16 74LS04, U17 74LS86, U18 74LS86, U19 74LS86, U2 74LS04, U20 74LS283, U21 74LS283, U22 74LS86, U23 74LS86, U24 74LS283, U25 74LS283, U26 74LS257, U27 74LS257, U28 74LS257, U29 74LS257, U3 74LS32, U30 74LS257, U31 74LS257, U32 74LS257, U33 74LS257, U34 74LS257, U35 74LS257, U36 74LS257, U37 74LS257, U38 74LS257, U39 74LS257, U4 74LS32, U40 74LS257, U41 74LS257, U42 74LS257, U43 74LS257, U44 74LS257, U45 74LS257, U46 74LS257, U47 74LS257, U48 74LS257, U49 74LS257, U5 74LS32, U50 74LS377, U51 74LS377, U52 74LS245, U53 74LS245, U54 74LS139, U55 74LS32, U56 74LS32, U57 74LS32, U58 74LS377, U59 74LS377, U6 74LS32, U60 74LS245, U61 74LS245, U62 74LS245, U63 74LS245, U64 74LS245, U65 74LS245, U66 74LS245, U67 74LS245, U68 74LS245, U69 74LS245, U7 74LS08, U70 74LS32, U71 74LS86, U72 74LS32, U73 74LS04, U74 74LS32, U75 74LS08, U8 74LS08, U9 74LS08

Commit message: Update PCB
Parts:
- moved U75 89.2 mm to (256.4, 25.8)
- moved C17 89.2 mm to (159.6, 21.8)
- moved C18 89.2 mm to (159.6, 24.3)
- moved C19 89.2 mm to (159.6, 26.8)
- moved C20 89.2 mm to (159.6, 29.3)
- moved C21 89.2 mm to (159.6, 31.9)
- moved C22 89.2 mm to (159.6, 34.4)
- moved C23 89.2 mm to (159.6, 36.9)
- moved C24 89.2 mm to (159.6, 39.4)
- moved C25 89.2 mm to (159.6, 41.9)
- moved C26 89.2 mm to (159.6, 101.6)
- moved C27 89.2 mm to (159.6, 104.1)
- moved C28 89.2 mm to (159.6, 106.6)
- moved C29 89.2 mm to (159.6, 109.1)
- moved C34 89.2 mm to (159.6, 79.2)
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
Commit message: ALU Pcb update
Parts:
- added H1: MountingHole_Pad, MountingHole:MountingHole_2.2mm_M2_DIN965_Pad, F.Cu at (23.0, 23.0)
- added H2: MountingHole_Pad, MountingHole:MountingHole_2.2mm_M2_DIN965_Pad, F.Cu at (217.0, 23.0)
- added H3: MountingHole_Pad, MountingHole:MountingHole_2.2mm_M2_DIN965_Pad, F.Cu at (217.0, 117.0)
- added H4: MountingHole_Pad, MountingHole:MountingHole_2.2mm_M2_DIN965_Pad, F.Cu at (23.0, 117.0)
- C1, C10, C11, C12, C13, C14, C15, C16, C17, C18, C19, C2, C20, C21, C22, C23, C24, C25, C26, C27, C28, C29, C3, C30, C31, C32, C33, C34, C35, C36, C37, C38, C39, C4, C40, C41, C42, C43, C44, C45, C46, C47, C48, C49, C5, C50, C51, C52, C53, C54, C55, C56, C57, C58, C59, C6, C60, C61, C62, C63, C64, C65, C66, C67, C68, C69, C7, C70, C71, C72, C73, C74, C75, C8, C9: value 10n -> 100nF; footprint Capacitor_SMD:C_0603_1608Metric -> Capacitor_SMD:C_0402_1005Metric
- D1: value Green LED -> green
- D2, D3, D4, D5: value Yellow LED -> Yellow
- J1, J2: value Conn_02x10_Odd_Even -> out; footprint Connector_PinHeader_2.54mm:PinHeader_2x10_P2.54mm_Horizontal -> mALUch_lib:PinHeader_2x10_P2.54mm_Horizontal
- U1, U10, U7, U75, U8, U9: value 74LS08 -> 7408; footprint Package_SO:SOIC-14_3.9x8.7mm_P1.27mm -> Package_SO:SO-14_3.9x8.65mm_P1.27mm
- U11, U12, U13, U14, U17, U18, U19, U22, U23, U71: value 74LS86 -> 7486; footprint Package_SO:SOIC-14_3.9x8.7mm_P1.27mm -> Package_SO:SO-14_3.9x8.65mm_P1.27mm
- U15, U16, U2, U73: value 74LS04 -> 7404; footprint Package_SO:SOIC-14_3.9x8.7mm_P1.27mm -> Package_SO:SO-14_3.9x8.65mm_P1.27mm
- U20, U21, U24, U25: value 74LS283 -> 74283
- U26, U27, U28, U29, U30, U31, U32, U33, U34, U35, U36, U37, U38, U39, U40, U41, U42, U43, U44, U45, U46, U47, U48, U49: value 74LS257 -> 74257
- U3, U4, U5, U55, U56, U57, U6, U70, U72, U74: value 74LS32 -> 7432; footprint Package_SO:SOIC-14_3.9x8.7mm_P1.27mm -> Package_SO:SO-14_3.9x8.65mm_P1.27mm
- U50, U51, U58, U59: value 74LS377 -> 74377; footprint Package_SO:SOIC-20W_7.5x12.8mm_P1.27mm -> Package_SO:SSOP-20_5.3x7.2mm_P0.65mm
- U52, U53, U60, U61, U62, U63, U64, U65, U66, U67, U68, U69: value 74LS245 -> 74245; footprint Package_SO:SOIC-20W_7.5x12.8mm_P1.27mm -> Package_SO:TSSOP-20_4.4x6.5mm_P0.65mm
- U54: value 74LS139 -> 74139
- moved C68 181.1 mm to (59.1, 93.5)
- moved C69 181.1 mm to (59.1, 96.0)
- moved U68 181.1 mm to (63.5, 85.0)
- moved U69 181.1 mm to (76.4, 85.0)
- moved C60 172.6 mm to (59.1, 115.0)
- moved C61 172.6 mm to (59.1, 117.5)
- moved U60 172.6 mm to (63.5, 106.5)
- moved U61 172.6 mm to (76.4, 106.5)
- moved C66 167.5 mm to (85.8, 0.10)
- moved C67 167.5 mm to (85.8, 2.62)
- moved U66 167.5 mm to (90.2, -8.32)
- moved U67 167.5 mm to (103.1, -8.32)
- moved R21 160.8 mm to (79.4, 35.1)
- moved R20 158.8 mm to (79.4, 33.1)
- moved R19 156.9 mm to (79.4, 31.2)
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Connections:
- J1 pad 11: /D11 -> /D12
- J1 pad 13: /D10 -> /D13
- J1 pad 14: /OP1 -> /OP2
- J1 pad 15: /D9 -> /D14
- J1 pad 17: /D8 -> /D15
- J1 pad 18: /OP0 -> /OP3
- J1 pad 3: /D15 -> /D8
- J1 pad 4: /OP3 -> /OP0
- J1 pad 5: /D14 -> /D9
- J1 pad 7: /D13 -> /D10
- J1 pad 8: /OP2 -> /OP1
- J1 pad 9: /D12 -> /D11
- J2 pad 10: /FC -> /FZ
- J2 pad 11: /D3 -> /D4
- J2 pad 12: /FZ -> /FC
- J2 pad 13: /D2 -> /D5
- J2 pad 15: /D1 -> /D6
- J2 pad 16: GND -> /FO
- J2 pad 17: /D0 -> /D7
- J2 pad 18: /CLK -> /D15
- J2 pad 3: /D7 -> /D0
- J2 pad 4: /D15 -> /CLK
- J2 pad 5: /D6 -> /D1
- J2 pad 6: /FO -> GND
- J2 pad 7: /D5 -> /D2
- J2 pad 9: /D4 -> /D3
- U23 pad 12: unconnected-(U23-Pad12) -> VCC
- U23 pad 13: unconnected-(U23-Pad13) -> VCC
- U57 pad 10: unconnected-(U57-Pad10) -> VCC
- U57 pad 12: unconnected-(U57-Pad12) -> VCC
- U57 pad 13: unconnected-(U57-Pad13) -> VCC
- U57 pad 9: unconnected-(U57-Pad9) -> VCC
- U73 pad 13: unconnected-(U73-Pad13) -> VCC
Other:
- board outline added: 200 x 100 mm

Commit message: alu board adjustement
Parts:
- moved U23 89.3 mm to (157.0, 69.8)
- moved U41 89.3 mm to (160.5, 105.2)
- moved U14 89.3 mm to (160.5, 128.2)
- moved H3 78.1 mm to (167.0, 177.0)
- moved C3 74.0 mm to (93.5, 141.9)
- moved C30 74.0 mm to (93.5, 94.6)
- moved C7 74.0 mm to (93.5, 119.5)
- moved D20 74.0 mm to (38.0, 102.6)
- moved R16 74.0 mm to (47.3, 101.1)
- moved R30 74.0 mm to (47.3, 129.2)
- moved R33 74.0 mm to (47.3, 135.1)
- moved U52 74.0 mm to (133.8, 156.6)
- moved U53 74.0 mm to (146.7, 156.6)
- moved U64 74.0 mm to (133.8, 135.1)
- moved U65 74.0 mm to (146.7, 135.1)
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Other:
- board size 200 x 100 mm -> 150 x 150 mm

Commit message: PCB
Parts:
- moved C70 291.6 mm to (343.1, -18.1), turned to 180 degrees
- moved U70 291.0 mm to (348.6, -14.2)
- moved C71 290.0 mm to (343.1, -6.41), turned to 180 degrees
- moved C72 288.7 mm to (343.1, 5.24), turned to 180 degrees
- moved C73 287.7 mm to (343.1, 16.9), turned to 180 degrees
- moved C74 287.0 mm to (343.1, 28.6), turned to 180 degrees
- moved C75 286.6 mm to (343.1, 40.2), turned to 180 degrees
- moved U71 280.6 mm to (348.6, -2.52)
- moved U72 270.7 mm to (348.6, 9.13)
- moved U73 261.2 mm to (348.6, 20.8)
- moved U74 252.1 mm to (348.6, 32.4)
- moved U54 250.2 mm to (345.3, 149.0)
- moved U55 249.6 mm to (345.3, 160.2)
- moved U75 243.5 mm to (348.6, 44.1)
- moved U56 241.6 mm to (345.3, 171.4)
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Connections:
- U21 pad 12: /A_BUS0 -> /A_BUS4
- U21 pad 14: /A_BUS1 -> /A_BUS5
- U21 pad 3: /A_BUS2 -> /A_BUS6
- U21 pad 5: /A_BUS3 -> /A_BUS7
- U24 pad 12: /A_BUS0 -> /A_BUS8
- U24 pad 14: /A_BUS1 -> /A_BUS9
- U24 pad 3: /A_BUS2 -> /A_BUS10
- U24 pad 5: /A_BUS3 -> /A_BUS11
- U25 pad 12: /A_BUS0 -> /A_BUS12
- U25 pad 14: /A_BUS1 -> /A_BUS13
- U25 pad 3: /A_BUS2 -> /A_BUS14
- U25 pad 5: /A_BUS3 -> /A_BUS15
Other:
- copper layers 2 -> 6

Commit message: Stuff and layout
Parts:
- moved U70 458.9 mm to (-108.4, 26.8)
- moved U71 449.5 mm to (-99.9, 26.8)
- moved U72 440.5 mm to (-91.5, 26.8)
- moved U73 431.7 mm to (-83.0, 26.8)
- moved U74 423.3 mm to (-74.6, 26.8)
- moved U75 415.1 mm to (-66.1, 26.8)
- moved C57 381.4 mm to (63.3, -83.7), turned to 0 degrees
- moved C56 375.1 mm to (63.3, -85.7), turned to 0 degrees
- moved C55 368.9 mm to (63.3, -87.6), turned to 0 degrees
- moved C53 340.4 mm to (67.3, -77.8)
- moved C52 339.5 mm to (67.3, -79.7), turned to 0 degrees
- moved C75 326.2 mm to (42.9, -87.7), turned to 0 degrees
- moved C74 322.5 mm to (42.9, -89.6), turned to 0 degrees
- moved C73 319.1 mm to (42.9, -91.6), turned to 0 degrees
- moved C72 316.0 mm to (42.9, -93.6), turned to 0 degrees
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Connections:
- U21 pad 12: /A_BUS4 -> /A_BUS0
- U21 pad 14: /A_BUS5 -> /A_BUS1
- U21 pad 3: /A_BUS6 -> /A_BUS2
- U21 pad 5: /A_BUS7 -> /A_BUS3
- U24 pad 12: /A_BUS8 -> /A_BUS0
- U24 pad 14: /A_BUS9 -> /A_BUS1
- U24 pad 3: /A_BUS10 -> /A_BUS2
- U24 pad 5: /A_BUS11 -> /A_BUS3
- U25 pad 12: /A_BUS12 -> /A_BUS0
- U25 pad 14: /A_BUS13 -> /A_BUS1
- U25 pad 3: /A_BUS14 -> /A_BUS2
- U25 pad 5: /A_BUS15 -> /A_BUS3
- U3 pad 11: /OR3 -> /OR1
- U3 pad 12: /A_BUS3 -> /B_BUS1
- U3 pad 13: /B_BUS3 -> /A_BUS1
- U3 pad 4: /A_BUS1 -> /A_BUS3
- U3 pad 5: /B_BUS1 -> /B_BUS3
- U3 pad 6: /OR1 -> /OR3
Routing:
- net /OR0: track 0.00 -> 17.3 mm
- net /A_BUS1: track 0.00 -> 15.4 mm, vias 0 -> 1
- net /OR1: track 0.00 -> 12.1 mm
- net /A_BUS0: track 0.00 -> 12.0 mm, vias 0 -> 1
- net /B_BUS1: track 0.00 -> 11.7 mm, vias 0 -> 1
- net /B_BUS0: track 0.00 -> 8.35 mm, vias 0 -> 1
- net /OR3: track 0.00 -> 1.45 mm
