File: PCB/Kicad/control_unit/ControlUnit.kicad_sch (KiCad schematic)
At the start: 3 parts, among them SW1 SW_DPST_x2, U4 74LS08

Commit message: control unit schematic
Parts:
- removed SW1: SW_DPST_x2, symbol Switch:SW_DPST_x2
- added SW1: SW_Push, Button_Switch_THT:SW_PUSH_6mm_H4.3mm, symbol Switch:SW_Push
- added Ubc3: 74LS04, Package_SO:SOIC-14_3.9x8.7mm_P1.27mm, symbol 74xx:74LS04
- Rcuc1: renamed from R33; footprint (none) -> Resistor_SMD:R_0402_1005Metric
- U4: footprint (none) -> Package_SO:SOIC-14_3.9x8.7mm_P1.27mm
Connections:
- net enter_int is gone; now on net mask_save: U4.3
- net leaveint is gone; now on net mask_restore: U4.11
- net VCC: now also SW1.1
- net next_instr: now also Ubc3.11
- net rst: now also SW1.2
- net ~{next_instr}: now also Ubc3.10
- no-connect marks 5 -> 7
Other:
- added sheet tempreg (reg16b.kicad_sch)
- sheet DecodeRom ports: added isstack, next_instr, regds, ~{instr_load}, ~{tempregwe}; removed instr_load, nextinstr, tempregwe
- sheet buscntrl ports: added tempreg[15..0]; removed none
- sheet cyclereg ports: added rst; removed ~{rst}
- sheet flags ports: added enterint, should_jump; removed shouldjump
- note added: "for whatever reason, few connections have to be wires instead of labels"
- company: (none) -> AGH Logic Unit
- title: (none) -> Control Unit Core

Commit message: control unit update
Parts:
- added C1: 100nF, Capacitor_SMD:C_0402_1005Metric, symbol Device:C
- U4: value 74LS08 -> 7408; footprint Package_SO:SOIC-14_3.9x8.7mm_P1.27mm -> Package_SO:SO-14_3.9x8.65mm_P1.27mm
- Ubc3: value 74LS04 -> 7404; footprint Package_SO:SOIC-14_3.9x8.7mm_P1.27mm -> Package_SO:SO-14_3.9x8.65mm_P1.27mm
Connections:
- net GND: now also C1.2
- net VCC: now also C1.1
