File: PCB/Kicad/control_unit/buscntrl.kicad_sch (KiCad schematic)
At the start: 3 parts, among them U31 74LS139, U38 74LS04, U43 74LS139

Commit message: control unit schematic
Parts:
- removed unit 6 of U38
- removed unit 5 of U38
- added unit 6 of Ubc3
- Ubc1: renamed from U31; footprint (none) -> Package_SO:SOIC-14_3.9x8.7mm_P1.27mm
- Ubc2: renamed from U43; footprint (none) -> Package_SO:SOIC-14_3.9x8.7mm_P1.27mm
- Ubc3: renamed from U38; footprint (none) -> Package_SO:SOIC-14_3.9x8.7mm_P1.27mm
Connections:
- net VCC: now also Ubc3.5, Ubc3.9, Ubc3.13
- net alusrc0: now also Ubc1.14 (A0); no longer Ubc1.13 (A1)
- net alusrc1: now also Ubc1.13 (A1); no longer Ubc1.14 (A0)
- net srcsrc: no longer Ubc1.11 (O1)
- net ~{src_regbusen}: no longer Ubc1.10 (O2)
- new net ~{alu_membusen}: Ubc1.11 (O1)
- new net ~{alu_regbusen}: Ubc1.10 (O2)
- no-connect marks 14 -> 18
Other:
- company: (none) -> AGH Logic Unit
- title: (none) -> Bus Control

Commit message: control unit update
Parts:
- added Cbc1, Cbc2, Cbc3: 100nF, Capacitor_SMD:C_0402_1005Metric, symbol Device:C
- Ubc1, Ubc2: value 74LS139 -> 74139; footprint Package_SO:SOIC-14_3.9x8.7mm_P1.27mm -> Package_SO:SOIC-16_3.9x9.9mm_P1.27mm
- Ubc3: value 74LS04 -> 7404; footprint Package_SO:SOIC-14_3.9x8.7mm_P1.27mm -> Package_SO:SO-14_3.9x8.65mm_P1.27mm
Connections:
- net GND: now also Cbc1.2, Cbc2.2, Cbc3.2
- net VCC: now also Cbc1.1, Cbc2.1, Cbc3.1
