File: PCB/Kicad/control_unit/instructionregister.kicad_sch (KiCad schematic)
At the start: 5 parts, among them U12 74LS257

Commit message: control unit schematic
Parts:
- Rir1: renamed from R34; footprint (none) -> Resistor_SMD:R_0402_1005Metric
- Rir2: renamed from R35; footprint (none) -> Resistor_SMD:R_0402_1005Metric
- Rir3: renamed from R36; footprint (none) -> Resistor_SMD:R_0402_1005Metric
- Rir4: renamed from R37; footprint (none) -> Resistor_SMD:R_0402_1005Metric
- Uinsr1: renamed from U12; footprint (none) -> Package_SO:SOIC-14_3.9x8.7mm_P1.27mm
Connections:
- net regid0: no longer Rir2.1, Rir3.1, Rir4.1
- net regid1: now also Rir2.1
- net regid2: now also Rir3.1
- net regid3: now also Rir4.1
Other:
- company: (none) -> AGH Logic Unit
- title: (none) -> Instruction Register
Changed lines of the file:
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@@
 	(generator_version "9.0")
 	(paper "A4")
+	(title_block
+		(title "Instruction Register")
+		(date "2026-03-11")
+		(rev "1")
+		(company "AGH Logic Unit")
+		(comment 1 "NOT Spice checked")
+		(comment 2 "review: -")
+		(comment 3 "author: Hubert Wójcik")
+	)
 	(text "when isstack goes high, mux is disconnected and pullup/down resistors act"
 		(exclude_from_sim no)
@@
 		(at 227.33 86.36)
 	)
+	(bus_entry
+		(at 160.02 80.01)
+		(size 2.54 -2.54)
+		(stroke
+			(width 0)
+			(type default)
+		)
+	)
 	(bus
 		(pts
@@
 	(bus
 		(pts
+			(xy 160.02 80.01) (xy 161.925 80.01)
+		)
+		(stroke
+			(width 0)
+			(type default)
+		)
+	)
+	(bus
+		(pts
 			(xy 104.14 80.01) (xy 118.11 80.01)
 		)
@@
 	(wire
 		(pts
+			(xy 162.56 76.835) (xy 175.26 76.835)
+		)
+		(stroke
+			(width 0)
+			(type default)
+		)
+	)
+	(wire
+		(pts
 			(xy 186.69 134.62) (xy 207.01 134.62)
 		)
@@
 		)
 	)
+	(wire
+		(pts
+			(xy 162.56 77.47) (xy 162.56 76.835)
+		)
+		(stroke
+			(width 0)
+			(type default)
+		)
+	)
+	(bus
+		(pts
+			(xy 157.48 80.01) (xy 160.02 80.01)
+		)
+		(stroke
+			(width 0)
+			(type default)
+		)
+	)
 	(label "instr[15..12]"
 		(at 198.12 69.85 180)
@@
 		)
 	)
-	(label "regid0"
+	(label "regid2"
 		(at 243.84 142.24 0)
 		(effects
@@
 		)
 	)
-	(label "regid0"
+	(label "regid3"
 		(at 254 142.24 0)
 		(effects
@@
 	)
 	(label "instr[10..8]"
-		(at 198.12 74.93 180)
+		(at 198.12 83.82 180)
 		(effects
 			(font
@@
 		)
 	)
+	(label "instr11"
+		(at 164.465 76.835 0)
+		(effects
+			(font
+				(size 1.27 1.27)
+			)
+			(justify left bottom)
+		)
+	)
 	(label "instr4"
 		(at 161.29 142.24 180)
@@
 	)
 	(label "instr[15..0]"
-		(at 157.48 80.01 0)
+		(at 161.925 80.01 0)
 		(effects
 			(font
@@
 		)
 	)
-	(label "instr11"
-		(at 198.12 72.39 180)
-		(effects
-			(font
-				(size 1.27 1.27)
-			)
-			(justify right bottom)
-		)
-	)
-	(label "regid0"
+	(label "regid1"
 		(at 233.68 142.24 0)
 		(effects
@@
 	(hierarchical_label "funct[2..0]"
 		(shape output)
-		(at 198.12 74.93 0)
+		(at 198.12 83.82 0)
 		(effects
 			(font
@@
 	(hierarchical_label "isimm"
 		(shape output)
-		(at 198.12 72.39 0)
+		(at 175.26 76.835 0)
 		(effects
 			(font
@@
 		(dnp no)
 		(fields_autoplaced yes)
-		(property "Reference" "R35"
+		(property "Reference" "Rir2"
 			(at 236.22 137.1599 0)
 			(effects
@@
 			)
 		)
-		(property "Footprint" ""
+		(property "Footprint" "Resistor_SMD:R_0402_1005Metric"
 			(at 235.458 138.43 90)
 			(effects
@@
 			(project "control_unit"
 				(path "/dccec861-b967-466c-843e-d6d1ad6064ce/a601307c-be83-4128-aa2e-f19df4dff19c/8dd513a7-9e42-4785-8158-c05d517a1257"
-					(reference "R35")
+					(reference "Rir2")
 					(unit 1)
 				)
@@
 		(dnp no)
 		(fields_autoplaced yes)
-		(property "Reference" "R37"
+		(property "Reference" "Rir4"
 			(at 256.54 144.7799 0)
 			(effects
@@
 			)
 		)
-		(property "Footprint" ""
+		(property "Footprint" "Resistor_SMD:R_0402_1005Metric"
 			(at 252.222 146.05 90)
 			(effects
@@
 			(project "control_unit"
 				(path "/dccec861-b967-466c-843e-d6d1ad6064ce/a601307c-be83-4128-aa2e-f19df4dff19c/8dd513a7-9e42-4785-8158-c05d517a1257"
-					(reference "R37")
+					(reference "Rir4")
 					(unit 1)
 				)
@@
 		(dnp no)
 		(fields_autoplaced yes)
-		(property "Reference" "R36"
+		(property "Reference" "Rir3"
 			(at 246.38 144.7799 0)
 			(effects
@@
 			)
 		)
-		(property "Footprint" ""
+		(property "Footprint" "Resistor_SMD:R_0402_1005Metric"
 			(at 242.062 146.05 90)
 			(effects
@@
 			(project "control_unit"
 				(path "/dccec861-b967-466c-843e-d6d1ad6064ce/a601307c-be83-4128-aa2e-f19df4dff19c/8dd513a7-9e42-4785-8158-c05d517a1257"
-					(reference "R36")
+					(reference "Rir3")
 					(unit 1)
 				)
@@
 		(dnp no)
 		(fields_autoplaced yes)
-		(property "Reference" "U12"
+		(property "Reference" "Uinsr1"
 			(at 176.1333 111.76 0)
 			(effects
@@
 			)
 		)
-		(property "Footprint" ""
+		(property "Footprint" "Package_SO:SOIC-14_3.9x8.7mm_P1.27mm"
 			(at 173.99 134.62 0)
 			(effects
@@
 			(project ""
 				(path "/dccec861-b967-466c-843e-d6d1ad6064ce/a601307c-be83-4128-aa2e-f19df4dff19c/8dd513a7-9e42-4785-8158-c05d517a1257"
-					(reference "U12")
+					(reference "Uinsr1")
 					(unit 1)
 				)
@@
 		(dnp no)
 		(fields_autoplaced yes)
-		(property "Reference" "R34"
+		(property "Reference" "Rir1"
 			(at 226.06 144.7799 0)
 			(effects
@@
 			)
 		)
-		(property "Footprint" ""
+		(property "Footprint" "Resistor_SMD:R_0402_1005Metric"
 			(at 221.742 146.05 90)
 			(effects
@@
 			(project "control_unit"
 				(path "/dccec861-b967-466c-843e-d6d1ad6064ce/a601307c-be83-4128-aa2e-f19df4dff19c/8dd513a7-9e42-4785-8158-c05d517a1257"
-					(reference "R34")
+					(reference "Rir1")
 					(unit 1)
 				)

Commit message: control unit update
Parts:
- added Cinsr1: 100nF, Capacitor_SMD:C_0402_1005Metric, symbol Device:C
- Uinsr1: value 74LS257 -> 74257; footprint Package_SO:SOIC-14_3.9x8.7mm_P1.27mm -> Package_SO:SOIC-16_3.9x9.9mm_P1.27mm
Connections:
- net GND: now also Cinsr1.2
- net VCC: now also Cinsr1.1
