File: PCB/Kicad/control_unit/ip.kicad_sch (KiCad schematic)
At the start: 5 parts, among them U10 74LS283, U11 74LS283, U20 ATF16V8Bxx-xxPU, U8 74LS283, U9 74LS283

Commit message: control unit schematic
Parts:
- Uip1: renamed from U8; footprint (none) -> Package_SO:SOIC-14_3.9x8.7mm_P1.27mm
- Uip2: renamed from U9; footprint (none) -> Package_SO:SOIC-14_3.9x8.7mm_P1.27mm
- Uip3: renamed from U10; footprint (none) -> Package_SO:SOIC-14_3.9x8.7mm_P1.27mm
- Uip4: renamed from U11; footprint (none) -> Package_SO:SOIC-14_3.9x8.7mm_P1.27mm
- renumbered U20 to Uip5
Connections:
- net GND: now also Uip5.6 (I5), Uip5.7 (I6), Uip5.8 (I7)
- no-connect marks 1 -> 5
Other:
- note added: "let's REALLY hope this works, otherwise oopsie woopsie"
- company: (none) -> AGH Logic Unit
- title: (none) -> Instruction Pointer
Changed lines of the file:
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@@
 	(generator_version "9.0")
 	(paper "A4")
+	(title_block
+		(title "Instruction Pointer")
+		(date "2026-03-11")
+		(rev "1")
+		(company "AGH Logic Unit")
+		(comment 1 "NOT Spice checked")
+		(comment 2 "review: -")
+		(comment 3 "author: Hubert Wójcik")
+	)
+	(text "let's REALLY hope this works, otherwise oopsie woopsie"
+		(exclude_from_sim no)
+		(at 121.92 22.86 0)
+		(effects
+			(font
+				(size 1.27 1.27)
+			)
+		)
+	)
 	(junction
 		(at 19.05 175.26)
@@
 	)
 	(junction
+		(at 111.76 55.88)
+		(diameter 0)
+		(color 0 0 0 0)
+	)
+	(junction
 		(at 251.46 130.81)
 		(diameter 0)
@@
 	)
 	(junction
+		(at 111.76 58.42)
+		(diameter 0)
+		(color 0 0 0 0)
+	)
+	(junction
 		(at 133.35 175.26)
 		(diameter 0)
@@
 		(at 158.75 165.1)
 	)
+	(no_connect
+		(at 132.08 50.8)
+	)
+	(no_connect
+		(at 132.08 58.42)
+	)
+	(no_connect
+		(at 132.08 55.88)
+	)
+	(no_connect
+		(at 132.08 53.34)
+	)
 	(wire
 		(pts
@@
 		)
 	)
-	(wire
+	(bus
 		(pts
-			(xy 82.55 165.1) (xy 90.17 165.1)
+			(xy 251.46 138.43) (xy 254 138.43)
 		)
 		(stroke
@@
 	(wire
 		(pts
-			(xy 19.05 175.26) (xy 19.05 177.8)
+			(xy 82.55 165.1) (xy 90.17 165.1)
 		)
 		(stroke
@@
 	(wire
 		(pts
-			(xy 95.25 175.26) (xy 95.25 177.8)
+			(xy 19.05 175.26) (xy 19.05 177.8)
 		)
 		(stroke
@@
 	(wire
 		(pts
-			(xy 251.46 113.03) (xy 254 113.03)
+			(xy 95.25 175.26) (xy 95.25 177.8)
 		)
 		(stroke
@@
 	(wire
 		(pts
-			(xy 251.46 130.81) (xy 254 130.81)
+			(xy 251.46 113.03) (xy 254 113.03)
 		)
 		(stroke
@@
 	(wire
 		(pts
-			(xy 251.46 135.89) (xy 254 135.89)
+			(xy 251.46 130.81) (xy 254 130.81)
 		)
 		(stroke
@@
 	(wire
 		(pts
-			(xy 251.46 138.43) (xy 254 138.43)
+			(xy 251.46 135.89) (xy 254 135.89)
 		)
 		(stroke
@@
 	(wire
 		(pts
+			(xy 95.25 58.42) (xy 111.76 58.42)
+		)
+		(stroke
+			(width 0)
+			(type default)
+		)
+	)
+	(wire
+		(pts
+			(xy 111.76 55.88) (xy 111.76 58.42)
+		)
+		(stroke
+			(width 0)
+			(type default)
+		)
+	)
+	(wire
+		(pts
 			(xy 251.46 118.11) (xy 254 118.11)
 		)
@@
 	(wire
 		(pts
+			(xy 111.76 53.34) (xy 111.76 55.88)
+		)
+		(stroke
+			(width 0)
+			(type default)
+		)
+	)
+	(wire
+		(pts
 			(xy 251.46 107.95) (xy 254 107.95)
 		)
@@
 		)
 	)
-	(wire
-		(pts
-			(xy 81.28 30.48) (xy 77.47 30.48)
-		)
-		(stroke
-			(width 0)
-			(type default)
-		)
-	)
 	(bus
 		(pts
@@
 	(hierarchical_label "ip[15..0]"
 		(shape output)
-		(at 81.28 30.48 0)
+		(at 77.47 30.48 0)
 		(effects
 			(font
@@
 		(dnp no)
 		(fields_autoplaced yes)
-		(property "Reference" "U8"
+		(property "Reference" "Uip1"
 			(at 33.8933 144.78 0)
 			(effects
@@
 			)
 		)
-		(property "Footprint" ""
+		(property "Footprint" "Package_SO:SOIC-14_3.9x8.7mm_P1.27mm"
 			(at 31.75 165.1 0)
 			(effects
@@
 			(project ""
 				(path "/dccec861-b967-466c-843e-d6d1ad6064ce/a601307c-be83-4128-aa2e-f19df4dff19c/c0031539-c4c3-432d-9a69-ce5a0aa72fa8"
-					(reference "U8")
+					(reference "Uip1")
 					(unit 1)
 				)
@@
 		(dnp no)
 		(fields_autoplaced yes)
-		(property "Reference" "U20"
+		(property "Reference" "Uip5"
 			(at 124.0633 33.02 0)
 			(effects
@@
 			(project ""
 				(path "/dccec861-b967-466c-843e-d6d1ad6064ce/a601307c-be83-4128-aa2e-f19df4dff19c/c0031539-c4c3-432d-9a69-ce5a0aa72fa8"
-					(reference "U20")
+					(reference "Uip5")
 					(unit 1)
 				)
@@
 		(dnp no)
 		(fields_autoplaced yes)
-		(property "Reference" "U10"
+		(property "Reference" "Uip3"
 			(at 110.0933 144.78 0)
 			(effects
@@
 			)
 		)
-		(property "Footprint" ""
+		(property "Footprint" "Package_SO:SOIC-14_3.9x8.7mm_P1.27mm"
 			(at 107.95 165.1 0)
 			(effects
@@
 			(project "control_unit"
 				(path "/dccec861-b967-466c-843e-d6d1ad6064ce/a601307c-be83-4128-aa2e-f19df4dff19c/c0031539-c4c3-432d-9a69-ce5a0aa72fa8"
-					(reference "U10")
+					(reference "Uip3")
 					(unit 1)
 				)
@@
 		(dnp no)
 		(fields_autoplaced yes)
-		(property "Reference" "U11"
+		(property "Reference" "Uip4"
 			(at 148.1933 144.78 0)
 			(effects
@@
 			)
 		)
-		(property "Footprint" ""
+		(property "Footprint" "Package_SO:SOIC-14_3.9x8.7mm_P1.27mm"
 			(at 146.05 165.1 0)
 			(effects
@@
 			(project "control_unit"
 				(path "/dccec861-b967-466c-843e-d6d1ad6064ce/a601307c-be83-4128-aa2e-f19df4dff19c/c0031539-c4c3-432d-9a69-ce5a0aa72fa8"
-					(reference "U11")
+					(reference "Uip4")
 					(unit 1)
 				)
@@
 		(dnp no)
 		(fields_autoplaced yes)
-		(property "Reference" "U9"
+		(property "Reference" "Uip2"
 			(at 71.9933 144.78 0)
 			(effects
@@
 			)
 		)
-		(property "Footprint" ""
+		(property "Footprint" "Package_SO:SOIC-14_3.9x8.7mm_P1.27mm"
 			(at 69.85 165.1 0)
 			(effects
@@
 			(project "control_unit"
 				(path "/dccec861-b967-466c-843e-d6d1ad6064ce/a601307c-be83-4128-aa2e-f19df4dff19c/c0031539-c4c3-432d-9a69-ce5a0aa72fa8"
-					(reference "U9")
+					(reference "Uip2")
+					(unit 1)
+				)
+			)
+		)
+	)
+	(symbol
+		(lib_id "power:GND")
+		(at 95.25 58.42 270)
+		(unit 1)
+		(exclude_from_sim no)
+		(in_bom yes)
+		(on_board yes)
+		(dnp no)
+		(fields_autoplaced yes)
+		(property "Reference" "#PWR0221"
+			(at 88.9 58.42 0)
+			(effects
+				(font
+					(size 1.27 1.27)
+				)
+				(hide yes)
+			)
+		)
+		(property "Value" "GND"
+			(at 91.44 58.4199 90)
+			(effects
+				(font
+					(size 1.27 1.27)
+				)
+				(justify right)
+			)
+		)
+		(property "Footprint" ""
+			(at 95.25 58.42 0)
+			(effects
+				(font
+					(size 1.27 1.27)
+				)
+				(hide yes)
+			)
+		)
+		(property "Datasheet" ""
+			(at 95.25 58.42 0)
+			(effects
+				(font
+					(size 1.27 1.27)
+				)
+				(hide yes)
+			)
+		)
+		(property "Description" "Power symbol creates a global label with name \"GND\" , ground"
+			(at 95.25 58.42 0)
+			(effects
+				(font
+					(size 1.27 1.27)
+				)
+				(hide yes)
+			)
+		)
+		(pin "1"
+		)
+		(instances
+			(project "control_unit"
+				(path "/dccec861-b967-466c-843e-d6d1ad6064ce/a601307c-be83-4128-aa2e-f19df4dff19c/c0031539-c4c3-432d-9a69-ce5a0aa72fa8"
+					(reference "#PWR0221")
 					(unit 1)
 				)

Commit message: control unit update
Parts:
- added Cip1, Cip2, Cip3, Cip4, Cip5: 100nF, Capacitor_SMD:C_0402_1005Metric, symbol Device:C
- Uip1, Uip2, Uip3, Uip4: value 74LS283 -> 74283; footprint Package_SO:SOIC-14_3.9x8.7mm_P1.27mm -> Package_SO:SOIC-16_3.9x9.9mm_P1.27mm
Connections:
- net GND: now also Cip1.2, Cip2.2, Cip3.2, Cip4.2, Cip5.2
- net VCC: now also Cip1.1, Cip2.1, Cip3.1, Cip4.1, Cip5.1
