File: PCB/Kicad/control_unit/control_unit.kicad_pcb (KiCad board)
At the start: 6 copper layers, 0 parts

Commit message: control unit schematic
Parts:
- added D1: green, Diode_SMD:D_0603_1608Metric, F.Cu at (124.3, 93.1)
- added Dd1: yellow, LED_SMD:LED_0603_1608Metric, F.Cu at (136.8, 27.2)
- added Dd10: yellow, LED_SMD:LED_0603_1608Metric, F.Cu at (140.9, 32.4)
- added Dd11: yellow, LED_SMD:LED_0603_1608Metric, F.Cu at (140.9, 35.0)
- added Dd12: yellow, LED_SMD:LED_0603_1608Metric, F.Cu at (140.9, 37.6)
- added Dd13: yellow, LED_SMD:LED_0603_1608Metric, F.Cu at (140.9, 40.2)
- added Dd14: yellow, LED_SMD:LED_0603_1608Metric, F.Cu at (140.9, 42.8)
- added Dd15: yellow, LED_SMD:LED_0603_1608Metric, F.Cu at (144.9, 27.2)
- added Dd16: yellow, LED_SMD:LED_0603_1608Metric, F.Cu at (144.9, 29.8)
- added Dd17: yellow, LED_SMD:LED_0603_1608Metric, F.Cu at (144.9, 32.4)
- added Dd18: yellow, LED_SMD:LED_0603_1608Metric, F.Cu at (144.9, 35.0)
- added Dd19: yellow, LED_SMD:LED_0603_1608Metric, F.Cu at (144.9, 37.6)
- added Dd2: yellow, LED_SMD:LED_0603_1608Metric, F.Cu at (136.8, 29.8)
- added Dd20: yellow, LED_SMD:LED_0603_1608Metric, F.Cu at (144.9, 40.2)
- added Dd21: yellow, LED_SMD:LED_0603_1608Metric, F.Cu at (144.9, 42.8)
- added Dd22: yellow, LED_SMD:LED_0603_1608Metric, F.Cu at (149.0, 27.2)
- added Dd23: yellow, LED_SMD:LED_0603_1608Metric, F.Cu at (149.0, 29.8)
- added Dd24: yellow, LED_SMD:LED_0603_1608Metric, F.Cu at (149.0, 32.4)
- added Dd25: yellow, LED_SMD:LED_0603_1608Metric, F.Cu at (149.0, 35.0)
- added Dd26: yellow, LED_SMD:LED_0603_1608Metric, F.Cu at (149.0, 37.6)
- added Dd3: yellow, LED_SMD:LED_0603_1608Metric, F.Cu at (136.8, 32.4)
- added Dd4: yellow, LED_SMD:LED_0603_1608Metric, F.Cu at (136.8, 35.0)
- added Dd5: yellow, LED_SMD:LED_0603_1608Metric, F.Cu at (136.8, 37.6)
- added Dd6: yellow, LED_SMD:LED_0603_1608Metric, F.Cu at (136.8, 40.2)
- added Dd7: yellow, LED_SMD:LED_0603_1608Metric, F.Cu at (136.8, 42.8)
- added Dd8: yellow, LED_SMD:LED_0603_1608Metric, F.Cu at (140.9, 27.2)
- added Dd9: yellow, LED_SMD:LED_0603_1608Metric, F.Cu at (140.9, 29.8)
- added Dr1: red, LED_SMD:LED_0603_1608Metric, F.Cu at (183.3, 27.2)
- added Dr10: red, LED_SMD:LED_0603_1608Metric, F.Cu at (187.4, 35.0)
- added Dr11: red, LED_SMD:LED_0603_1608Metric, F.Cu at (187.4, 37.6)
- added Dr12: red, LED_SMD:LED_0603_1608Metric, F.Cu at (187.4, 40.2)
- added Dr13: red, LED_SMD:LED_0603_1608Metric, F.Cu at (191.4, 27.2)
- added Dr14: red, LED_SMD:LED_0603_1608Metric, F.Cu at (191.4, 29.8)
- added Dr15: red, LED_SMD:LED_0603_1608Metric, F.Cu at (191.4, 32.4)
- added Dr16: red, LED_SMD:LED_0603_1608Metric, F.Cu at (191.4, 35.0)
- added Dr17: red, LED_SMD:LED_0603_1608Metric, F.Cu at (155.1, 27.2)
- added Dr18: red, LED_SMD:LED_0603_1608Metric, F.Cu at (155.1, 29.8)
- added Dr19: red, LED_SMD:LED_0603_1608Metric, F.Cu at (155.1, 32.4)
- added Dr2: red, LED_SMD:LED_0603_1608Metric, F.Cu at (183.3, 29.8)
- added Dr20: red, LED_SMD:LED_0603_1608Metric, F.Cu at (155.1, 35.0)
- added Dr21: red, LED_SMD:LED_0603_1608Metric, F.Cu at (155.1, 37.6)
- added Dr22: red, LED_SMD:LED_0603_1608Metric, F.Cu at (155.1, 40.2)
- added Dr23: red, LED_SMD:LED_0603_1608Metric, F.Cu at (159.1, 27.2)
- added Dr24: red, LED_SMD:LED_0603_1608Metric, F.Cu at (159.1, 29.8)
- added Dr25: red, LED_SMD:LED_0603_1608Metric, F.Cu at (159.1, 32.4)
- added Dr26: red, LED_SMD:LED_0603_1608Metric, F.Cu at (159.1, 35.0)
- added Dr27: red, LED_SMD:LED_0603_1608Metric, F.Cu at (159.1, 37.6)
- added Dr28: red, LED_SMD:LED_0603_1608Metric, F.Cu at (159.1, 40.2)
- added Dr29: red, LED_SMD:LED_0603_1608Metric, F.Cu at (163.2, 27.2)
- added Dr3: red, LED_SMD:LED_0603_1608Metric, F.Cu at (183.3, 32.4)
- added Dr30: red, LED_SMD:LED_0603_1608Metric, F.Cu at (163.2, 29.8)
- added Dr31: red, LED_SMD:LED_0603_1608Metric, F.Cu at (163.2, 32.4)
- added Dr32: red, LED_SMD:LED_0603_1608Metric, F.Cu at (163.2, 35.0)
- added Dr33: red, LED_SMD:LED_0603_1608Metric, F.Cu at (169.2, 27.2)
- added Dr34: red, LED_SMD:LED_0603_1608Metric, F.Cu at (169.2, 29.8)
- added Dr35: red, LED_SMD:LED_0603_1608Metric, F.Cu at (169.2, 32.4)
- added Dr36: red, LED_SMD:LED_0603_1608Metric, F.Cu at (169.2, 35.0)
- added Dr37: red, LED_SMD:LED_0603_1608Metric, F.Cu at (169.2, 37.6)
- added Dr38: red, LED_SMD:LED_0603_1608Metric, F.Cu at (169.2, 40.2)
- added Dr39: red, LED_SMD:LED_0603_1608Metric, F.Cu at (173.2, 27.2)
- added Dr4: red, LED_SMD:LED_0603_1608Metric, F.Cu at (183.3, 35.0)
- added Dr40: red, LED_SMD:LED_0603_1608Metric, F.Cu at (173.2, 29.8)
- added Dr41: red, LED_SMD:LED_0603_1608Metric, F.Cu at (173.2, 32.4)
- added Dr42: red, LED_SMD:LED_0603_1608Metric, F.Cu at (173.2, 35.0)
- added Dr43: red, LED_SMD:LED_0603_1608Metric, F.Cu at (173.2, 37.6)
- added Dr44: red, LED_SMD:LED_0603_1608Metric, F.Cu at (173.2, 40.2)
- added Dr45: red, LED_SMD:LED_0603_1608Metric, F.Cu at (177.3, 27.2)
- added Dr46: red, LED_SMD:LED_0603_1608Metric, F.Cu at (177.3, 29.8)
- added Dr47: red, LED_SMD:LED_0603_1608Metric, F.Cu at (177.3, 32.4)
- added Dr48: red, LED_SMD:LED_0603_1608Metric, F.Cu at (177.3, 35.0)
- added Dr5: red, LED_SMD:LED_0603_1608Metric, F.Cu at (183.3, 37.6)
- added Dr6: red, LED_SMD:LED_0603_1608Metric, F.Cu at (183.3, 40.2)
- added Dr7: red, LED_SMD:LED_0603_1608Metric, F.Cu at (187.4, 27.2)
- added Dr8: red, LED_SMD:LED_0603_1608Metric, F.Cu at (187.4, 29.8)
- added Dr9: red, LED_SMD:LED_0603_1608Metric, F.Cu at (187.4, 32.4)
- added H1: MountingHole_Pad, MountingHole:MountingHole_2.2mm_M2_DIN965_Pad, F.Cu at (119.6, 94.5)
- added H2: MountingHole_Pad, MountingHole:MountingHole_2.2mm_M2_DIN965_Pad, F.Cu at (119.6, 99.9)
- added H3: MountingHole_Pad, MountingHole:MountingHole_2.2mm_M2_DIN965_Pad, F.Cu at (119.6, 105.2)
- added H4: MountingHole_Pad, MountingHole:MountingHole_2.2mm_M2_DIN965_Pad, F.Cu at (119.6, 110.6)
- added J1: Conn_02x10_Odd_Even, Connector_PinHeader_2.54mm:PinHeader_2x10_P2.54mm_Horizontal, F.Cu at (77.8, 161.7)
- added J2: Conn_02x10_Odd_Even, Connector_PinHeader_2.54mm:PinHeader_2x10_P2.54mm_Horizontal, F.Cu at (119.2, 66.7)
- added J3: Conn_02x10_Odd_Even, Connector_PinHeader_2.54mm:PinHeader_2x10_P2.54mm_Horizontal, F.Cu at (135.1, 66.7)
- added J4: Conn_02x10_Odd_Even, Connector_PinHeader_2.54mm:PinHeader_2x10_P2.54mm_Horizontal, F.Cu at (151.0, 66.7)
- added J5: Conn_02x10_Odd_Even, Connector_PinHeader_2.54mm:PinHeader_2x10_P2.54mm_Horizontal, F.Cu at (166.9, 66.7)
- added J6: Conn_02x10_Odd_Even, Connector_PinHeader_2.54mm:PinHeader_2x10_P2.54mm_Horizontal, F.Cu at (182.8, 66.7)
- added J7: Conn_02x10_Odd_Even, Connector_PinHeader_2.54mm:PinHeader_2x10_P2.54mm_Horizontal, F.Cu at (198.8, 66.7)
- added R33: 10k, Resistor_SMD:R_0402_1005Metric, F.Cu at (121.5, 26.7)
- added Rcr1: 10k, Resistor_SMD:R_0402_1005Metric, F.Cu at (131.9, 15.9)
- added Rcr2: 10k, Resistor_SMD:R_0402_1005Metric, F.Cu at (131.9, 17.9)
- added Rcr3: 10k, Resistor_SMD:R_0402_1005Metric, F.Cu at (131.9, 19.9)
- added Rcr4: 10k, Resistor_SMD:R_0402_1005Metric, F.Cu at (131.9, 21.9)
- added Rcuc1: 10k, Resistor_SMD:R_0402_1005Metric, F.Cu at (129.5, 97.3)
- added Rd1: 680, Resistor_SMD:R_0402_1005Metric, F.Cu at (136.3, 45.1)
- added Rd10: 680, Resistor_SMD:R_0402_1005Metric, F.Cu at (139.2, 49.0)
- added Rd11: 680, Resistor_SMD:R_0402_1005Metric, F.Cu at (139.2, 51.0)
- added Rd12: 680, Resistor_SMD:R_0402_1005Metric, F.Cu at (139.2, 53.0)
- added Rd13: 680, Resistor_SMD:R_0402_1005Metric, F.Cu at (139.2, 55.0)
- added Rd14: 680, Resistor_SMD:R_0402_1005Metric, F.Cu at (139.2, 57.0)
- added Rd15: 680, Resistor_SMD:R_0402_1005Metric, F.Cu at (142.1, 45.1)
- added Rd16: 680, Resistor_SMD:R_0402_1005Metric, F.Cu at (142.1, 47.0)
- added Rd17: 680, Resistor_SMD:R_0402_1005Metric, F.Cu at (142.1, 49.0)
- added Rd18: 680, Resistor_SMD:R_0402_1005Metric, F.Cu at (142.1, 51.0)
- added Rd19: 680, Resistor_SMD:R_0402_1005Metric, F.Cu at (142.1, 53.0)
- added Rd2: 680, Resistor_SMD:R_0402_1005Metric, F.Cu at (136.3, 47.0)
- added Rd20: 680, Resistor_SMD:R_0402_1005Metric, F.Cu at (142.1, 55.0)
- added Rd21: 680, Resistor_SMD:R_0402_1005Metric, F.Cu at (142.1, 57.0)
- added Rd22: 680, Resistor_SMD:R_0402_1005Metric, F.Cu at (145.0, 45.1)
- added Rd23: 680, Resistor_SMD:R_0402_1005Metric, F.Cu at (145.0, 47.0)
- added Rd24: 680, Resistor_SMD:R_0402_1005Metric, F.Cu at (145.0, 49.0)
- added Rd25: 680, Resistor_SMD:R_0402_1005Metric, F.Cu at (145.0, 51.0)
- added Rd26: 680, Resistor_SMD:R_0402_1005Metric, F.Cu at (145.0, 53.0)
- added Rd3: 680, Resistor_SMD:R_0402_1005Metric, F.Cu at (136.3, 49.0)
- added Rd4: 680, Resistor_SMD:R_0402_1005Metric, F.Cu at (136.3, 51.0)
- added Rd5: 680, Resistor_SMD:R_0402_1005Metric, F.Cu at (136.3, 53.0)
- added Rd6: 680, Resistor_SMD:R_0402_1005Metric, F.Cu at (136.3, 55.0)
- added Rd7: 680, Resistor_SMD:R_0402_1005Metric, F.Cu at (136.3, 57.0)
- added Rd8: 680, Resistor_SMD:R_0402_1005Metric, F.Cu at (139.2, 45.1)
- added Rd9: 680, Resistor_SMD:R_0402_1005Metric, F.Cu at (139.2, 47.0)
- added Rio3: 680, Resistor_SMD:R_0402_1005Metric, F.Cu at (123.7, 95.4)
- added Rir1: 10k, Resistor_SMD:R_0402_1005Metric, F.Cu at (129.5, 101.3)
- added Rir2: 10k, Resistor_SMD:R_0402_1005Metric, F.Cu at (129.5, 103.3)
- added Rir3: 10k, Resistor_SMD:R_0402_1005Metric, F.Cu at (129.5, 105.3)
- added Rir4: 10k, Resistor_SMD:R_0402_1005Metric, F.Cu at (129.5, 107.2)
- added Rpd1: 10k, Resistor_SMD:R_0402_1005Metric, F.Cu at (136.8, 15.9)
- added Rpd10: 10k, Resistor_SMD:R_0402_1005Metric, F.Cu at (142.6, 17.9)
- added Rpd11: 10k, Resistor_SMD:R_0402_1005Metric, F.Cu at (142.6, 19.9)
- added Rpd12: 10k, Resistor_SMD:R_0402_1005Metric, F.Cu at (142.6, 21.9)
- added Rpd13: 10k, Resistor_SMD:R_0402_1005Metric, F.Cu at (145.5, 15.9)
- added Rpd14: 10k, Resistor_SMD:R_0402_1005Metric, F.Cu at (145.5, 17.9)
- added Rpd15: 10k, Resistor_SMD:R_0402_1005Metric, F.Cu at (145.5, 19.9)
- added Rpd16: 10k, Resistor_SMD:R_0402_1005Metric, F.Cu at (145.5, 21.9)
- added Rpd17: 10k, Resistor_SMD:R_0402_1005Metric, F.Cu at (150.4, 15.9)
- added Rpd18: 10k, Resistor_SMD:R_0402_1005Metric, F.Cu at (150.4, 17.9)
- added Rpd19: 10k, Resistor_SMD:R_0402_1005Metric, F.Cu at (150.4, 19.9)
- added Rpd2: 10k, Resistor_SMD:R_0402_1005Metric, F.Cu at (136.8, 17.9)
- added Rpd20: 10k, Resistor_SMD:R_0402_1005Metric, F.Cu at (150.4, 21.9)
- added Rpd21: 10k, Resistor_SMD:R_0402_1005Metric, F.Cu at (153.4, 15.9)
- added Rpd22: 10k, Resistor_SMD:R_0402_1005Metric, F.Cu at (153.4, 17.9)
- added Rpd23: 10k, Resistor_SMD:R_0402_1005Metric, F.Cu at (153.4, 19.9)
- added Rpd24: 10k, Resistor_SMD:R_0402_1005Metric, F.Cu at (153.4, 21.9)
- added Rpd25: 10k, Resistor_SMD:R_0402_1005Metric, F.Cu at (156.3, 15.9)
- added Rpd26: 10k, Resistor_SMD:R_0402_1005Metric, F.Cu at (156.3, 17.9)
- added Rpd27: 10k, Resistor_SMD:R_0402_1005Metric, F.Cu at (156.3, 19.9)
- added Rpd28: 10k, Resistor_SMD:R_0402_1005Metric, F.Cu at (156.3, 21.9)
- added Rpd29: 10k, Resistor_SMD:R_0402_1005Metric, F.Cu at (159.2, 15.9)
- added Rpd3: 10k, Resistor_SMD:R_0402_1005Metric, F.Cu at (136.8, 19.9)
- added Rpd30: 10k, Resistor_SMD:R_0402_1005Metric, F.Cu at (159.2, 17.9)
- added Rpd31: 10k, Resistor_SMD:R_0402_1005Metric, F.Cu at (159.2, 19.9)
- added Rpd32: 10k, Resistor_SMD:R_0402_1005Metric, F.Cu at (159.2, 21.9)
- added Rpd34: 10k, Resistor_SMD:R_0402_1005Metric, F.Cu at (121.5, 28.7)
- added Rpd35: 10k, Resistor_SMD:R_0402_1005Metric, F.Cu at (121.5, 30.7)
- added Rpd36: 10k, Resistor_SMD:R_0402_1005Metric, F.Cu at (121.5, 32.7)
- added Rpd37: 10k, Resistor_SMD:R_0402_1005Metric, F.Cu at (124.4, 26.7)
- added Rpd38: 10k, Resistor_SMD:R_0402_1005Metric, F.Cu at (124.4, 28.7)
- added Rpd39: 10k, Resistor_SMD:R_0402_1005Metric, F.Cu at (124.4, 30.7)
- added Rpd4: 10k, Resistor_SMD:R_0402_1005Metric, F.Cu at (136.8, 21.9)
- added Rpd40: 10k, Resistor_SMD:R_0402_1005Metric, F.Cu at (124.4, 32.7)
- added Rpd41: 10k, Resistor_SMD:R_0402_1005Metric, F.Cu at (127.3, 26.7)
- added Rpd42: 10k, Resistor_SMD:R_0402_1005Metric, F.Cu at (127.3, 28.7)
- added Rpd43: 10k, Resistor_SMD:R_0402_1005Metric, F.Cu at (127.3, 30.7)
- added Rpd44: 10k, Resistor_SMD:R_0402_1005Metric, F.Cu at (127.3, 32.7)
- added Rpd45: 10k, Resistor_SMD:R_0402_1005Metric, F.Cu at (130.2, 26.7)
- added Rpd46: 10k, Resistor_SMD:R_0402_1005Metric, F.Cu at (130.2, 28.7)
- added Rpd47: 10k, Resistor_SMD:R_0402_1005Metric, F.Cu at (130.2, 30.7)
- added Rpd48: 10k, Resistor_SMD:R_0402_1005Metric, F.Cu at (130.2, 32.7)
- added Rpd5: 10k, Resistor_SMD:R_0402_1005Metric, F.Cu at (139.7, 15.9)
- added Rpd6: 10k, Resistor_SMD:R_0402_1005Metric, F.Cu at (139.7, 17.9)
- added Rpd7: 10k, Resistor_SMD:R_0402_1005Metric, F.Cu at (139.7, 19.9)
- added Rpd8: 10k, Resistor_SMD:R_0402_1005Metric, F.Cu at (139.7, 21.9)
- added Rpd9: 10k, Resistor_SMD:R_0402_1005Metric, F.Cu at (142.6, 15.9)
- added Rr1: 680, Resistor_SMD:R_0402_1005Metric, F.Cu at (182.8, 42.5)
- added Rr10: 680, Resistor_SMD:R_0402_1005Metric, F.Cu at (188.6, 44.5)
- added Rr11: 680, Resistor_SMD:R_0402_1005Metric, F.Cu at (188.6, 46.5)
- added Rr12: 680, Resistor_SMD:R_0402_1005Metric, F.Cu at (188.6, 48.4)
- added Rr13: 680, Resistor_SMD:R_0402_1005Metric, F.Cu at (191.5, 42.5)
- added Rr14: 680, Resistor_SMD:R_0402_1005Metric, F.Cu at (191.5, 44.5)
- added Rr15: 680, Resistor_SMD:R_0402_1005Metric, F.Cu at (191.5, 46.5)
- added Rr16: 680, Resistor_SMD:R_0402_1005Metric, F.Cu at (191.5, 48.4)
- added Rr17: 680, Resistor_SMD:R_0402_1005Metric, F.Cu at (154.5, 42.5)
- added Rr18: 680, Resistor_SMD:R_0402_1005Metric, F.Cu at (154.5, 44.5)
- added Rr19: 680, Resistor_SMD:R_0402_1005Metric, F.Cu at (154.5, 46.5)
- added Rr2: 680, Resistor_SMD:R_0402_1005Metric, F.Cu at (182.8, 44.5)
- added Rr20: 680, Resistor_SMD:R_0402_1005Metric, F.Cu at (154.5, 48.4)
- added Rr21: 680, Resistor_SMD:R_0402_1005Metric, F.Cu at (157.4, 42.5)
- added Rr22: 680, Resistor_SMD:R_0402_1005Metric, F.Cu at (157.4, 44.5)
- added Rr23: 680, Resistor_SMD:R_0402_1005Metric, F.Cu at (157.4, 46.5)
- added Rr24: 680, Resistor_SMD:R_0402_1005Metric, F.Cu at (157.4, 48.4)
- added Rr25: 680, Resistor_SMD:R_0402_1005Metric, F.Cu at (160.3, 42.5)
- added Rr26: 680, Resistor_SMD:R_0402_1005Metric, F.Cu at (160.3, 44.5)
- added Rr27: 680, Resistor_SMD:R_0402_1005Metric, F.Cu at (160.3, 46.5)
- added Rr28: 680, Resistor_SMD:R_0402_1005Metric, F.Cu at (160.3, 48.4)
- added Rr29: 680, Resistor_SMD:R_0402_1005Metric, F.Cu at (163.2, 42.5)
- added Rr3: 680, Resistor_SMD:R_0402_1005Metric, F.Cu at (182.8, 46.5)
- added Rr30: 680, Resistor_SMD:R_0402_1005Metric, F.Cu at (163.2, 44.5)
- added Rr31: 680, Resistor_SMD:R_0402_1005Metric, F.Cu at (163.2, 46.5)
- added Rr32: 680, Resistor_SMD:R_0402_1005Metric, F.Cu at (163.2, 48.4)
- added Rr33: 680, Resistor_SMD:R_0402_1005Metric, F.Cu at (168.6, 42.5)
- added Rr34: 680, Resistor_SMD:R_0402_1005Metric, F.Cu at (168.6, 44.5)
- added Rr35: 680, Resistor_SMD:R_0402_1005Metric, F.Cu at (168.6, 46.5)
- added Rr36: 680, Resistor_SMD:R_0402_1005Metric, F.Cu at (168.6, 48.4)
- added Rr37: 680, Resistor_SMD:R_0402_1005Metric, F.Cu at (171.5, 42.5)
- added Rr38: 680, Resistor_SMD:R_0402_1005Metric, F.Cu at (171.5, 44.5)
- added Rr39: 680, Resistor_SMD:R_0402_1005Metric, F.Cu at (171.5, 46.5)
- added Rr4: 680, Resistor_SMD:R_0402_1005Metric, F.Cu at (182.8, 48.4)
- added Rr40: 680, Resistor_SMD:R_0402_1005Metric, F.Cu at (171.5, 48.4)
- added Rr41: 680, Resistor_SMD:R_0402_1005Metric, F.Cu at (174.4, 42.5)
- added Rr42: 680, Resistor_SMD:R_0402_1005Metric, F.Cu at (174.4, 44.5)
- added Rr43: 680, Resistor_SMD:R_0402_1005Metric, F.Cu at (174.4, 46.5)
- added Rr44: 680, Resistor_SMD:R_0402_1005Metric, F.Cu at (174.4, 48.4)
- added Rr45: 680, Resistor_SMD:R_0402_1005Metric, F.Cu at (177.3, 42.5)
- added Rr46: 680, Resistor_SMD:R_0402_1005Metric, F.Cu at (177.3, 44.5)
- added Rr47: 680, Resistor_SMD:R_0402_1005Metric, F.Cu at (177.3, 46.5)
- added Rr48: 680, Resistor_SMD:R_0402_1005Metric, F.Cu at (177.3, 48.4)
- added Rr5: 680, Resistor_SMD:R_0402_1005Metric, F.Cu at (185.7, 42.5)
- added Rr6: 680, Resistor_SMD:R_0402_1005Metric, F.Cu at (185.7, 44.5)
- added Rr7: 680, Resistor_SMD:R_0402_1005Metric, F.Cu at (185.7, 46.5)
- added Rr8: 680, Resistor_SMD:R_0402_1005Metric, F.Cu at (185.7, 48.4)
- added Rr9: 680, Resistor_SMD:R_0402_1005Metric, F.Cu at (188.6, 42.5)
- added SW1: SW_Push, Button_Switch_THT:SW_PUSH_6mm_H4.3mm, F.Cu at (155.5, 160.8)
- added U4: 74LS08, Package_SO:SOIC-14_3.9x8.7mm_P1.27mm, F.Cu at (148.3, 158.6)
- added U57: 16to1_MUX__CD74HC4067M96, mALUch_lib:SOIC127P1030X265-24N, F.Cu at (35.3, 120.6)
- added Ubc1: 74LS139, Package_SO:SOIC-14_3.9x8.7mm_P1.27mm, F.Cu at (160.7, 139.7)
- added Ubc2: 74LS139, Package_SO:SOIC-14_3.9x8.7mm_P1.27mm, F.Cu at (160.7, 131.2)
- added Ubc3: 74LS04, Package_SO:SOIC-14_3.9x8.7mm_P1.27mm, F.Cu at (148.3, 150.1)
- added Ubd1: 74HC245, Package_SO:SOIC-20W_7.5x12.8mm_P1.27mm, F.Cu at (18.9, 85.6)
- added Ubd10: 74HC245, Package_SO:SOIC-20W_7.5x12.8mm_P1.27mm, F.Cu at (59.6, 52.7)
- added Ubd11: 74HC245, Package_SO:SOIC-20W_7.5x12.8mm_P1.27mm, F.Cu at (46.7, 69.2)
- added Ubd12: 74HC245, Package_SO:SOIC-20W_7.5x12.8mm_P1.27mm, F.Cu at (59.6, 69.2)
- added Ubd13: 74HC245, Package_SO:SOIC-20W_7.5x12.8mm_P1.27mm, F.Cu at (18.9, 52.7)
- added Ubd14: 74HC245, Package_SO:SOIC-20W_7.5x12.8mm_P1.27mm, F.Cu at (31.8, 52.7)
- added Ubd15: 74HC245, Package_SO:SOIC-20W_7.5x12.8mm_P1.27mm, F.Cu at (18.9, 36.2)
- added Ubd16: 74HC245, Package_SO:SOIC-20W_7.5x12.8mm_P1.27mm, F.Cu at (31.8, 36.2)
- added Ubd17: 74HC245, Package_SO:SOIC-20W_7.5x12.8mm_P1.27mm, F.Cu at (46.7, 19.7)
- added Ubd18: 74HC245, Package_SO:SOIC-20W_7.5x12.8mm_P1.27mm, F.Cu at (59.6, 19.7)
- added Ubd19: 74HC245, Package_SO:SOIC-20W_7.5x12.8mm_P1.27mm, F.Cu at (18.9, 102.1)
- added Ubd2: 74HC245, Package_SO:SOIC-20W_7.5x12.8mm_P1.27mm, F.Cu at (31.8, 85.6)
- added Ubd20: 74HC245, Package_SO:SOIC-20W_7.5x12.8mm_P1.27mm, F.Cu at (31.8, 102.1)
- added Ubd3: 74HC245, Package_SO:SOIC-20W_7.5x12.8mm_P1.27mm, F.Cu at (74.5, 69.2)
- added Ubd4: 74HC245, Package_SO:SOIC-20W_7.5x12.8mm_P1.27mm, F.Cu at (87.5, 69.2)
- added Ubd5: 74HC245, Package_SO:SOIC-20W_7.5x12.8mm_P1.27mm, F.Cu at (46.7, 85.6)
- added Ubd6: 74HC245, Package_SO:SOIC-20W_7.5x12.8mm_P1.27mm, F.Cu at (59.6, 85.6)
- added Ubd7: 74HC245, Package_SO:SOIC-20W_7.5x12.8mm_P1.27mm, F.Cu at (18.9, 69.2)
- added Ubd8: 74HC245, Package_SO:SOIC-20W_7.5x12.8mm_P1.27mm, F.Cu at (31.8, 69.2)
- added Ubd9: 74HC245, Package_SO:SOIC-20W_7.5x12.8mm_P1.27mm, F.Cu at (46.7, 52.7)
- added Ubu1: 74HC245, Package_SO:SOIC-20W_7.5x12.8mm_P1.27mm, F.Cu at (74.5, 52.7)
- added Ubu10: 74HC245, Package_SO:SOIC-20W_7.5x12.8mm_P1.27mm, F.Cu at (87.5, 102.1)
- added Ubu11: 74HC245, Package_SO:SOIC-20W_7.5x12.8mm_P1.27mm, F.Cu at (74.5, 36.2)
- added Ubu12: 74HC245, Package_SO:SOIC-20W_7.5x12.8mm_P1.27mm, F.Cu at (87.5, 36.2)
- added Ubu13: 74HC245, Package_SO:SOIC-20W_7.5x12.8mm_P1.27mm, F.Cu at (46.7, 36.2)
- added Ubu14: 74HC245, Package_SO:SOIC-20W_7.5x12.8mm_P1.27mm, F.Cu at (59.6, 36.2)
- added Ubu15: 74HC245, Package_SO:SOIC-20W_7.5x12.8mm_P1.27mm, F.Cu at (74.5, 19.7)
- added Ubu16: 74HC245, Package_SO:SOIC-20W_7.5x12.8mm_P1.27mm, F.Cu at (87.5, 19.7)
- added Ubu2: 74HC245, Package_SO:SOIC-20W_7.5x12.8mm_P1.27mm, F.Cu at (87.5, 52.7)
- added Ubu3: 74HC245, Package_SO:SOIC-20W_7.5x12.8mm_P1.27mm, F.Cu at (46.7, 102.1)
- added Ubu4: 74HC245, Package_SO:SOIC-20W_7.5x12.8mm_P1.27mm, F.Cu at (59.6, 102.1)
- added Ubu5: 74HC245, Package_SO:SOIC-20W_7.5x12.8mm_P1.27mm, F.Cu at (18.9, 19.7)
- added Ubu6: 74HC245, Package_SO:SOIC-20W_7.5x12.8mm_P1.27mm, F.Cu at (31.8, 19.7)
- added Ubu7: 74HC245, Package_SO:SOIC-20W_7.5x12.8mm_P1.27mm, F.Cu at (74.5, 85.6)
- added Ubu8: 74HC245, Package_SO:SOIC-20W_7.5x12.8mm_P1.27mm, F.Cu at (87.5, 85.6)
- added Ubu9: 74HC245, Package_SO:SOIC-20W_7.5x12.8mm_P1.27mm, F.Cu at (74.5, 102.1)
- added Ucr1: 74LS283, Package_SO:SOIC-14_3.9x8.7mm_P1.27mm, F.Cu at (148.3, 139.7)
- added Ucr2: 74LS257, Package_SO:SOIC-14_3.9x8.7mm_P1.27mm, F.Cu at (148.3, 131.2)
- added Ucr3: 74LS377, Package_SO:SSOP-20_5.3x7.2mm_P0.65mm, F.Cu at (125.2, 19.3)
- added Ud1: KM28C64A, Package_DIP:DIP-28_W15.24mm, F.Cu at (99.2, 15.6)
- added Ud2: KM28C64A, Package_DIP:DIP-28_W15.24mm, F.Cu at (99.1, 52.5)
- added Ud3: KM28C64A, Package_DIP:DIP-28_W15.24mm, F.Cu at (99.0, 89.5)
- added Ud4: KM28C64A, Package_DIP:DIP-28_W15.24mm, F.Cu at (98.9, 126.0)
- added Uf1: 74LS257, Package_SO:SOIC-14_3.9x8.7mm_P1.27mm, F.Cu at (123.6, 158.6)
- added Uf2: 74LS377, Package_SO:SSOP-20_5.3x7.2mm_P0.65mm, F.Cu at (166.7, 112.8)
- added Uf3: 74LS04, Package_SO:SOIC-14_3.9x8.7mm_P1.27mm, F.Cu at (123.6, 150.1)
- added Uf4: 74LS32, Package_SO:SOIC-14_3.9x8.7mm_P1.27mm, F.Cu at (123.6, 141.7)
- added Uf5: 74LS86, Package_SO:SOIC-14_3.9x8.7mm_P1.27mm, F.Cu at (123.6, 133.2)
- added Uf6: 74LS257, Package_SO:SOIC-14_3.9x8.7mm_P1.27mm, F.Cu at (123.6, 124.8)
- added Uf7: 74LS377, Package_SO:SSOP-20_5.3x7.2mm_P0.65mm, F.Cu at (157.9, 112.8)
- added Uinsr1: 74LS257, Package_SO:SOIC-14_3.9x8.7mm_P1.27mm, F.Cu at (136.0, 122.8)
- added Uip1: 74LS283, Package_SO:SOIC-14_3.9x8.7mm_P1.27mm, F.Cu at (136.0, 158.6)
- added Uip2: 74LS283, Package_SO:SOIC-14_3.9x8.7mm_P1.27mm, F.Cu at (136.0, 150.1)
- added Uip3: 74LS283, Package_SO:SOIC-14_3.9x8.7mm_P1.27mm, F.Cu at (136.0, 141.7)
- added Uip4: 74LS283, Package_SO:SOIC-14_3.9x8.7mm_P1.27mm, F.Cu at (136.0, 133.2)
- added Uip5: ATF16V8Bxx-xxPU, Package_DIP:DIP-20_W7.62mm, F.Cu at (16.8, 114.1)
- added Uir1: 74LS257, Package_SO:SSOP-20_5.3x7.2mm_P0.65mm, F.Cu at (125.2, 40.1)
- added Uir2: 74LS377, Package_SO:SSOP-20_5.3x7.2mm_P0.65mm, F.Cu at (125.2, 48.9)
- added Ur1: 74LS377, Package_SO:SSOP-20_5.3x7.2mm_P0.65mm, F.Cu at (157.9, 100.3)
- added Ur2: 74LS377, Package_SO:SSOP-20_5.3x7.2mm_P0.65mm, F.Cu at (166.7, 100.3)
- added Ur3: 74LS377, Package_SO:SSOP-20_5.3x7.2mm_P0.65mm, F.Cu at (138.3, 112.8)
- added Ur4: 74LS377, Package_SO:SSOP-20_5.3x7.2mm_P0.65mm, F.Cu at (147.1, 112.8)
- added Ur5: 74LS377, Package_SO:SSOP-20_5.3x7.2mm_P0.65mm, F.Cu at (138.3, 100.3)
- added Ur6: 74LS377, Package_SO:SSOP-20_5.3x7.2mm_P0.65mm, F.Cu at (147.1, 100.3)
Other:
- board outline added: 200 x 150 mm

Commit message: control unit update
Parts:
- added C1: 100nF, Capacitor_SMD:C_0402_1005Metric, F.Cu at (62.0, 130.5)
- added C10: 100nF, Capacitor_SMD:C_0402_1005Metric, F.Cu at (51.8, 92.0)
- added C11: 100nF, Capacitor_SMD:C_0402_1005Metric, F.Cu at (88.5, 40.8)
- added C12: 100nF, Capacitor_SMD:C_0402_1005Metric, F.Cu at (88.5, 42.7)
- added C13: 100nF, Capacitor_SMD:C_0402_1005Metric, F.Cu at (88.5, 44.7)
- added C14: 100nF, Capacitor_SMD:C_0402_1005Metric, F.Cu at (88.5, 46.7)
- added C2: 100nF, Capacitor_SMD:C_0402_1005Metric, F.Cu at (29.4, 92.7)
- added C3: 100nF, Capacitor_SMD:C_0402_1005Metric, F.Cu at (87.0, 117.3)
- added C4: 100nF, Capacitor_SMD:C_0402_1005Metric, F.Cu at (114.9, 59.9)
- added C5: 100nF, Capacitor_SMD:C_0402_1005Metric, F.Cu at (88.5, 38.8)
- added C6: 100nF, Capacitor_SMD:C_0402_1005Metric, F.Cu at (88.0, 78.1)
- added C7: 100nF, Capacitor_SMD:C_0402_1005Metric, F.Cu at (51.8, 78.1)
- added C8: 100nF, Capacitor_SMD:C_0402_1005Metric, F.Cu at (69.9, 92.0)
- added C9: 100nF, Capacitor_SMD:C_0402_1005Metric, F.Cu at (88.0, 92.0)
- added Cbc1: 100nF, Capacitor_SMD:C_0402_1005Metric, F.Cu at (84.1, 143.9)
- added Cbc2: 100nF, Capacitor_SMD:C_0402_1005Metric, F.Cu at (86.1, 143.9)
- added Cbc3: 100nF, Capacitor_SMD:C_0402_1005Metric, F.Cu at (88.1, 143.9)
- added Cbd1: 100nF, Capacitor_SMD:C_0402_1005Metric, F.Cu at (69.6, 104.3)
- added Cbd10: 100nF, Capacitor_SMD:C_0402_1005Metric, F.Cu at (90.0, 92.0)
- added Cbd11: 100nF, Capacitor_SMD:C_0402_1005Metric, F.Cu at (53.8, 92.0)
- added Cbd12: 100nF, Capacitor_SMD:C_0402_1005Metric, F.Cu at (68.9, 117.3)
- added Cbd13: 100nF, Capacitor_SMD:C_0402_1005Metric, F.Cu at (70.9, 117.3)
- added Cbd14: 100nF, Capacitor_SMD:C_0402_1005Metric, F.Cu at (29.4, 78.7)
- added Cbd15: 100nF, Capacitor_SMD:C_0402_1005Metric, F.Cu at (31.3, 78.7)
- added Cbd18: 100nF, Capacitor_SMD:C_0402_1005Metric, F.Cu at (128.9, 59.9)
- added Cbd19: 100nF, Capacitor_SMD:C_0402_1005Metric, F.Cu at (128.9, 61.9)
- added Cbd2: 100nF, Capacitor_SMD:C_0402_1005Metric, F.Cu at (50.8, 117.3)
- added Cbd20: 100nF, Capacitor_SMD:C_0402_1005Metric, F.Cu at (87.7, 104.3)
- added Cbd21: 100nF, Capacitor_SMD:C_0402_1005Metric, F.Cu at (89.7, 104.3)
- added Cbd22: 100nF, Capacitor_SMD:C_0402_1005Metric, F.Cu at (29.1, 105.0)
- added Cbd23: 100nF, Capacitor_SMD:C_0402_1005Metric, F.Cu at (31.0, 105.0)
- added Cbd24: 100nF, Capacitor_SMD:C_0402_1005Metric, F.Cu at (142.9, 59.9)
- added Cbd25: 100nF, Capacitor_SMD:C_0402_1005Metric, F.Cu at (142.9, 61.9)
- added Cbd26: 100nF, Capacitor_SMD:C_0402_1005Metric, F.Cu at (51.5, 104.3)
- added Cbd27: 100nF, Capacitor_SMD:C_0402_1005Metric, F.Cu at (53.5, 104.3)
- added Cbd28: 100nF, Capacitor_SMD:C_0402_1005Metric, F.Cu at (52.8, 117.3)
- added Cbd3: 100nF, Capacitor_SMD:C_0402_1005Metric, F.Cu at (31.3, 92.7)
- added Cbd4: 100nF, Capacitor_SMD:C_0402_1005Metric, F.Cu at (89.0, 117.3)
- added Cbd5: 100nF, Capacitor_SMD:C_0402_1005Metric, F.Cu at (114.9, 61.9)
- added Cbd6: 100nF, Capacitor_SMD:C_0402_1005Metric, F.Cu at (71.6, 104.3)
- added Cbd7: 100nF, Capacitor_SMD:C_0402_1005Metric, F.Cu at (90.0, 78.1)
- added Cbd8: 100nF, Capacitor_SMD:C_0402_1005Metric, F.Cu at (53.8, 78.1)
- added Cbd9: 100nF, Capacitor_SMD:C_0402_1005Metric, F.Cu at (71.9, 92.0)
- added Cbu16: 100nF, Capacitor_SMD:C_0402_1005Metric, F.Cu at (69.9, 78.1)
- added Cbu17: 100nF, Capacitor_SMD:C_0402_1005Metric, F.Cu at (71.9, 78.1)
- added Cinsr1: 100nF, Capacitor_SMD:C_0402_1005Metric, F.Cu at (100.0, 135.5)
- added Cinsr2: 100nF, Capacitor_SMD:C_0402_1005Metric, F.Cu at (93.5, 46.0)
- added Cinsr4: 100nF, Capacitor_SMD:C_0402_1005Metric, F.Cu at (16.7, 151.4)
- added Cip1: 100nF, Capacitor_SMD:C_0402_1005Metric, F.Cu at (116.5, 42.6)
- added Cip2: 100nF, Capacitor_SMD:C_0402_1005Metric, F.Cu at (116.5, 44.6)
- added Cip3: 100nF, Capacitor_SMD:C_0402_1005Metric, F.Cu at (116.5, 46.5)
- added Cip4: 100nF, Capacitor_SMD:C_0402_1005Metric, F.Cu at (116.5, 48.5)
- added Cip5: 100nF, Capacitor_SMD:C_0402_1005Metric, F.Cu at (116.5, 50.5)
- added Cir1: 100nF, Capacitor_SMD:C_0402_1005Metric, F.Cu at (37.2, 118.0)
- added Cir2: 100nF, Capacitor_SMD:C_0402_1005Metric, F.Cu at (39.1, 118.0)
- added Cr1: 100nF, Capacitor_SMD:C_0402_1005Metric, F.Cu at (93.5, 71.5)
- added Cr2: 100nF, Capacitor_SMD:C_0402_1005Metric, F.Cu at (93.5, 48.0)
- added Cr3: 100nF, Capacitor_SMD:C_0402_1005Metric, F.Cu at (93.5, 73.5)
- added Cr4: 100nF, Capacitor_SMD:C_0402_1005Metric, F.Cu at (16.7, 153.4)
- added J8: in, mALUch_lib:PinHeader_2x10_P2.54mm_Horizontal, F.Cu at (24.5, 42.9)
- D1: footprint Diode_SMD:D_0603_1608Metric -> LED_SMD:LED_0603_1608Metric
- J1, J2, J3, J4, J5, J6, J7: value Conn_02x10_Odd_Even -> in; footprint Connector_PinHeader_2.54mm:PinHeader_2x10_P2.54mm_Horizontal -> mALUch_lib:PinHeader_2x10_P2.54mm_Horizontal
- U4: value 74LS08 -> 7408; footprint Package_SO:SOIC-14_3.9x8.7mm_P1.27mm -> Package_SO:SO-14_3.9x8.65mm_P1.27mm
- U57: value 16to1_MUX__CD74HC4067M96 -> 744067; footprint mALUch_lib:SOIC127P1030X265-24N -> Package_SO:TSSOP-24_4.4x7.8mm_P0.65mm
- Ubc1, Ubc2: value 74LS139 -> 74139; footprint Package_SO:SOIC-14_3.9x8.7mm_P1.27mm -> Package_SO:SOIC-16_3.9x9.9mm_P1.27mm
- Ubc3, Uf3: value 74LS04 -> 7404; footprint Package_SO:SOIC-14_3.9x8.7mm_P1.27mm -> Package_SO:SO-14_3.9x8.65mm_P1.27mm
- Ubd1, Ubd10, Ubd11, Ubd12, Ubd13, Ubd14, Ubd15, Ubd16, Ubd17, Ubd18, Ubd19, Ubd2, Ubd20, Ubd3, Ubd4, Ubd5, Ubd6, Ubd7, Ubd8, Ubd9, Ubu1, Ubu10, Ubu11, Ubu12, Ubu13, Ubu14, Ubu15, Ubu16, Ubu2, Ubu3, Ubu4, Ubu5, Ubu6, Ubu7, Ubu8, Ubu9: value 74HC245 -> 74245; footprint Package_SO:SOIC-20W_7.5x12.8mm_P1.27mm -> Package_SO:TSSOP-20_4.4x6.5mm_P0.65mm
- Ucr1, Uip1, Uip2, Uip3, Uip4: value 74LS283 -> 74283; footprint Package_SO:SOIC-14_3.9x8.7mm_P1.27mm -> Package_SO:SOIC-16_3.9x9.9mm_P1.27mm
- Ucr2, Uf1, Uf6, Uinsr1: value 74LS257 -> 74257; footprint Package_SO:SOIC-14_3.9x8.7mm_P1.27mm -> Package_SO:SOIC-16_3.9x9.9mm_P1.27mm
- Ucr3, Uf2, Uf7, Uir2, Ur1, Ur2, Ur3, Ur4, Ur5, Ur6: value 74LS377 -> 74377
- Uf4: value 74LS32 -> 7432; footprint Package_SO:SOIC-14_3.9x8.7mm_P1.27mm -> Package_SO:SO-14_3.9x8.65mm_P1.27mm
- Uf5: value 74LS86 -> 7486; footprint Package_SO:SOIC-14_3.9x8.7mm_P1.27mm -> Package_SO:SO-14_3.9x8.65mm_P1.27mm
- Uir1: value 74LS257 -> 74257; footprint Package_SO:SSOP-20_5.3x7.2mm_P0.65mm -> Package_SO:SOIC-16_3.9x9.9mm_P1.27mm
- moved J5 155.0 mm to (24.5, 128.0), turned to 180 degrees
- moved Rcr1 148.7 mm to (40.8, 133.5), turned to 90 degrees
- moved Rcr2 145.9 mm to (42.8, 133.5), turned to 90 degrees
- moved Ucr3 145.4 mm to (44.2, 140.1), turned to 90 degrees
- moved Ud1 144.9 mm to (108.4, 160.2), turned to 90 degrees
- moved Rcr3 143.1 mm to (44.8, 133.5), turned to 90 degrees
- moved H4 141.7 mm to (15.0, 15.0), turned to 90 degrees
- moved Rcr4 140.3 mm to (46.8, 133.5), turned to 90 degrees
- moved Ur6 134.7 mm to (20.5, 146.1), turned to 0 degrees
- moved J4 130.6 mm to (24.5, 99.0), turned to 180 degrees
- moved Uf3 130.4 mm to (67.0, 32.7), turned to 0 degrees
- moved Uip1 123.8 mm to (119.3, 35.9), turned to 0 degrees
- moved Ur5 123.5 mm to (20.5, 137.3), turned to 0 degrees
- moved H1 122.9 mm to (15.0, 159.0), turned to 90 degrees
- moved Uf2 121.4 mm to (68.0, 42.2), turned to 0 degrees
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Connections:
- J4 pad 11: /membus11 -> /membus12
- J4 pad 13: /membus10 -> /membus13
- J4 pad 15: /membus9 -> /membus14
- J4 pad 17: /membus8 -> /membus15
- J4 pad 18: GND -> /clk
- J4 pad 3: /membus15 -> /membus8
- J4 pad 4: /clk -> GND
- J4 pad 5: /membus14 -> /membus9
- J4 pad 7: /membus13 -> /membus10
- J4 pad 9: /membus12 -> /membus11
- J5 pad 10: /memop2 -> GND
- J5 pad 11: /membus3 -> /membus4
- J5 pad 12: GND -> /memop2
- J5 pad 13: /membus2 -> /membus5
- J5 pad 14: /memop1 -> GND
- J5 pad 15: /membus1 -> /membus6
- J5 pad 17: /membus0 -> /membus7
- J5 pad 18: /memop0 -> GND
- J5 pad 3: /membus7 -> /membus0
- J5 pad 4: GND -> /memop0
- J5 pad 5: /membus6 -> /membus1
- J5 pad 7: /membus5 -> /membus2
- J5 pad 8: GND -> /memop1
- J5 pad 9: /membus4 -> /membus3
Other:
- board size 200 x 150 mm -> 150 x 150 mm
- board text added: "V mem V"
- board text added: "^ power supply ^"

Commit message: buscntrl placed
Parts:
- removed C1, C10, C11, C12, C13, C14, C2, C3, C4, C5, C6, C7, C8, C9, Cbc1, Cbc2, Cbc3, Cbd1, Cbd10, Cbd11, Cbd12, Cbd13, Cbd14, Cbd15, Cbd18, Cbd19, Cbd2, Cbd20, Cbd21, Cbd22, Cbd23, Cbd24, Cbd25, Cbd26, Cbd27, Cbd28, Cbd3, Cbd4, Cbd5, Cbd6, Cbd7, Cbd8, Cbd9, Cbu16, Cbu17, Cinsr1, Cinsr2, Cinsr4, Cip1, Cip2, Cip3, Cip4, Cip5, Cir1, Cir2, Cr1, Cr2, Cr3, Cr4: 100nF, Capacitor_SMD:C_0402_1005Metric
- removed D1: green, LED_SMD:LED_0603_1608Metric
- removed Dd1, Dd10, Dd11, Dd12, Dd13, Dd14, Dd15, Dd16, Dd17, Dd18, Dd19, Dd2, Dd20, Dd21, Dd22, Dd23, Dd24, Dd25, Dd26, Dd3, Dd4, Dd5, Dd6, Dd7, Dd8, Dd9: yellow, LED_SMD:LED_0603_1608Metric
- removed Dr1, Dr10, Dr11, Dr12, Dr13, Dr14, Dr15, Dr16, Dr17, Dr18, Dr19, Dr2, Dr20, Dr21, Dr22, Dr23, Dr24, Dr25, Dr26, Dr27, Dr28, Dr29, Dr3, Dr30, Dr31, Dr32, Dr33, Dr34, Dr35, Dr36, Dr37, Dr38, Dr39, Dr4, Dr40, Dr41, Dr42, Dr43, Dr44, Dr45, Dr46, Dr47, Dr48, Dr5, Dr6, Dr7, Dr8, Dr9: red, LED_SMD:LED_0603_1608Metric
- removed R33, Rcr1, Rcr2, Rcr3, Rcr4, Rcuc1, Rir1, Rir2, Rir3, Rir4, Rpd1, Rpd10, Rpd11, Rpd12, Rpd13, Rpd14, Rpd15, Rpd16, Rpd17, Rpd18, Rpd19, Rpd2, Rpd20, Rpd21, Rpd22, Rpd23, Rpd24, Rpd25, Rpd26, Rpd27, Rpd28, Rpd29, Rpd3, Rpd30, Rpd31, Rpd32, Rpd34, Rpd35, Rpd36, Rpd37, Rpd38, Rpd39, Rpd4, Rpd40, Rpd41, Rpd42, Rpd43, Rpd44, Rpd45, Rpd46, Rpd47, Rpd48, Rpd5, Rpd6, Rpd7, Rpd8, Rpd9: 10k, Resistor_SMD:R_0402_1005Metric
- removed Rd1, Rd10, Rd11, Rd12, Rd13, Rd14, Rd15, Rd16, Rd17, Rd18, Rd19, Rd2, Rd20, Rd21, Rd22, Rd23, Rd24, Rd25, Rd26, Rd3, Rd4, Rd5, Rd6, Rd7, Rd8, Rd9, Rio3, Rr1, Rr10, Rr11, Rr12, Rr13, Rr14, Rr15, Rr16, Rr17, Rr18, Rr19, Rr2, Rr20, Rr21, Rr22, Rr23, Rr24, Rr25, Rr26, Rr27, Rr28, Rr29, Rr3, Rr30, Rr31, Rr32, Rr33, Rr34, Rr35, Rr36, Rr37, Rr38, Rr39, Rr4, Rr40, Rr41, Rr42, Rr43, Rr44, Rr45, Rr46, Rr47, Rr48, Rr5, Rr6, Rr7, Rr8, Rr9: 680, Resistor_SMD:R_0402_1005Metric
- moved Ubc3 200.8 mm to (255.5, 154.0)
- moved Ucr2 199.4 mm to (207.0, 33.4), turned to 180 degrees
- moved Ucr1 195.9 mm to (197.5, 33.1), turned to 180 degrees
- moved U57 188.7 mm to (269.1, 54.3)
- moved SW1 187.5 mm to (179.0, -4.00)
- moved Ucr3 185.5 mm to (187.5, 22.4), turned to 0 degrees
- moved Uf1 180.9 mm to (257.0, 38.9)
- moved Uf5 177.0 mm to (259.5, 55.1)
- moved Uf2 176.6 mm to (244.5, 47.2), turned to 180 degrees
- moved Uf7 176.6 mm to (244.0, 37.2)
- moved Uf3 171.3 mm to (233.5, 72.9)
- moved Ur2 168.2 mm to (257.6, 91.8)
- moved Ur1 160.5 mm to (246.1, 92.2)
- moved Uf4 159.3 mm to (233.0, 55.8)
- moved Ubc1 151.5 mm to (46.5, -7.17), turned to 180 degrees
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Routing:
- net /membus15: track 0.00 -> 306.4 mm, vias 0 -> 11
- net /membus14: track 0.00 -> 304.3 mm, vias 0 -> 11
- net /membus11: track 0.00 -> 304.0 mm, vias 0 -> 11
- net /membus10: track 0.00 -> 302.7 mm, vias 0 -> 11
- net /membus13: track 0.00 -> 302.2 mm, vias 0 -> 11
- net /membus12: track 0.00 -> 299.4 mm, vias 0 -> 11
- net /membus9: track 0.00 -> 297.7 mm, vias 0 -> 11
- net /membus8: track 0.00 -> 294.8 mm, vias 0 -> 11
- net /regbus13: track 0.00 -> 255.1 mm, vias 0 -> 10
- net /regbus12: track 0.00 -> 251.7 mm, vias 0 -> 10
- net /regbus11: track 0.00 -> 245.9 mm, vias 0 -> 10
- net /regbus10: track 0.00 -> 245.2 mm, vias 0 -> 10
- net /regbus9: track 0.00 -> 240.9 mm, vias 0 -> 10
- net /regbus8: track 0.00 -> 239.6 mm, vias 0 -> 10
- net /regbus15: track 0.00 -> 236.6 mm, vias 0 -> 10
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Other:
- board text added: "buscntrl"
- board text added: "cyclereg"
- board text added: "flags"
- board text added: "instruction register"
- board text added: "intreg"
- board text added: "ip"
- board text added: "tempreg"

Commit message: every ic on layout
Parts:
- U57, Ubd19, Ubd20, Uf1, Uf2, Uf3, Uf4, Uf5, Uf6, Uf7, Uinsr1, Uip1, Uip2, Uip3, Uip4, Ur3, Ur4: moved to B.Cu
- moved Ur2 229.2 mm to (37.0, 154.0)
- moved Ur1 229.1 mm to (25.5, 154.0)
- moved Uip4 225.7 mm to (35.5, 97.0), turned to 90 degrees
- moved U57 218.5 mm to (53.5, 19.0), turned to 180 degrees
- moved Uf1 214.9 mm to (43.0, 19.8), turned to 180 degrees
- moved Uf7 212.5 mm to (31.5, 33.0), turned to 180 degrees
- moved Uf5 207.2 mm to (53.5, 32.5), turned to 180 degrees
- moved Uip3 203.9 mm to (49.0, 97.0), turned to 90 degrees
- moved Uf2 202.0 mm to (43.0, 33.0)
- moved Uf6 201.9 mm to (31.5, 19.8), turned to 180 degrees
- moved Uip2 197.4 mm to (62.8, 97.0), turned to 90 degrees
- moved Uip1 175.2 mm to (76.5, 97.0), turned to 90 degrees
- moved Uf3 173.8 mm to (64.5, 32.5), turned to 180 degrees
- moved Uf4 161.2 mm to (73.5, 32.5), turned to 180 degrees
- moved Ubc3 147.3 mm to (136.0, 68.0), turned to 0 degrees
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Routing:
- net /clk: track 3.25 -> 728.3 mm, vias 0 -> 3
- net /ControlUnit/srcsrc: track 0.00 -> 151.5 mm, vias 0 -> 2
- net /ControlUnit/intidsaved0: track 0.00 -> 148.8 mm, vias 0 -> 2
- net /ControlUnit/intidsaved2: track 0.00 -> 148.5 mm, vias 0 -> 2
- net /ioid0: track 0.00 -> 148.4 mm, vias 0 -> 4
- net /ControlUnit/intidsaved1: track 0.00 -> 148.3 mm, vias 0 -> 2
- net /iobus7: track 42.7 -> 180.7 mm, vias 3 -> 4
- net /iobus6: track 41.0 -> 177.9 mm, vias 3 -> 4
- net /iobus5: track 39.7 -> 175.4 mm, vias 3 -> 4
- net /iobus4: track 38.2 -> 172.5 mm, vias 3 -> 4
- net /ControlUnit/next_instr: track 0.00 -> 133.4 mm, vias 0 -> 2
- net /iobus3: track 37.6 -> 170.7 mm, vias 3 -> 4
- net /iobus2: track 36.7 -> 169.4 mm, vias 3 -> 4
- net /iobus1: track 37.1 -> 169.7 mm, vias 3 -> 4
- net /iobus0: track 37.4 -> 169.5 mm, vias 3 -> 4
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