File: PCB/Kicad/gpu/gpu/gpu.kicad_sch (KiCad schematic)
At the start: 0 parts

Commit message: Kicad implementation
Parts:
- added VRAM1: 71342LA20PFG8, mALUch_lib:QFP80P1600X1600X160-64N, symbol 71342LA20PFG8:71342LA20PFG8
- added char_rom1: AT28C64B-15PU, Package_DIP:DIP-28_W15.24mm_SMDSocket_SmallPads, symbol AT28C64B-15PU:AT28C64B-15PU
- added pixel_mux1: 74LS151, Package_DIP:DIP-16_W8.89mm_SMDSocket_LongPads, symbol 74xx:74LS151
Connections:
- new net GND: VRAM1.25 (GND), VRAM1.55 (~{CER}), VRAM1.59 (R/~{WL}), char_rom1.2 (A12), char_rom1.20 (~{CE}), char_rom1.22 (~{OE}), pixel_mux1.7 (~{E}), pixel_mux1.8 (GND)
- new net Hcount0: pixel_mux1.11 (S0)
- new net Hcount1: pixel_mux1.10 (S1)
- new net Hcount2: pixel_mux1.9 (S2)
- new net Hcount3: VRAM1.47 (A0R)
- new net Hcount4: VRAM1.46 (A1R)
- new net Hcount5: VRAM1.45 (A2R)
- new net Hcount6: VRAM1.44 (A3R)
- new net Hcount7: VRAM1.43 (A4R)
- new net Hcount8: VRAM1.42 (A5R)
- new net HostA0: VRAM1.2 (A0L)
- new net HostA1: VRAM1.3 (A1L)
- new net HostA10: VRAM1.62 (A10L)
- new net HostA11: VRAM1.61 (A11L)
- new net HostA2: VRAM1.4 (A2L)
- new net HostA3: VRAM1.5 (A3L)
- new net HostA4: VRAM1.6 (A4L)
- new net HostA5: VRAM1.7 (A5L)
- new net HostA6: VRAM1.8 (A6L)
- new net HostA7: VRAM1.10 (A7L)
- new net HostA8: VRAM1.11 (A8L)
- new net HostA9: VRAM1.12 (A9L)
- new net HostD0: VRAM1.14 (I/O0L)
- new net HostD1: VRAM1.15 (I/O1L)
- new net HostD2: VRAM1.16 (I/O2L)
- new net HostD3: VRAM1.17 (I/O3L)
- new net HostD4: VRAM1.19 (I/O4L)
- new net HostD5: VRAM1.20 (I/O5L)
- new net HostD6: VRAM1.21 (I/O6L)
- new net HostD7: VRAM1.22 (I/O7L)
- new net Output/PixIn: pixel_mux1.5 (Z)
- new net ReadA10: VRAM1.51 (A10R)
- new net ReadA11: VRAM1.52 (A11R)
- new net ReadA6: VRAM1.41 (A6R)
- new net ReadA7: VRAM1.39 (A7R)
- new net ReadA8: VRAM1.38 (A8R)
- new net ReadA9: VRAM1.37 (A9R)
- new net ReadD0: VRAM1.26 (I/O0R)
- new net ReadD1: VRAM1.27 (I/O1R)
- new net ReadD2: VRAM1.28 (I/O2R)
- new net ReadD3: VRAM1.29 (I/O3R)
- new net ReadD4: VRAM1.31 (I/O4R)
- new net ReadD5: VRAM1.32 (I/O5R)
- new net ReadD6: VRAM1.33 (I/O6R)
- new net ReadD7: VRAM1.34 (I/O7R)
- new net VCC: VRAM1.1 (~{OEL}), VRAM1.53 (~{SEM_R}), VRAM1.54 (R/~{WR}), VRAM1.57 (VCC), VRAM1.60 (~{SEML}), char_rom1.27 (~{WE}), char_rom1.28 (VCC), pixel_mux1.16 (VCC)
- new net Vcount0: char_rom1.21 (A10)
- new net Vcount1: char_rom1.23 (A11)
- new net Vcount2: char_rom1.24 (A9)
- new net Vcount3: char_rom1.25 (A8)
- new net charRow0: char_rom1.14 (GND), pixel_mux1.4 (I0)
- new net charRow1: char_rom1.13 (I/O2), pixel_mux1.3 (I1)
- new net charRow2: char_rom1.12 (I/O1), pixel_mux1.2 (I2)
- new net charRow3: char_rom1.11 (I/O0), pixel_mux1.1 (I3)
- new net charRow4: char_rom1.15 (I/O3), pixel_mux1.15 (I4)
- new net charRow5: char_rom1.16 (I/O4), pixel_mux1.14 (I5)
- new net charRow6: char_rom1.17 (I/O5), pixel_mux1.13 (I6)
- new net charRow7: char_rom1.18 (I/O6), pixel_mux1.12 (I7)
- new net charRow8: char_rom1.19 (I/O7)
- new net nHostW: VRAM1.58 (~{CEL})
- new net readD0: char_rom1.10 (A0)
- new net readD1: char_rom1.9 (A1)
- new net readD2: char_rom1.8 (A2)
- new net readD3: char_rom1.7 (A3)
- new net readD4: char_rom1.6 (A4)
- new net readD5: char_rom1.5 (A5)
- new net readD6: char_rom1.4 (A6)
- new net readD7: char_rom1.3 (A7)
- no-connect marks 0 -> 17
Other:
- added sheet Output (output.kicad_sch)
- sheet VGA Synchronization ports: added HSYNC_OUT, Hcount, VSYNC_OUT, Vcount, Vis, nRST, pixel_clk; removed none
- sheet commands ports: added BG[0..7], CLK, FG[0..7], IOWE, io[0..15]; removed none
- note added: "Host Interface"
- note added: "OUTPUT"
